File: pcb/r2-mainboard/fpga_config.kicad_sch (KiCad schematic)
At the start: 0 parts

Commit message: R2: WP5 -- fpga_config ported (bank 2, config pins, clock, JTAG)
Units 3 and 5 of the XC6SLX16: bank 2's I/O, the dedicated configuration pins,
the 33.33 MHz oscillator and the JTAG group. Ported by tools/port_r1.py; the new
content this sheet needs (config NOR, the M1 strap change, the debug header, an
INIT_B pull-up) is NOT here yet and comes next.

A STALE RAIL, CAUGHT BY THE NETLIST DIFF
R1 spreads the FPGA's decoupling across sheets, so five of the DDR bank's VCCO
capacitors are drawn on fpga_config rather than fpga_ddr. They ported across as
`+1V35` -- the name retired in 8b69e01 when the bank moved to 1.5 V. ERC was
silent about it; the netlist diff showed a new 5-node +1V35 net appearing out of
nowhere. Fixed through RAILS, and +1V5 now carries C316/C448/C457/C485/C489
alongside the existing power_mon shunt. fpga_ddr carries the same name in five
places and will need the same treatment.

That is the third time this session that a netlist node-diff caught something
ERC did not: the U11 deletion, the fpga_io cross-sheet short, and now this.

R1 LEAVES INIT_B UNCONNECTED
FPGA_INIT is a *local* label on R1 whose net has exactly one member, U41.R3 --
no pull-up, no route anywhere. The HIER mapping assumed it was a sheet-level
signal and the tool's own guard rejected it, which is how it came to light. It
stays local through the port so the sheet matches R1, but it matters more in R2
than in R1: with self-boot, INIT_B low is how firmware tells a CRC error from
"still configuring" when DONE never arrives. Giving it a pull-up and a route to
the MCU is a separate change.

THE 14 LVDS BALLS ARE DROPPED
R2 deletes the PTN3460 that drove the FPD-Link input, so those balls have no
source. Left as constrained-but-floating LVDS_33 inputs with DIFF_TERM enabled,
seven differential buffers would sit at an indeterminate common mode where they
can self-oscillate and draw current -- in the reading state, the one number R2
exists to reduce. The owner's decision (2026-08-12) is to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
Parts:
- added C316, C326, C392, C393, C448, C449, C450, C456: 22uF/6.3V, Capacitor_SMD:C_0603_1608Metric, symbol Device:C
- added C457, C482, C483, C484: 4.7uF/6.3V, Capacitor_SMD:C_0402_1005Metric, symbol Device:C
- added C485, C486, C487, C488, C489, C490, C507: 470nF/25V, Capacitor_SMD:C_0402_1005Metric, symbol Device:C
- added R335, R336: 5.1K/1%, Resistor_SMD:R_0402_1005Metric, symbol Device:R
- added R337: 1K/1%, Resistor_SMD:R_0402_1005Metric, symbol Device:R
- added R409: 33R/1%, Resistor_SMD:R_0402_1005Metric, symbol Device:R
- added U41: XC6SLX-FTG256, footprints:Xilinx_FTG256, symbol symbols:XC6SLX-FTG256
- added X1: 33.33MHz, Oscillator:Oscillator_SMD_Abracon_ASE-4Pin_3.2x2.5mm, symbol Oscillator:ASE-xxxMHz
Connections:
- new net: R409.1, X1.3 (OUT)
- new net +1V5: C316.1, C448.1, C457.1, C485.1, C489.1
- new net +3V3: C326.1, C392.1, C393.1, C449.1, C450.1, C456.1, C482.1, C483.1, C484.1, C486.1, C487.1, C488.1, C490.1, C507.2, R335.1, R337.1, U41.N10 (VCCO_2), U41.N11 (IO_L13P_M1_2), U41.N7 (VCCO_2), U41.R4 (VCCO_2), U41.R8 (VCCO_2), U41.T11 (IO_L1N_M0_CMPMISO_2), X1.1 (EN), X1.4 (Vdd)
- new net FPGA_CLK33: R409.2, U41.M9 (IO_L29P_GCLK3_2)
- new net FPGA_CS: U41.L10 (IO_L16P_2)
- new net FPGA_DONE: R337.2, U41.P13 (DONE_2)
- new net FPGA_INIT: U41.R3 (IO_L65P_INIT_B_2)
- new net FPGA_MISO: U41.T10 (IO_L3N_MOSI_CSI_B_MISO0_2)
- new net FPGA_MOSI: U41.P10 (IO_L3P_D0_DIN_MISO_MISO1_2)
- new net FPGA_PROG#: R335.2, U41.T2 (PROGRAM_B_2)
- new net FPGA_SCLK: U41.R11 (IO_L1P_CCLK_2)
- new net FPGA_SUSP: R336.1, U41.P14 (SUSPEND)
- new net FPGA_TCK: U41.C14 (TCK)
- new net FPGA_TDI: U41.C12 (TDI)
- new net FPGA_TDO: U41.E14 (TDO)
- new net FPGA_TMS: U41.A15 (TMS)
- new net GND: C316.2, C326.2, C392.2, C393.2, C448.2, C449.2, C450.2, C456.2, C457.2, C482.2, C483.2, C484.2, C485.2, C486.2, C487.2, C488.2, C489.2, C490.2, C507.1, R336.2, X1.2 (GND)
- no-connect marks 0 -> 32
Other:
- note added: "VCCO0"
- note added: "VCCO1"
- note added: "VCCO2"
- note added: "VCCO3"
- company: (none) -> Copyright 2025 Modos Tech Inc

Commit message: R2: WP5 -- fpga_config gains the config NOR, master-SPI strap and INIT_B pull-up
The new content the port could not carry. tools/patch_fpga_config_nor.py builds it
with schgen and splices it into the ported sheet, so the port stays reproducible
and this stays separately reviewable.

THE MODE STRAP IS ONE WIRE
UG380 Table 2-1: Master Serial/SPI is M[1:0] = 01 with CCLK an output; Slave
Serial, which R1 uses, is 11. R1 straps both mode pins high, so only M1 moves --
#PWR0261 on ball N11 (IO_L13P_M1_2) goes from +3V3 to GND. UG380 also requires
the mode pins be tied directly to ground or VCCO_2 rather than through resistors,
so this is a wire and not a pull-down. Verified in the netlist: N11 -> GND,
T11 -> +3V3.

THE NOR
W25Q128JVSIQ, LCSC C97521, a JLC Basic part at $1.22 -- already scouted in
NOTES-R2-hardware-facts.md. 16 MB where the plan asked for 4, taken anyway
because Basic parts carry no per-part setup fee. KiCad has both the symbol
(Memory_Flash:W25Q128JVS, a derived symbol that schgen flattens from
W25Q32JVSS) and the footprint (SOIC-8_5.3x5.3mm_P1.27mm), so nothing is authored.

CSO_B on ball T3 was unconnected in R1 -- the one pin master-SPI needs was
already free. Its no-connect flag is removed and it now carries NOR_CS#, along
with R410 (10k pull-up) and R411 (100R series limit on the SoM's chip select,
because the FPGA drives CSO_B during configuration and the two contend if
software gets the order wrong). ~WP and ~HOLD are tied high on a shared stub:
bitgen runs SPI_buswidth:1, so IO2 and IO3 are never data and must not float.

The pull-up matters more than it looks. bitgen currently runs
-g UnusedPin:PullDown and CSO_B is not in the UCF, so after configuration the
FPGA would weakly hold the flash *selected* while CSR traffic clocks past it.
The agreed fix is on the gateware side -- assign CSO_B and drive it high in
top.v -- and R410 is the board's backstop either way. That gateware edit is not
made yet.

An on-sheet note explains the one genuinely con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
Parts:
- added C508: 100nF/16V, Capacitor_SMD:C_0402_1005Metric, symbol Device:C
- added R410: 10k, Resistor_SMD:R_0402_1005Metric, symbol Device:R
- added R411: 100R, Resistor_SMD:R_0402_1005Metric, symbol Device:R
- added R414: 4.7k, Resistor_SMD:R_0402_1005Metric, symbol Device:R
- added U42: W25Q128JVSIQ, Package_SO:SOIC-8_5.3x5.3mm_P1.27mm, symbol Memory_Flash:W25Q128JVS
Connections:
- net +3V3: now also C508.1, R410.1, R414.1, U42.3 (~{WP}/IO_{2}), U42.7 (~{HOLD}/~{RESET}/IO_{3}), U42.8 (VCC); no longer U41.N11 (IO_L13P_M1_2)
- net FPGA_INIT: now also R414.2
- net FPGA_MISO: now also U42.5 (DI/IO_{0})
- net FPGA_MOSI: now also U42.2 (DO/IO_{1})
- net FPGA_SCLK: now also U42.6 (CLK)
- net GND: now also U41.N11 (IO_L13P_M1_2), C508.2, U42.4 (GND)
- net NOR_CS#: now reaches U41.T3 (IO_L65N_CSO_B_2)
- net NOR_CS#: now also R410.2, R411.2, U42.1 (~{CS})
- new net NOR_CS: R411.1
- no-connect marks 32 -> 30
Other:
- note added: "Config NOR -- the FPGA boots itself: master SPI,"
- note added: "FPGA_MISO drives the NOR's DI. Three masters share"
- note added: "LOOK inverted: FPGA_MOSI is data toward the FPGA, so it"
- note added: "M[1:0]=01 (UG380 Table 2-1), CCLK an output while"
- note added: "configuring. The net names are host-centric and only"
- note added: "lands on the FPGA's DIN pin and on the NOR's DO, and"
- note added: "these wires -- see docs/fpga.md for the direction table."
