File: pcb/r2-mainboard/fpga_config.kicad_sch (KiCad schematic)
At the start: 30 parts, among them U41 XC6SLX-FTG256, U42 W25Q128JVSIQ, X1 33.33MHz

Commit message: R2: WP5 -- NOR IO2/IO3 reach the FPGA, so x4 boot stays a software change
Owner's decision, 2026-08-13, after the numbers came out of UG380 and DS162.

The config NOR exists to cut resume latency: R1 reloads the bitstream from the
MCU's SPIFFS on every wake and measures 360-400 ms, and +1V2_FPGA is off in
standby so that happens every time. Self-boot only pays if it is faster, and
how much faster is set by the configuration clock rate and the SPI bus width.

    bitstream                3,731,264 bits   UG380 Table 5-5, XC6SLX16
    max master CCLK          40 MHz           DS162 FMCCK, -3 speed grade
    master CCLK tolerance    +-50%            DS162 FMCCKTOL

    x1 @ ConfigRate 2 (today) 1866 ms typ   <- 5x WORSE than R1
    x1 @ ConfigRate 22         170 ms typ   (339 ms worst case)
    x4 @ ConfigRate 22          42 ms typ   ( 85 ms worst case)

Bus width is the only one of the two with a board cost, and it was nearly free
now and a respin later. UG380 Figure 2-13's x4 connection was already wired
except its top two rows: MISO[2] (N12) to the flash's WP#/IO2 and MISO[3] (P12)
to HOLD#/IO3. Both balls were spare and no-connect flagged -- no .ucf ever names
them, because they are dedicated configuration pins.

On the NOR side pins 3 and 7 were tied hard to +3V3, which is right for x1 and
wrong for x4; Figure 2-13 note 4 asks for pull-ups to VCCO_2 instead, so the tie
becomes R412/R413, 10k. Nothing about the board's behaviour changes today: in x1
the pull-ups hold WP#/HOLD# high exactly as the hard tie did.

Two consequences belong to Caster, not to the schematic, and are written on the
page and into the commit rather than silently assumed:
  - ConfigRate must be raised or the NOR is a latency *regression*
  - -g UnusedPin:PullDown would pull N12/P12 against the new 10k pull-ups after
    configuration. Harmless (the NOR is idle, and a SoM-driven NOR write holds
    PROG# low so the FPGA tri-states and the pull-ups win), but it should be an
    explicit PULLUP c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
Parts:
- added R412, R413: 10k, Resistor_SMD:R_0402_1005Metric, symbol Device:R
Connections:
- net +3V3: now also R412.1, R413.1; no longer U42.3 (~{WP}/IO_{2}), U42.7 (~{HOLD}/~{RESET}/IO_{3})
- net NOR_IO2: now reaches U41.N12 (IO_L12P_D1_MISO2_2)
- net NOR_IO2: now also U42.3 (~{WP}/IO_{2}), R412.2
- net NOR_IO3: now reaches U41.P12 (IO_L12N_D2_MISO3_2)
- net NOR_IO3: now also U42.7 (~{HOLD}/~{RESET}/IO_{3}), R413.2
- no-connect marks 30 -> 28
Other:
- note added: "Nothing changes in x1: the pull-ups hold WP#/HOLD# high as the tie did."
- note added: "Owed in Caster: -g ConfigRate 2 -> 22 (2 makes self-boot 1.9 s, five times"
- note added: "R412/R413 and the two nets to N12/P12 exist so that master-SPI x4 boot is"
- note added: "a gateware change, not a respin. UG380 Fig 2-13; its note 4 requires these"
- note added: "on N12/P12 so -g UnusedPin:PullDown does not fight R412/R413."
- note added: "pull-ups to VCCO_2, which is why pins 3/7 are no longer tied hard to +3V3."
- note added: "slower than R1's 360-400 ms), -g Binary:no -> yes, and a PULLUP constraint"

Commit message: R2: MPNs into the schematic -- and five caps carry the wrong part number
Sourcing data lived in docs/*.md, not in the schematic, so the BOM the
fab would read had 3 of 96 lines with an MPN. Resolved every LCSC code
already on the board against LCSC's own catalogue and wrote MPN +
Manufacturer back: 53 -> 60 lines, 218 components. Added LCSC codes for
L10-L13, U42 and J22/J23 from the per-sheet docs.

Verified before writing: 321 refs and 519 nets identical before and
after, no duplicated properties, pre-existing MPNs untouched.

Cross-checking each passive value against the part its LCSC code
actually names found five wrong ones, all of them the ADC sense-divider
filter caps on power_mon:

  C91                 1nF/50V  carries C131394  = 100 nF
  C163 C164 C168 C169 1nF/25V  carries C6119801 = 470 nF

Left unwritten rather than cementing the error. C1523 (0402B102K500NT,
1 nF 50 V X7R 0402, JLC Basic, 5.3 M stock) covers both positions.

Also held back: U41, whose C39313 is XC6SLX16-**2**FTG256C while
fpga.md specifies the -3 speed grade.

frontlight.md cites C1848394 as the FPC connector on J22/J23; that code
is TPS22914BYFPR. The 6-pin sibling of J24's C5213749 is C5213748.

Co-Authored-By: Claude Opus 5 <noreply@anthropic.com>
Claude-Session: https://claude.ai/code/session_01MnesETWABbVdbcVnCKfKVs
Parts:
- C316, C326, C392, C393, C448, C449, C450, C456: MPN (none) -> CL10A226MQ8NRNC; Manufacturer (none) -> Samsung Electro-Mechanics
- C457, C482, C483, C484: MPN (none) -> CL05A475MQ5NRNC; Manufacturer (none) -> Samsung Electro-Mechanics
- C485, C486, C487, C488, C489, C490, C507: MPN (none) -> CGA0402X5R474K250GT; Manufacturer (none) -> HRE
- R335, R336: MPN (none) -> 0402WGF5101TCE; Manufacturer (none) -> UNI-ROYAL
- R337: MPN (none) -> 0402WGF1001TCE; Manufacturer (none) -> UNI-ROYAL
- R409: MPN (none) -> 0402WGF330JTCE; Manufacturer (none) -> UNI-ROYAL
- U42: LCSC (none) -> C97521; MPN (none) -> W25Q128JVSIQ; Manufacturer (none) -> Winbond
- X1: MPN (none) -> 1532H-33.333JWVDTSL; Manufacturer (none) -> HCI
