File: pcb/r2-mainboard/fpga_config.kicad_sch (KiCad schematic)
At the start: 32 parts, among them U41 XC6SLX-FTG256, U42 W25Q128JVSIQ, X1 33.33MHz

Commit message: R2: the six approved edits, and one of them was already done
Owner-approved 2026-08-19, KiCad closed for the pass.

1. R225 22k -> 20.5K/1%, LCSC C57105 (0402WGF2052TCE, UNI-ROYAL, the
   family the rest of the board already uses). Rendered and checked:
   R224 390k over R225 20.5k with R213 100k injecting VGH_DAC, so
   20.5||100 = 17.01k and VGH = 1.2 x (1 + 390/17.01) = 28.71 V at
   DAC = 0 -- exactly epd-port.md 10.3's target.
2. The five sense-divider caps that carried codes for the wrong
   capacitance -> C1523 (0402B102K500NT, 1 nF 50 V X7R, JLC Basic,
   5.3 M stock). One part covers both the 25 V and 50 V positions.
2b. R88/R224 -> C54920667 (HRC0402F3903DNTO, 390k 1%, 20 k stock).
   C25782 had 14 units against two per board. The owner found this one;
   both obvious alternatives were traps -- C23150 is 0603, and C44937
   is 3.9 ohm despite "390K" in its part number.
3. C147 set DNP rather than deleted. panel.md 7 had already ruled that
   J6.7/J6.44 stay; that covered the pins but not the capacitor on the
   dead net. DNP drops it from placement, keeps the topology of a frozen
   sheet untouched, and leaves the footprint if a future panel drives
   the rail. in_bom stays yes -- that is this board's convention for all
   13 DNP parts, so they show up flagged rather than vanishing.
4. Ten duplicate #PWR references renumbered to #PWR1112-1121 on the
   battery sheet, which was the colliding side in every case.
5. J3 was already deleted on 2026-08-15. No work needed.
6. Specter -> Reflow across 22 files: 14 sheets, 7 generators, the
   project file. .history/ deliberately untouched.

Verified as one change: netlist before and after has 518 nets with
identical pin membership, and epd_power and epd were rendered to PNG and
inspected.

Docs updated to match: epd-port.md 10 is applied rather than designed,
frontlight.md 1 loses the "9 in series is inferred" hedge (the vendor
listing confirms 2 x 9), and io-expansion.md 4's "only guess on this
sheet" is resolved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
Other:
- title: Glider-R2 / Specter mainboard -> Glider-R2 / Reflow mainboard
Changed lines of the file:
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@@
 	(paper "A4")
 	(title_block
-		(title "Glider-R2 / Specter mainboard")
+		(title "Glider-R2 / Reflow mainboard")
 		(date "2026-08-07")
 		(rev "A")

Commit message: R2: two interrupts that could never fire, and the SoM footprint
The EXTI collisions mcu.md §3.4 found are applied. An EXTI line is picked
by the pin's *number*, so TOUCH_INT# on PC3 was fighting PD3 GAUGE_ALRT#
and PEN_INT# on PC6 was fighting PD6 QON_SNS -- as drawn neither touch nor
pen could raise an interrupt at all. Each swaps with an output, which needs
no line, so it costs nothing. FL_INT# gets PB12 at the same time, which was
frontlight.md §10.3's own first suggestion; §9's later push for PB7 was
wrong, because PC7 KEY_PREV# holds EXTI7.

518 -> 517 nets, the drop being the PB12 unconnected- pseudo-net, and
exactly five membership changes. Every hierarchical label in the project
now has a counterpart -- DANGLING_OK is empty and ERC excluding
footprint_link_issues is 32, down from 105.

The PCM-071 footprint is built rather than downloaded, because two drawings
have landed that over-determine it: Samtec's own vector land pattern (parsed
from the content stream, every measurement agreeing with a printed dimension
to under 1 um) and L-1038e.A5 Figure 7, which is a carrier-board drawing.
The trap it contains is that the alignment hole is NOT on the connector's
centreline -- it is 1.054 mm from one row and 5.118 from the other, and
Figure 7 dimensions the holes, so assuming a centred hole puts both
connectors 2.06 mm out. The check worth trusting is the one nothing forces:
the B and C rows land 0.982 and 0.998 mm inside the module's edges.

Also: U41's speed grade is settled -2 -- LCSC has no -3 in FTG256 at all,
and caster.xise's -3 is ISE's untouched default (valueState="default"), not
a choice anyone made. But -2's MCB is rated 667 Mb/s against the 666.67 this
design runs, so fpga.md §1.1 asks for one free ISE build before the order.

And a bring-up landmine: epd_pos_rails_good() accepts VGH <= 28.0 V while
R2's own R225 change puts it at 28.41 V nominal. A correctly built board
would fatal() at every EPD power-up. epd-port.md §10.5.

Co-Authored-By: Claude Op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
Parts:
- U41: MPN (none) -> XC6SLX16-2FTG256C; Manufacturer (none) -> AMD/XILINX
Changed lines of the file:
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@@
+			)
+		)
+		(property "MPN" "XC6SLX16-2FTG256C"
+			(at 144.78 58.42 0)
+			(hide yes)
+			(show_name no)
+			(do_not_autoplace no)
+			(effects
+				(font
+					(size 1.27 1.27)
+				)
+			)
+		)
+		(property "Manufacturer" "AMD/XILINX"
+			(at 144.78 60.96 0)
+			(hide yes)
+			(show_name no)
+			(do_not_autoplace no)
+			(effects
+				(font
+					(size 1.27 1.27)
+				)
 			)
 		)
