File: pcb/r2-mainboard/mcu.kicad_sch (KiCad schematic)
At the start: 0 parts

Commit message: R2: capture mcu.kicad_sch -- STM32G0 housekeeping and the pin assignment
WP3. The sheet is small; the deliverable is the pin assignment, which is
one-shot because STM32 peripheral functions are fixed to particular pins.
Every choice is checked against datasheets/stm32g0b1.pdf (DS13560 Rev 1)
Table 12 column "LQFP64 - GP" and Tables 13-20.

STM32G0B1RCT6, LQFP-64, C3034735 (6029 in stock, $1.67). Chosen for its two
12-bit DACs -- R1 drives VCOM and VGH from DAC_CHANNEL_1/2, and most of the
G0 line has no DAC -- and for 60 I/O against a signal count of 49. Stop 1
with the RTC running is 3.7 uA typ, so the always-on domain costs ~14 uW.

Two decisions worth the reading:

- The SoM, not the MCU, drives Caster's CSR bus. Caster/rtl/csr.v is a 4-wire
  SPI slave carrying waveform LUTs, OSD bitmaps and per-page op commands; R1
  held that data in SPIFFS beside the MCU, and R2 deletes that flash. The MCU
  keeps only FPGA_PROG#/DONE/SUSP, which are power-domain signals. Decided by
  the hardware owner.
- The power button never touches the MCU's supply domain. QON idles at 4.3 V
  behind a 200 k internal pull-up (bq25890.pdf), and in ship mode +3V3_AON
  does not exist at all -- so SW20 shorts QON straight to GND, the MCU only
  listens through R41, and PD6 must have its internal pulls disabled.

EXTI lines are deconflicted by hand: on G0 an EXTI line is selected by pin
number across all ports, so the three wake sources and four charger inputs
each take a distinct index. That constraint is invisible in a pin count.

Verified: ERC 186 violations, one real (the +3V3_AON PWR_FLAG on the battery
sheet, still yours to delete); a script re-read the exported netlist and
asserted all 50 assignments land on the port they claim and that the
unconnected set is exactly the 11 reserved pins; cross-sheet names and
directions match power and battery exactly. battery.kicad_sch and
power.kicad_sch are untouched.

Co-Authored-By: Claude Opus 5 <noreply@anthropic.com>
Claude-Session: https://c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
Parts:
- added C40: 4.7uF/10V, Capacitor_SMD:C_0603_1608Metric, symbol Device:C
- added C41, C42, C44, C45, C48, C49, C50: 100nF/16V, Capacitor_SMD:C_0402_1005Metric, symbol Device:C
- added C43: 1uF/16V, Capacitor_SMD:C_0402_1005Metric, symbol Device:C
- added C46, C47: 18pF/50V, Capacitor_SMD:C_0402_1005Metric, symbol Device:C
- added D20: GREEN, LED_SMD:LED_0603_1608Metric, symbol Device:LED
- added FB20: 120R@100M, Inductor_SMD:L_0402_1005Metric, symbol Device:FerriteBead
- added J20: SWD (DNP), Connector_PinHeader_2.54mm:PinHeader_1x05_P2.54mm_Vertical, symbol Connector_Generic:Conn_01x05
- added R40: 10k, Resistor_SMD:R_0402_1005Metric, symbol Device:R
- added R41, R44: 1k, Resistor_SMD:R_0402_1005Metric, symbol Device:R
- added R42, R43: 100k, Resistor_SMD:R_0402_1005Metric, symbol Device:R
- added SW20, SW21, SW22: SW, Button_Switch_SMD:SW_Push_1P1T_XKB_TS-1187A, symbol Switch:SW_Push
- added U20: STM32G0B1RCT6, Package_QFP:LQFP-64_10x10mm_P0.5mm, symbol MCU_ST_STM32G0:STM32G0B1RCTx
- added Y20: 32.768kHz, Crystal:Crystal_SMD_3215-2Pin_3.2x1.5mm, symbol Device:Crystal
Connections:
- new net: D20.2 (A), R44.1
- new net +3V3_AON: C40.1, C41.1, C42.1, D20.1 (K), FB20.1, J20.1 (Pin_1), R42.1, R43.1, U20.6 (VBAT), U20.8 (VDD)
- new net +3V3_VREF: C43.1, C44.1, FB20.2, U20.7 (VREF+)
- new net CHG_CE#: U20.55 (PD5)
- new net CHG_INT#: U20.50 (PD0)
- new net CHG_OTG: U20.57 (PB3)
- new net CHG_PG#: U20.52 (PD2)
- new net CHG_QON#: C50.1, R41.2, SW20.1
- new net CHG_STAT#: U20.54 (PD4)
- new net EPD_POS_EN: U20.28 (PB1)
- new net EPD_PWR_EN: U20.27 (PB0)
- new net EPD_THROT: U20.31 (PB11)
- new net FL_EN: U20.59 (PB5)
- new net FL_PWM1: U20.60 (PB6)
- new net FL_PWM2: U20.61 (PB7)
- new net FPGA_DONE: U20.34 (PB14)
- new net FPGA_PROG#: U20.33 (PB13)
- new net FPGA_SUSP: U20.35 (PB15)
- new net GAUGE_ALRT#: U20.53 (PD3)
- new net GND: C40.2, C41.2, C42.2, C43.2, C44.2, C45.2, C46.2, C47.2, C48.2, C49.2, C50.2, J20.3 (Pin_3), R40.2, SW20.2, SW21.2, SW22.2, U20.9 (VSS)
- new net KEY_NEXT#: C49.1, R43.2, SW22.1, U20.40 (PD8)
- new net KEY_PREV#: C48.1, R42.2, SW21.1, U20.39 (PC7)
- new net LED_STAT#: R44.2, U20.15 (PC2)
- new net MCU_EN_3V3: U20.11 (PF1)
- new net MCU_EN_5V: U20.10 (PF0)
- new net MCU_EN_DDR: U20.14 (PC1)
- new net MCU_EN_FPGA_CORE: U20.13 (PC0)
- new net MCU_NRST: C45.1, J20.5 (Pin_5), U20.12 (PF2)
- new net MCU_RXD: U20.42 (PA10/UCPD1_DBCC2)
- new net MCU_SWCLK: J20.2 (Pin_2), R40.1, U20.46 (PA14)
- new net MCU_SWDIO: J20.4 (Pin_4), U20.45 (PA13)
- new net MCU_TXD: U20.37 (PA9/UCPD1_DBCC1)
- new net OSC32_IN: C46.1, U20.4 (PC14), Y20.1
- new net OSC32_OUT: C47.1, U20.5 (PC15), Y20.2
- new net PG_1V2: U20.2 (PC12)
- new net PG_1V35: U20.1 (PC11)
- new net PG_3V3: U20.3 (PC13)
- new net QON_SNS: R41.1, U20.56 (PD6)
- new net SCL_AON: U20.62 (PB8)
- new net SDA_AON: U20.63 (PB9)
- new net SOM_IRQ#: U20.58 (PB4)
- new net SOM_RESET#: U20.47 (PA15)
- new net SOM_WAKE#: U20.36 (PA8)
- new net VBUS_DET: U20.51 (PD1)
- new net VBUS_MEA: U20.24 (PA7)
- new net VCOM_DAC: U20.21 (PA4)
- new net VCOM_EN: U20.29 (PB2)
- new net VCOM_MEA: U20.23 (PA6)
- new net VCOM_MEA_EN: U20.30 (PB10)
- new net VGH_DAC: U20.22 (PA5)
- new net VGH_MEA: U20.19 (PA2)
- new net VGL_MEA: U20.20 (PA3)
- new net VN_MEA: U20.18 (PA1)
- new net VP_MEA: U20.17 (PA0)
- no-connect marks 0 -> 11
Other:
- note added: "+5V_DCDC. docs/mcu.md §4."
- note added: "200 k internal pull-up (bq25890.pdf) and PD6 is a 5 V-tolerant FT pin, so firmware must leave that pin's internal pull-up/pull-down"
- note added: "32.768 kHz LSE"
- note added: "4-wire SPI slave, and the LUT/OSD data it carries lives on the SoM's"
- note added: "Buttons"
- note added: "CL = C1·C2/(C1+C2) + Cstray. A 12.5 pF crystal with ~3 pF of stray"
- note added: "Confirm before layout, and check drive level. docs/mcu.md §9."
- note added: "DISABLED (Table 21 note 2). A 15 s hold forces a BATFET reset, so a clean shutdown has to finish well inside 12 s."
- note added: "Figure 15, p.65: 100 nF + 4.7 uF on VDD/VDDA, 100 nF + 1 uF on VREF+."
- note added: "J20 is pads only, not fitted — the device has to stay thin. Order"
- note added: "LAYOUT — the caution under that figure asks for these directly at, or"
- note added: "MCU_TXD and MCU_RXD are named from the MCU's point of view. On"
- note added: "R40: PA14 is SWCLK *and* BOOT0 (Table 12, p.53). Reset already"
- note added: "Reset and SWD"
- note added: "SOM_WAKE#, SOM_IRQ#, SOM_RESET# and FPGA_PROG# are open-drain: they"
- note added: "SW20 shorts CHG_QON# straight to GND — what the charger expects, and the only path that still works with the MCU unpowered:"
- note added: "Sheet interface"
- note added: "Status LED"
- note added: "Supply and decoupling"
- note added: "The SoM, not the MCU, drives Caster's CSR bus — Caster/rtl/csr.v is a"
- note added: "UART TX idles high, so firmware must release it before cutting"
- note added: "VDD/VDDA (8) VBAT (6)"
- note added: "VDDA is merged into the VDD pin on STM32G0, so FB20 isolates the ADC"
- note added: "VREF+ (7)"
- note added: "applies an internal pull-down (note 4) and nBOOT_SEL defaults to"
- note added: "below, their own pins: C40/C41 at pin 8, C43/C44 at pin 7."
- note added: "booting from the option bytes; R40 makes that unconditional."
- note added: "eMMC. The MCU keeps only FPGA_PROG#/DONE/SUSP, which are power-domain"
- note added: "enabling it drives the buffer output back into the rail. docs/mcu.md §5.2."
- note added: "gives 18 pF each. Y20's actual CL is NOT verified — Epson FC-135"
- note added: "in ship mode the BATFET is off, so with no USB attached +VSYS and therefore +3V3_AON do not exist. QON idles at 4.3 V from a"
- note added: "land on dies the MCU itself can unpower, and their pull-ups belong on"
- note added: "matches CN4 on ST Nucleo boards (3V3, SWCLK, GND, SWDIO, NRST) so a"
- note added: "page back PC7 / EXTI7"
- note added: "page forward PD8 / EXTI8"
- note added: "power PD6 / EXTI6"
- note added: "reference and nothing else. VREFBUF must stay DISABLED in firmware:"
- note added: "ships in 12.5 / 9 / 7 pF and the LCSC listing does not say which."
- note added: "signals. docs/mcu.md §2.1."
- note added: "som.kicad_sch, MCU_TXD lands on the SoM's UART RX and MCU_RXD on its TX."
- note added: "stock ST-LINK cable fits if a header is soldered on for bring-up."
- note added: "the far sheet, referenced to the far rail. MCU_TXD is push-pull and a"
- note added: "to battery.kicad_sch (I2C also to power_mon)"
- note added: "to epd_power.kicad_sch and power_mon.kicad_sch"
- note added: "to fpga_config, som and frontlight"
- note added: "to power.kicad_sch"

Commit message: R2: port epd, epd_power and power_mon from R1
WP4. These three sheets are copied from pcb/mainboard/ rather than redrawn,
because the acceptance criterion is "is it the same as R1" -- copying keeps
every part, value, coordinate and wire, so the two can be diffed directly.
tools/port_r1.py does it and only ever reads R1.

Result: epd and epd_power are provably identical to R1. R1's netlist was
exported from a scratch copy and the partition of each sheet's pins into nets
compared with R2's, undoing the designator renames first: 49/49 and 44/44 net
groups, identical. power_mon differs in exactly four groups, all intended.

103 of 128 parts keep their exact R1 designator; only collisions are renamed,
+200 for R/C and +20 for U/L so the R1 number stays readable inside the new one.
Other transforms: global labels become hierarchical labels (they are different
nets in KiCad, so a mixed project would have failed to connect silently);
I2C1_* becomes *_AON; three transistor symbols moved library in KiCad 10;
SY8120 and MT9700 are lifted into r2.kicad_sym because they are not in
pcb_common at all -- in R1 they survive only as embedded definitions.

power_mon's two video-decoder channels are gone with the ADV7611, so three
shunts are repurposed without any topology change: U22 now measures the SoM's
input current, the always-on domain, and the frontlight from +VSYS. All three
INA3221s move to +3V3_AON -- on a switched rail their I2C pins would clamp the
always-on bus, and power-down IQ is 0.5 uA typ, so the always-on domain finally
becomes measurable.

Two open items closed by reading R1 properly:

- The EPD chain cannot run from +VSYS. LGS5145 is a buck with a 4.5 V minimum,
  used here as an inverting buck-boost; in steady state it sees ~25 V, but at
  startup the negative rail is at 0 V and 3.0 V from a flat cell will not start
  it. power.md §9 closed.
- Negative rails are measured by dividing between the rail and +3V3_DCDC, not
  to ground. Carried over unchanged, with a f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
Parts:
- added R45: 1k, Resistor_SMD:R_0402_1005Metric, symbol Device:R
Connections:
- net EPD_PWR_EN: now also R45.2; no longer U20.27 (PB0)
- new net EPD_PWR_EN_MCU: R45.1, U20.27 (PB0)
Other:
- note added: "EPD_PWR_EN series"
- note added: "over-current trip must win against the MCU. R45 limits that fight to"
- note added: "power_mon's U21 drives this net open-drain from CRITICAL, so an"
- note added: "~3.3 mA. PB0 can also be read back to see the trip. docs/epd-port.md §4."

Commit message: R2: battery sheet review pass 1, plus notes and parts scratch
Rework battery.kicad_sch and its spec after the first review round, and
carry the follow-on touch-ups into the other R2 sheets. Adds the
Analyse_battery.md review write-up, the patch_battery_review1.py script
that applied it, and a parts/ scratch list.

Co-Authored-By: Claude Opus 5 <noreply@anthropic.com>
Changed lines of the file:
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@@
-	(wire
-		(pts
-			(xy 261.62 237.49) (xy 261.62 252.73)
-		)
-		(stroke
-			(width 0)
-			(type default)
-		)
-	)
 	(wire
 		(pts
@@
 	(wire
 		(pts
-			(xy 261.62 237.49) (xy 261.62 233.68)
-		)
-		(stroke
+			(xy 261.62 233.68) (xy 261.62 252.73)
+		)
+		(stroke

Commit message: R2: mcu sheet review pass 1, plus an R1 comparison
mcu.kicad_sch was reviewed against manual-analysis/Analysis_mcu.md and patched in
place by tools/patch_mcu_review1.py; gen_mcu.py was not re-run.

C42 is deleted. stm32g0b1.pdf Figure 15 (p.65) is the whole of ST's decoupling
scheme and it shows no capacitor on VBAT. With no coin cell fitted, pin 6 (VBAT)
is strapped to the same +3V3_AON net as pin 8 (VDD/VDDA) two pitches away, and
that net already carries C40 4.7 uF + C41 100 nF -- the figure's specified pair.
C42 was a third capacitor on an already-decoupled net.

SW21/SW22, the page buttons, move from TS-1187A-B-A-B to Panasonic EVQPLHA15:
same 1.6 N force and 1.5 mm travel, so the feel is unchanged, but 500 k cycles
instead of 100 k. At a plausible ~200 page turns a day the old part is rated for
about 1.4 years, and these are the most-actuated components on the board. SW20
stays a TS-1187A -- it is the power button, pressed rarely, and JLC Basic.

FB20 stays, but the doc now says plainly that no datasheet asks for it: Figure 15
feeds VREF+ with 100 nF + 1 uF and no series element. It is inherited from R1's
FB3, which was justified because the H750 brings VDDA out as its own pin; the G0
merges VDDA into VDD, so VREF+ is the only node left to filter. What makes it
safe is DCR rather than impedance -- Table 21 caps VREF+ at min(VDD + 0.4, 4.0) V
and BLM15AG121SN1D is 190 mOhm, so 0.19 mV at 1 mA. A resistor there would be a
hazard, and that constraint is now recorded on the part itself.

The 8 MHz the review found is the HSE, not Y20: Table 42 lists fOSC_IN as 4/8/48
MHz min/typ/max and Figure 20 is captioned "Typical application with an 8 MHz
crystal". Y20 is the LSE -- Table 43, on PC14/PC15. No HSE is fitted, which is
what frees PF0/PF1 for MCU_EN_5V/MCU_EN_3V3.

Datasheet 3.5 (p.16) lists the boot loader's interfaces and two are already on
this sheet: USART on PA9/PA10 (= MCU_TXD/MCU_RXD, with the SoM at the far end)
and USB on PA11/PA12 (two of the eleven spa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
Parts:
- removed C42: 100nF/16V, Capacitor_SMD:C_0402_1005Metric, symbol Device:C
- SW21, SW22: footprint Button_Switch_SMD:SW_Push_1P1T_XKB_TS-1187A -> Button_Switch_SMD:SW_SPST_Panasonic_EVQPL_3PL_5PL_PT_A15; LCSC C318884 -> C79172
Other:
- note added: "VDD/VDDA (8) + VBAT (6) - one net"
- note removed: "VDD/VDDA (8) VBAT (6)"
- moved on the sheet: R45
Changed lines of the file:
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@@
 	(text "VREF+ (7)"
 		(exclude_from_sim no)
-		(at 80.01 71.12 0)
+		(at 76.2 74.168 0)
 		(effects
 			(font
@@
 		)
 	)
-	(text "VDD/VDDA (8)        VBAT (6)"
+	(text "VDD/VDDA (8) + VBAT (6) - one net"
 		(exclude_from_sim no)
 		(at 21.59 68.58 0)
@@
 	)
 	(junction
-		(at 50.8 45.72)
-		(diameter 0)
-		(color 0 0 0 0)
-	)
-	(junction
 		(at 48.26 129.54)
 		(diameter 0)
@@
 	(wire
 		(pts
-			(xy 50.8 53.34) (xy 50.8 60.96)
-		)
-		(stroke
-			(width 0)
-			(type default)
-		)
-	)
-	(wire
-		(pts
 			(xy 289.56 62.23) (xy 297.18 62.23)
 		)
@@
 	(wire
 		(pts
-			(xy 299.72 190.5) (xy 316.23 190.5)
+			(xy 318.77 187.96) (xy 335.28 187.96)
 		)
 		(stroke
@@
 	(wire
 		(pts
-			(xy 323.85 190.5) (xy 345.44 190.5)
+			(xy 342.9 187.96) (xy 364.49 187.96)
 		)
 		(stroke
@@
 	)
 	(label "EPD_PWR_EN"
-		(at 345.44 190.5 0)
+		(at 364.49 187.96 0)
 		(effects
 			(font
@@
 	)
 	(label "EPD_PWR_EN_MCU"
-		(at 299.72 190.5 180)
+		(at 318.77 187.96 180)
 		(effects
 			(font
@@
 			)
 		)
-		(property "Footprint" "Button_Switch_SMD:SW_Push_1P1T_XKB_TS-1187A"
+		(property "Footprint" "Button_Switch_SMD:SW_SPST_Panasonic_EVQPL_3PL_5PL_PT_A15"
 			(at 165.1 246.38 0)
 			(hide yes)
@@
 			)
 		)
-		(property "Description" ""
+		(property "Description" "Page-turn tact switch — 1.6 N, 1.5 mm travel, 500 k cycles, 4.9×4.9 mm J-lead (Panasonic EVQPLHA15, LCSC C79172). Chosen for cycle life: the 100 k-cycle TS-1187A is ~1.4 years at 200 turns/day"
 			(at 165.1 246.38 0)
 			(hide yes)
@@
 			)
 		)
-		(property "LCSC" "C318884"
+		(property "LCSC" "C79172"
 			(at 165.1 246.38 0)
 			(hide yes)
@@
 			)
 		)
-		(property "Description" ""
+		(property "Description" "LSE load capacitor for Y20 — 18 pF assumes a 12.5 pF crystal and ~3 pF stray (docs/mcu.md §5.4). Y20's actual CL is unconfirmed; AN2867 is the selection reference named by Table 43"
 			(at 48.26 133.35 0)
 			(hide yes)
@@
 			)
 		)
-		(property "Description" ""
+		(property "Description" "1 µF on VREF+ — stm32g0b1.pdf Figure 15 p.65 (100 nF + 1 µF)"
 			(at 88.9 69.85 0)
 			(hide yes)
@@
 			)
 		)
-		(property "Description" ""
+		(property "Description" "32.768 kHz LSE crystal for the RTC (Epson FC-135, LCSC C32346, JLC Basic). This is the LSE, not the HSE: no HSE is fitted, and the 8 MHz in stm32g0b1.pdf Table 42 / Figure 20 is fOSC_IN typ for the HSE. LSE spec is Table 43 p.85; tSU 2 s. CL unconfirmed — see §9"
 			(at 60.96 129.54 0)
 			(hide yes)
@@
 			)
 		)
-		(property "Description" ""
+		(property "Description" "4.7 µF bulk for VDD/VDDA (pin 8) and VBAT (pin 6), which share +3V3_AON — stm32g0b1.pdf Figure 15 p.65: 1 × 100 nF + 1 × 4.7 µF"
 			(at 25.4 49.53 0)
 			(hide yes)
@@
 	)
 	(symbol
-		(lib_id "Device:C")
-		(at 50.8 49.53 0)
-		(unit 1)
-		(body_style 1)
-		(exclude_from_sim no)
-		(in_bom yes)
-		(on_board yes)
-		(in_pos_files yes)
-		(dnp no)
-		(property "Reference" "C42"
-			(at 53.34 48.26 0)
-			(show_name no)
-			(do_not_autoplace no)
-			(effects
-				(font
-					(size 1.27 1.27)
-				)
-				(justify left)
-			)
-		)
-		(property "Value" "100nF/16V"
-			(at 53.34 51.562 0)
-			(show_name no)
-			(do_not_autoplace no)
-			(effects
-				(font
-					(size 1.27 1.27)
-				)
-				(justify left)
-			)
-		)
-		(property "Footprint" "Capacitor_SMD:C_0402_1005Metric"
-			(at 50.8 49.53 0)
-			(hide yes)
-			(show_name no)
-			(do_not_autoplace no)
-			(effects
-				(font
-					(size 1.27 1.27)
-				)
-			)
-		)
-		(property "Datasheet" ""
-			(at 50.8 49.53 0)
-			(hide yes)
-			(show_name no)
-			(do_not_autoplace no)
-			(effects
-				(font
-					(size 1.27 1.27)
-				)
-			)
-		)
-		(property "Description" ""
-			(at 50.8 49.53 0)
-			(hide yes)
-			(show_name no)
-			(do_not_autoplace no)
-			(effects
-				(font
-					(size 1.27 1.27)
-				)
-			)
-		)
-		(pin "1"
-		)
-		(pin "2"
-		)
-		(instances
-			(project "r2"
-				(path "/dee825bf-c2f1-415d-afdf-cf702072a6e8/a89f58f8-b115-4f71-9806-30f9bff6e587"
-					(reference "C42")
-					(unit 1)
-				)
-			)
-		)
-	)
-	(symbol
 		(lib_id "symbols:+V")
 		(at 205.74 226.06 0)
@@
 			)
 		)
-		(property "Description" ""
+		(property "Description" "Ferrite bead 120 Ω @ 100 MHz, DCR 190 mΩ, 550 mA, 0402 (Murata BLM15AG121SN1D, LCSC C85812). Isolates VREF+ from the digital rail. The low DCR is the load-bearing spec: stm32g0b1.pdf Table 21 caps VREF+ at min(VDD + 0.4, 4.0) V, so nothing with real series impedance may sit here — a resistor would be a hazard, this is <0.2 mV at 1 mA. Not required by Figure 15; see docs/mcu.md §12.2"
 			(at 76.2 49.53 0)
 			(hide yes)
@@
 	(symbol
 		(lib_id "Device:R")
-		(at 320.04 190.5 90)
+		(at 339.09 187.96 90)
 		(unit 1)
 		(body_style 1)
@@
 		(dnp no)
 		(property "Reference" "R45"
-			(at 320.04 185.42 270)
+			(at 339.09 182.88 270)
 			(show_name no)
 			(do_not_autoplace no)
@@
 		)
 		(property "Value" "1k"
-			(at 320.04 196.85 270)
+			(at 339.852 185.166 270)
 			(show_name no)
 			(do_not_autoplace no)
@@
 		)
 		(property "Footprint" "Resistor_SMD:R_0402_1005Metric"
-			(at 320.04 190.5 270)
+			(at 339.09 187.96 270)
 			(hide yes)
 			(show_name no)
@@
 		)
 		(property "Datasheet" ""
-			(at 320.04 190.5 270)
+			(at 339.09 187.96 270)
 			(hide yes)
 			(show_name no)
@@
 		)
 		(property "Description" ""
-			(at 320.04 190.5 270)
+			(at 339.09 187.96 270)
 			(hide yes)
 			(show_name no)
@@
 			)
 		)
-		(property "Description" ""
+		(property "Description" "100 nF decoupling at VDD/VDDA pin 8 — stm32g0b1.pdf Figure 15 p.65. With C40 this is the whole of ST's scheme for this pin pair; no separate VBAT capacitor is called for"
 			(at 38.1 49.53 0)
 			(hide yes)
@@
 			)
 		)
-		(property "Footprint" "Button_Switch_SMD:SW_Push_1P1T_XKB_TS-1187A"
+		(property "Footprint" "Button_Switch_SMD:SW_SPST_Panasonic_EVQPL_3PL_5PL_PT_A15"
 			(at 220.98 246.38 0)
 			(hide yes)
@@
 			)
 		)
-		(property "Description" ""
+		(property "Description" "Page-turn tact switch — 1.6 N, 1.5 mm travel, 500 k cycles, 4.9×4.9 mm J-lead (Panasonic EVQPLHA15, LCSC C79172). Chosen for cycle life: the 100 k-cycle TS-1187A is ~1.4 years at 200 turns/day"
 			(at 220.98 246.38 0)
 			(hide yes)
@@
 			)
 		)
-		(property "LCSC" "C318884"
+		(property "LCSC" "C79172"
 			(at 220.98 246.38 0)
 			(hide yes)
@@
 	)
 	(symbol
-		(lib_id "power:GND")
-		(at 50.8 60.96 0)
-		(unit 1)
-		(body_style 1)
-		(exclude_from_sim no)
-		(in_bom yes)
-		(on_board yes)
-		(in_pos_files yes)
-		(dnp no)
-		(property "Reference" "#PWR305"
-			(at 50.8 60.96 0)
-			(hide yes)
-			(show_name no)
-			(do_not_autoplace no)
-			(effects
-				(font
-					(size 1.27 1.27)
-				)
-			)
-		)
-		(property "Value" "GND"
-			(at 50.8 64.77 0)
-			(show_name no)
-			(do_not_autoplace no)
-			(effects
-				(font
-					(size 1.27 1.27)
-				)
-			)
-		)
-		(property "Footprint" ""
-			(at 50.8 60.96 0)
-			(hide yes)
-			(show_name no)
-			(do_not_autoplace no)
-			(effects
-				(font
-					(size 1.27 1.27)
-				)
-			)
-		)
-		(property "Datasheet" ""
-			(at 50.8 60.96 0)
-			(hide yes)
-			(show_name no)
-			(do_not_autoplace no)
-			(effects
-				(font
-					(size 1.27 1.27)
-				)
-			)
-		)
-		(property "Description" ""
-			(at 50.8 60.96 0)
-			(hide yes)
-			(show_name no)
-			(do_not_autoplace no)
-			(effects
-				(font
-					(size 1.27 1.27)
-				)
-			)
-		)
-		(pin "1"
-		)
-		(instances
-			(project "r2"
-				(path "/dee825bf-c2f1-415d-afdf-cf702072a6e8/a89f58f8-b115-4f71-9806-30f9bff6e587"
-					(reference "#PWR305")
-					(unit 1)
-				)
-			)
-		)
-	)
-	(symbol
 		(lib_id "Device:C")
 		(at 149.86 256.54 0)
@@
 			)
 		)
-		(property "Description" ""
+		(property "Description" "Power button — shorts CHG_QON# to GND galvanically, the only ship-mode exit needing neither a cable nor a live I²C host (bq25890.pdf §9.2.10.2). 1.6 N, 100 k cycles is ample for a rarely-pressed key (XKB TS-1187A-B-A-B, LCSC C318884, JLC Basic)"
 			(at 276.86 246.38 0)
 			(hide yes)
@@
 			)
 		)
-		(property "Description" ""
+		(property "Description" "LSE load capacitor for Y20 — 18 pF assumes a 12.5 pF crystal and ~3 pF stray (docs/mcu.md §5.4). Y20's actual CL is unconfirmed; AN2867 is the selection reference named by Table 43"
 			(at 73.66 133.35 0)
 			(hide yes)
@@
 			)
 		)
-		(property "Description" ""
+		(property "Description" "100 nF on VREF+ — stm32g0b1.pdf Figure 15 p.65 (100 nF + 1 µF)"
 			(at 101.6 69.85 0)
 			(hide yes)
