File: pcb/r2-mainboard/mcu.kicad_sch (KiCad schematic)
At the start: 24 parts, among them J20 SWD (DNP), SW20 SW, SW21 SW, SW22 SW, U20 STM32G0B1RCT6, Y20 32.768kHz

Commit message: R2: WP5 groundwork -- Xilinx/Micron datasheets, LX16 fix, DDR bank to 1.5 V
Steps 1-3 of the WP5 plan. No FPGA sheet is drawn yet; this is the evidence base
and the one power change that had to land before fpga_ddr can be.

DATASHEETS
AMD's documentation portal no longer serves PDFs at any of the old xilinx.com
paths -- every URL returns the same 2.5 KB JavaScript shell -- so these came from
the Wayback Machine: ds162 (DC & Switching), ug380 (Configuration), ug381
(SelectIO), ug393 (PCB Design). The hardware owner supplied mt41k64m16 from
DigiKey after micron.com proved unreachable. UG385 Packaging was deliberately
skipped at 15.8 MB, since pcb_common's XC6SLX-FTG256 symbol already encodes bank
membership in its pin names.

THE FPGA IS AN LX16, NOT AN LX9
NOTES-R2-plan.md's architecture diagram said XC6SLX9 and
NOTES-R2-hardware-facts.md carried a BOM row for XC6SLX9-2FTG256C at $6.10 --
stock and price for the wrong device. The gateware targets xc6slx16-ftg256-3 in
four places (caster.xise Device/Package/Speed Grade, par/ise_flow.sh,
par/ise_run.txt, mig.prj TargetFPGA) and R1's own schematic says
XC6SLX16-FTG256. An LX9 is not a drop-in: the MIG's C3_SMALL_DEVICE parameter
exists specifically for xc6slx9 packages, so it would need the memory controller
regenerated. LCSC stock and price for the LX16 are marked for re-query rather
than guessed.

DDR BANK 1.35 V -> 1.5 V
Caster's UCF constrains all 48 DDR pins as SSTL15_II / DIFF_SSTL15_II /
LVCMOS15, and ds162.pdf Table 7 specifies SSTL15_II only over VCCO
1.425-1.575 V with VREF 0.69-0.81 V. The committed rail was 1.344 V -- 81 mV
below the VCCO minimum, with a half-rail VREF of 0.672 V below its minimum too.
Spartan-6 has no 1.35 V I/O standard to relabel the gateware to: SSTL135 appears
nowhere in ds162.pdf or ug381.pdf, and LVCMOS15 and the HSTL standards still
stop at 1.4 V. R1 runs the same way and works, but on a different layout, and
neither board can be tested from here.

mt41k64m16.pdf p.1 makes the fix fr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
Connections:
- net PG_1V35 renamed PG_1V5
Changed lines of the file:
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@@
 		)
 	)
-	(label "PG_1V35"
+	(label "PG_1V5"
 		(at 114.3 180.34 180)
 		(effects
@@
 		)
 	)
-	(label "PG_1V35"
+	(label "PG_1V5"
 		(at 220.98 82.55 180)
 		(effects
@@
 		)
 	)
-	(hierarchical_label "PG_1V35"
+	(hierarchical_label "PG_1V5"
 		(shape input)
 		(at 228.6 82.55 0)

Commit message: R2: WP5 -- one debug footprint for SWD+JTAG, and INIT_B reaches the MCU
Both changes to mcu.kicad_sch, decided by the hardware owner 2026-08-12.

J20 BECOMES A 2x6 CARRYING BOTH TARGETS
R1 fits J5, a 2x6 1.27 mm socket carrying FPGA JTAG *and* MCU SWD, populated. R2
had only J20, a 1x5 2.54 mm SWD footprint. The combined footprint lands here
rather than on fpga_config because fpga_config already exports FPGA_TCK/TDI/TDO/
TMS as sheet pins from the port -- four labels added to one sheet, instead of
three local nets reclassified on another.

Pinout is R1's J5 order with its pin-10 ground given to MCU_NRST, which R1's
header does not carry:

   1 FPGA_TCK    2 GND        7 FPGA_TMS    8 GND
   3 FPGA_TDI    4 GND        9 MCU_SWCLK  10 MCU_NRST
   5 FPGA_TDO    6 GND       11 MCU_SWDIO  12 +3V3_AON

Signal/ground interleaving is kept on the JTAG half, the half that runs at any
speed. +3V3_AON rather than +3V3 for the adapter's reference: both are 3.3 V, but
the always-on rail is the one guaranteed to be up when you are trying to work out
why nothing else is. Still pads only, not fitted.

The MCU's SWD nets stay local to this sheet, as docs/mcu.md 8 says they should;
it is the four JTAG names that cross, and they were already crossing.

INIT_B REACHES THE MCU ON PC10
PC10 (pin 64) gives up its no-connect flag. A plain GPIO, not one of the four
ADC-capable spares which are worth keeping analog, and EXTI10 is unused so the
signal can interrupt rather than be polled.

It earns the pin because self-boot changes the failure mode: a corrupt NOR image
shows up only as DONE never asserting, which is indistinguishable from "the NOR
never answered". INIT_B low separates the two. R1 never needed this, because its
MCU fed the bitstream and therefore knew what it had sent.

R1'S NOTE WAS LEFT BEHIND AND IS NOW FALSE
The sheet carried R1's note saying J20's "order matches CN4 on ST Nucleo boards
(3V3, SWCLK, GND, SWDIO, NRST) so a stock ST-LINK cable fits". That describes the
1x5 foo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
Parts:
- removed J20: SWD (DNP), Connector_PinHeader_2.54mm:PinHeader_1x05_P2.54mm_Vertical, symbol Connector_Generic:Conn_01x05
- added J20: SWD+JTAG (DNP), Connector_PinSocket_1.27mm:PinSocket_2x06_P1.27mm_Vertical_SMD, symbol Connector_Generic:Conn_02x06_Odd_Even
Connections:
- net +3V3_AON: now also J20.12 (Pin_12)
- net GND: now also J20.2 (Pin_2), J20.4 (Pin_4), J20.6 (Pin_6), J20.8 (Pin_8)
- net MCU_NRST: now also J20.10 (Pin_10)
- net MCU_SWCLK: now also J20.9 (Pin_9)
- net MCU_SWDIO: now also J20.11 (Pin_11)
- net FPGA_INIT: now reaches U20.64 (PC10)
- new net FPGA_TCK: J20.1 (Pin_1)
- new net FPGA_TDI: J20.3 (Pin_3)
- new net FPGA_TDO: J20.5 (Pin_5)
- new net FPGA_TMS: J20.7 (Pin_7)
- no-connect marks 11 -> 10
Other:
- note added: "FPGA JTAG + MCU SWD, R1's J5 order, pin 10 given to MCU_NRST."
- note added: "J20 is pads only, not fitted. One footprint for both targets:"
- note added: "PC10 carries FPGA_INIT: INIT_B low tells a config error from a"
- note added: "silent NOR when DONE never arrives. EXTI10 is free for it."
- note removed: "J20 is pads only, not fitted — the device has to stay thin. Order"
- note removed: "matches CN4 on ST Nucleo boards (3V3, SWCLK, GND, SWDIO, NRST) so a"
- note removed: "stock ST-LINK cable fits if a header is soldered on for bring-up."

Commit message: R2: WP8 -- som drawn; the hierarchy has no dangling interfaces left
tools/gen_som.py draws som.kicad_sch: PCM-071 units 1, 3 and 4 (unit 2, the DPI
link, is on dpi_in), the microSD on MMC1, and the last 12 interface nets.
patch_mcu_pg_som.py claims PC8 for PG_SOM at the MCU end. Root state: 100 names,
100 joined, 0 one-sided -- wire_root.py's DANGLING_OK is now empty, so anything
one-sided from here is a genuinely forgotten interface rather than pending work.

TWO PINS CHOSEN THAT docs/som.md HAD LEFT OPEN. PHYTEC's manual never uses the
word "wake" -- it is not in the document -- so the answer came from TI's AM62x
datasheet (SPRSP58C) instead. Cross-referencing every X1 pin's AM62x ball
against the datasheet's pin-mux table shows exactly 22 X1 pins reach an
MCU_GPIO0_*, i.e. a GPIO in the MCU always-on domain that survives DeepSleep;
the other ~170 signal pins are MAIN-domain and could not wake the module
whatever firmware did. Among those 22, CAN is the one function a reader can
never want:

    SOM_WAKE#  A58  X_MCU_MCAN0_RX  ball B3  = MCU_GPIO0_14
    SOM_IRQ#   A57  X_MCU_MCAN0_TX  ball D6  = MCU_GPIO0_13

Confirm at bring-up, and the doc says so: "Partial IO" is a different low-power
mode from DeepSleep, and PHYTEC demonstrated GPIO wake from Suspend-to-RAM
without naming the pin. The domain is proven; the specific pin is not. Moving
to another of the 22 is a one-net edit, which is why the choice came from that
set. A59/A60 are the next candidates and sit on the same symbol unit.

A SECOND SILENT SHORT, and the netlist caught it after the render did not. The
first fix for a +VBUS power symbol colliding with the USB labels dropped a
vertical wire 10.16 mm to clear them -- and that wire ran through the label
anchors four rows below, shorting SOM_IRQ# and SOM_WAKE# to +VBUS. Both nets
simply vanished from the netlist. ERC reported nothing, because nothing was
illegal. Fixed by giving the symbol room horizontally instead, on a row where
it cannot touch anything.
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
Connections:
- net PG_SOM: now reaches U20.48 (PC8)
- no-connect marks 10 -> 9
Changed lines of the file:
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@@
 	)
 	(no_connect
-		(at 124.46 172.72)
-	)
-	(no_connect
 		(at 124.46 160.02)
 	)
@@
 		)
 	)
+	(wire
+		(pts
+			(xy 124.46 172.72) (xy 114.3 172.72)
+		)
+		(stroke
+			(width 0)
+			(type default)
+		)
+	)
+	(hierarchical_label "PG_SOM"
+		(shape input)
+		(at 114.3 172.72 180)
+		(effects
+			(font
+				(size 1.27 1.27)
+			)
+			(justify left)
+		)
+	)

Commit message: R2: WP6b -- io_expansion drawn; Stage C capture is complete
Two FPC connectors, two gated rails, seven MCU pins, everything DNP.
NOTES-R2-plan.md constraint 3 wants touch and pen "addable without a respin";
this sheet is that provision, and it is honest about which half of the promise
is certain:

  certain  -- the seven MCU pins exist and are routed, and +3V3_TOUCH /
              +3V3_PEN exist. Those are what would otherwise force a
              whole-board respin.
  a guess  -- the FPC pad order, because neither the touch controller nor the
              digitizer is chosen and the panel is not either.

docs/io-expansion.md 5 puts that in front of the owner as the last open
decision in Stage C, with three ways to close it, rather than burying it.

PC4/PC5 are USART3_TX/RX at AF0 -- verified in stm32g0b1.pdf's
alternate-function table, both free, and the one allocation here that is not
interchangeable. The other five are ordinary GPIO. Touch adds no I2C pins: it
joins the existing always-on bus, and SCL_AON/SDA_AON now carry J22.3/J22.4
alongside the charger, gauge and three INA3221s. Two spares remain, and which
two was deliberate -- PA12 (USB-DP capable) and PB12 (ADC-capable) are the two
with a capability the rest lack.

Everything DNP is coherent, not lazy: with no connector fitted there is no
load, so a fitted load switch would be two parts powering nothing. It also
means these two TPS22914s consume none of the thin LCSC stock epd-port.md 7
flags, so that stays a two-part problem.

A FOURTH SILENT SHORT, and this time the tooling caught it before the netlist
did. The connectors' GND pins dropped from their own label column and ran
straight through the two anchors below -- putting SCL_AON, SDA_AON, PEN_TXD
and PEN_RXD on GND. The entire always-on I2C bus was shorted to ground and ERC
said nothing.

So schgen.Sheet.check_label_crossings() now runs inside render() for every
generator: no wire may pass *through* a label anchor it does not end at. Ending
at an a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
Connections:
- net TOUCH_INT#: now reaches U20.16 (PC3)
- net PEN_TXD: now reaches U20.25 (PC4)
- net PEN_RXD: now reaches U20.26 (PC5)
- net PEN_INT#: now reaches U20.38 (PC6)
- net TOUCH_RST#: now reaches U20.41 (PD9)
- net MCU_EN_TOUCH: now reaches U20.43 (PA9/PA11)
- net MCU_EN_PEN: now reaches U20.49 (PC9)
- no-connect marks 9 -> 2
Changed lines of the file:
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@@
 	)
 	(no_connect
-		(at 180.34 134.62)
-	)
-	(no_connect
 		(at 180.34 185.42)
 	)
 	(no_connect
-		(at 124.46 175.26)
-	)
-	(no_connect
-		(at 124.46 167.64)
-	)
-	(no_connect
-		(at 124.46 165.1)
-	)
-	(no_connect
 		(at 180.34 139.7)
 	)
-	(no_connect
-		(at 124.46 162.56)
-	)
-	(no_connect
-		(at 124.46 160.02)
-	)
-	(no_connect
-		(at 124.46 147.32)
-	)
 	(wire
 		(pts
@@
 		(effects
 			(font
+				(size 1.27 1.27)
+			)
+			(justify right)
+		)
+	)
+	(wire
+		(pts
+			(xy 124.46 160.02) (xy 114.3 160.02)
+		)
+		(stroke
+			(width 0)
+			(type default)
+		)
+	)
+	(hierarchical_label "TOUCH_INT#"
+		(shape input)
+		(at 114.3 160.02 180)
+		(effects
+			(font
+				(size 1.27 1.27)
+			)
+			(justify right)
+		)
+	)
+	(wire
+		(pts
+			(xy 124.46 162.56) (xy 114.3 162.56)
+		)
+		(stroke
+			(width 0)
+			(type default)
+		)
+	)
+	(hierarchical_label "PEN_TXD"
+		(shape output)
+		(at 114.3 162.56 180)
+		(effects
+			(font
+				(size 1.27 1.27)
+			)
+			(justify right)
+		)
+	)
+	(wire
+		(pts
+			(xy 124.46 165.1) (xy 114.3 165.1)
+		)
+		(stroke
+			(width 0)
+			(type default)
+		)
+	)
+	(hierarchical_label "PEN_RXD"
+		(shape input)
+		(at 114.3 165.1 180)
+		(effects
+			(font
+				(size 1.27 1.27)
+			)
+			(justify right)
+		)
+	)
+	(wire
+		(pts
+			(xy 124.46 167.64) (xy 114.3 167.64)
+		)
+		(stroke
+			(width 0)
+			(type default)
+		)
+	)
+	(hierarchical_label "PEN_INT#"
+		(shape input)
+		(at 114.3 167.64 180)
+		(effects
+			(font
+				(size 1.27 1.27)
+			)
+			(justify right)
+		)
+	)
+	(wire
+		(pts
+			(xy 124.46 147.32) (xy 114.3 147.32)
+		)
+		(stroke
+			(width 0)
+			(type default)
+		)
+	)
+	(hierarchical_label "TOUCH_RST#"
+		(shape output)
+		(at 114.3 147.32 180)
+		(effects
+			(font
+				(size 1.27 1.27)
+			)
+			(justify right)
+		)
+	)
+	(wire
+		(pts
+			(xy 124.46 175.26) (xy 114.3 175.26)
+		)
+		(stroke
+			(width 0)
+			(type default)
+		)
+	)
+	(hierarchical_label "MCU_EN_PEN"
+		(shape output)
+		(at 114.3 175.26 180)
+		(effects
+			(font
+				(size 1.27 1.27)
+			)
+			(justify right)
+		)
+	)
+	(wire
+		(pts
+			(xy 180.34 134.62) (xy 190.5 134.62)
+		)
+		(stroke
+			(width 0)
+			(type default)
+		)
+	)
+	(hierarchical_label "MCU_EN_TOUCH"
+		(shape output)
+		(at 190.5 134.62 0)
+		(effects
+			(font
