File: pcb/r2-mainboard/mcu.kicad_sch (KiCad schematic)
At the start: 28 parts, among them J400 SWD+JTAG (DNP), Q400 AO3400A, SW400 EVQPUC02K, SW401 SW, SW402 SW, U400 STM32G0B1RCT6, Y400 32.768kHz

Commit message: routing
Changed lines of the file:
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@@
 	)
 	(junction
-		(at 101.6 195.58)
-		(diameter 0)
-		(color 0 0 0 0)
-	)
-	(junction
-		(at 101.6 200.66)
-		(diameter 0)
-		(color 0 0 0 0)
-	)
-	(junction
 		(at 48.26 129.54)
 		(diameter 0)
@@
 	)
 	(junction
+		(at 101.6 195.58)
+		(diameter 0)
+		(color 0 0 0 0)
+	)
+	(junction
 		(at 261.62 241.3)
 		(diameter 0)
@@
 	)
 	(junction
+		(at 101.6 193.04)
+		(diameter 0)
+		(color 0 0 0 0)
+	)
+	(junction
 		(at 205.74 246.38)
 		(diameter 0)
@@
 	(wire
 		(pts
-			(xy 83.82 205.74) (xy 71.12 205.74)
+			(xy 73.66 207.01) (xy 71.12 207.01)
 		)
 		(stroke
@@
 	(wire
 		(pts
+			(xy 73.66 205.74) (xy 83.82 205.74)
+		)
+		(stroke
+			(width 0)
+			(type default)
+		)
+	)
+	(wire
+		(pts
 			(xy 57.15 129.54) (xy 48.26 129.54)
 		)
@@
 	(wire
 		(pts
+			(xy 101.6 210.82) (xy 101.6 205.74)
+		)
+		(stroke
+			(width 0)
+			(type default)
+		)
+	)
+	(wire
+		(pts
 			(xy 124.46 129.54) (xy 114.3 129.54)
 		)
@@
 	(wire
 		(pts
-			(xy 101.6 193.04) (xy 101.6 210.82)
+			(xy 110.49 193.04) (xy 110.49 195.58)
 		)
 		(stroke
@@
 	(wire
 		(pts
+			(xy 101.6 205.74) (xy 96.52 205.74)
+		)
+		(stroke
+			(width 0)
+			(type default)
+		)
+	)
+	(wire
+		(pts
 			(xy 289.56 62.23) (xy 297.18 62.23)
 		)
@@
 	(wire
 		(pts
+			(xy 101.6 195.58) (xy 101.6 198.12)
+		)
+		(stroke
+			(width 0)
+			(type default)
+		)
+	)
+	(wire
+		(pts
 			(xy 220.98 62.23) (xy 228.6 62.23)
 		)
@@
 	(wire
 		(pts
-			(xy 83.82 203.2) (xy 71.12 203.2)
+			(xy 72.39 204.47) (xy 71.12 204.47)
 		)
 		(stroke
@@
 	(wire
 		(pts
-			(xy 96.52 205.74) (xy 106.68 205.74)
+			(xy 101.6 210.82) (xy 106.68 210.82)
 		)
 		(stroke
@@
 	(wire
 		(pts
+			(xy 72.39 204.47) (xy 72.39 203.2)
+		)
+		(stroke
+			(width 0)
+			(type default)
+		)
+	)
+	(wire
+		(pts
 			(xy 96.52 203.2) (xy 119.38 203.2)
 		)
@@
 	(wire
 		(pts
+			(xy 101.6 193.04) (xy 110.49 193.04)
+		)
+		(stroke
+			(width 0)
+			(type default)
+		)
+	)
+	(wire
+		(pts
 			(xy 180.34 162.56) (xy 190.5 162.56)
 		)
@@
 	(wire
 		(pts
+			(xy 73.66 207.01) (xy 73.66 205.74)
+		)
+		(stroke
+			(width 0)
+			(type default)
+		)
+	)
+	(wire
+		(pts
 			(xy 180.34 160.02) (xy 190.5 160.02)
 		)
@@
 	(wire
 		(pts
+			(xy 101.6 193.04) (xy 101.6 195.58)
+		)
+		(stroke
+			(width 0)
+			(type default)
+		)
+	)
+	(wire
+		(pts
+			(xy 101.6 198.12) (xy 101.6 200.66)
+		)
+		(stroke
+			(width 0)
+			(type default)
+		)
+	)
+	(wire
+		(pts
 			(xy 124.46 127) (xy 114.3 127)
 		)
@@
 	(wire
 		(pts
+			(xy 72.39 203.2) (xy 83.82 203.2)
+		)
+		(stroke
+			(width 0)
+			(type default)
+		)
+	)
+	(wire
+		(pts
 			(xy 220.98 146.05) (xy 228.6 146.05)
 		)
@@
 	)
 	(label "MCU_SWCLK"
-		(at 71.12 203.2 180)
+		(at 71.12 204.47 180)
 		(effects
 			(font
@@
 	)
 	(label "MCU_SWDIO"
-		(at 71.12 205.74 180)
+		(at 71.12 207.01 180)
 		(effects
 			(font
@@
 	(symbol
 		(lib_id "power:GND")
-		(at 101.6 210.82 0)
+		(at 110.49 195.58 0)
 		(unit 1)
 		(body_style 1)
@@
 		(dnp no)
 		(property "Reference" "#PWR351"
-			(at 101.6 210.82 0)
+			(at 110.49 195.58 0)
 			(hide yes)
 			(show_name no)
@@
 		)
 		(property "Value" "GND"
-			(at 101.6 214.63 0)
+			(at 110.49 199.39 0)
 			(show_name no)
 			(do_not_autoplace no)
@@
 		)
 		(property "Footprint" ""
-			(at 101.6 210.82 0)
+			(at 110.49 195.58 0)
 			(hide yes)
 			(show_name no)
@@
 		)
 		(property "Datasheet" ""
-			(at 101.6 210.82 0)
+			(at 110.49 195.58 0)
 			(hide yes)
 			(show_name no)
@@
 		)
 		(property "Description" ""
-			(at 101.6 210.82 0)
+			(at 110.49 195.58 0)
 			(hide yes)
 			(show_name no)
@@
 	(symbol
 		(lib_id "symbols:+V")
-		(at 106.68 205.74 0)
+		(at 106.68 210.82 0)
 		(unit 1)
 		(body_style 1)
@@
 		(dnp no)
 		(property "Reference" "#PWR352"
-			(at 106.68 205.74 0)
+			(at 106.68 210.82 0)
 			(hide yes)
 			(show_name no)
@@
 		)
 		(property "Value" "+3V3_AON"
-			(at 106.68 209.55 0)
+			(at 107.95 206.756 0)
 			(show_name no)
 			(do_not_autoplace no)
@@
 		)
 		(property "Footprint" ""
-			(at 106.68 205.74 0)
+			(at 106.68 210.82 0)
 			(hide yes)
 			(show_name no)
@@
 		)
 		(property "Datasheet" ""
-			(at 106.68 205.74 0)
+			(at 106.68 210.82 0)
 			(hide yes)
 			(show_name no)
@@
 		)
 		(property "Description" ""
-			(at 106.68 205.74 0)
+			(at 106.68 210.82 0)
 			(hide yes)
 			(show_name no)
@@
 		(dnp yes)
 		(property "Reference" "J400"
-			(at 88.9 193.04 0)
+			(at 89.916 188.468 0)
 			(show_name no)
 			(do_not_autoplace no)

Commit message: Schematics update for new chip.
Parts:
- C401, C403, C404, C407, C408, C409: value 100nF/16V -> 100nF/50V
- C402: value 1uF/16V -> 1uF/25V
- R400: value 10k -> 10k/1%
- R401, R404, R405, R407: value 1k -> 1k/1%
- R402, R403, R406: value 100k -> 100k/1%
- R408: value 1M -> 1M/1%
Changed lines of the file:
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@@
 			)
 		)
-		(property "Value" "1uF/16V"
+		(property "Value" "1uF/25V"
 			(at 91.44 71.882 0)
 			(show_name no)
@@
 			)
 		)
-		(property "Value" "100k"
+		(property "Value" "100k/1%"
 			(at 332.74 243.84 0)
 			(show_name no)
@@
 			)
 		)
-		(property "Value" "1k"
+		(property "Value" "1k/1%"
 			(at 339.852 185.166 270)
 			(show_name no)
@@
 			)
 		)
-		(property "Value" "100nF/16V"
+		(property "Value" "100nF/50V"
 			(at 259.08 258.572 0)
 			(show_name no)
@@
 			)
 		)
-		(property "Value" "100nF/16V"
+		(property "Value" "100nF/50V"
 			(at 40.64 51.562 0)
 			(show_name no)
@@
 			)
 		)
-		(property "Value" "1k"
+		(property "Value" "1k/1%"
 			(at 335.28 224.79 270)
 			(show_name no)
@@
 			)
 		)
-		(property "Value" "100nF/16V"
+		(property "Value" "100nF/50V"
 			(at 203.2 258.572 0)
 			(show_name no)
@@
 			)
 		)
-		(property "Value" "100nF/16V"
+		(property "Value" "100nF/50V"
 			(at 35.56 196.342 0)
 			(show_name no)
@@
 			)
 		)
-		(property "Value" "100k"
+		(property "Value" "100k/1%"
 			(at 203.2 235.712 0)
 			(show_name no)
@@
 			)
 		)
-		(property "Value" "100nF/16V"
+		(property "Value" "100nF/50V"
 			(at 147.32 258.572 0)
 			(show_name no)
@@
 			)
 		)
-		(property "Value" "1k"
+		(property "Value" "1k/1%"
 			(at 259.08 231.902 0)
 			(show_name no)
@@
 			)
 		)
-		(property "Value" "1M"
+		(property "Value" "1M/1%"
 			(at 383.54 238.76 0)
 			(show_name no)
@@
 			)
 		)
-		(property "Value" "1k"
+		(property "Value" "1k/1%"
 			(at 44.45 278.13 270)
 			(show_name no)
@@
 			)
 		)
-		(property "Value" "100nF/16V"
+		(property "Value" "100nF/50V"
 			(at 104.14 71.882 0)
 			(show_name no)
@@
 			)
 		)
-		(property "Value" "100k"
+		(property "Value" "100k/1%"
 			(at 147.32 235.712 0)
 			(show_name no)
@@
 			)
 		)
-		(property "Value" "10k"
+		(property "Value" "10k/1%"
 			(at 101.6 239.522 0)
 			(show_name no)
