File: pcb/r2-mainboard/som.kicad_sch (KiCad schematic)
At the start: 0 parts

Commit message: R2: WP8 -- som drawn; the hierarchy has no dangling interfaces left
tools/gen_som.py draws som.kicad_sch: PCM-071 units 1, 3 and 4 (unit 2, the DPI
link, is on dpi_in), the microSD on MMC1, and the last 12 interface nets.
patch_mcu_pg_som.py claims PC8 for PG_SOM at the MCU end. Root state: 100 names,
100 joined, 0 one-sided -- wire_root.py's DANGLING_OK is now empty, so anything
one-sided from here is a genuinely forgotten interface rather than pending work.

TWO PINS CHOSEN THAT docs/som.md HAD LEFT OPEN. PHYTEC's manual never uses the
word "wake" -- it is not in the document -- so the answer came from TI's AM62x
datasheet (SPRSP58C) instead. Cross-referencing every X1 pin's AM62x ball
against the datasheet's pin-mux table shows exactly 22 X1 pins reach an
MCU_GPIO0_*, i.e. a GPIO in the MCU always-on domain that survives DeepSleep;
the other ~170 signal pins are MAIN-domain and could not wake the module
whatever firmware did. Among those 22, CAN is the one function a reader can
never want:

    SOM_WAKE#  A58  X_MCU_MCAN0_RX  ball B3  = MCU_GPIO0_14
    SOM_IRQ#   A57  X_MCU_MCAN0_TX  ball D6  = MCU_GPIO0_13

Confirm at bring-up, and the doc says so: "Partial IO" is a different low-power
mode from DeepSleep, and PHYTEC demonstrated GPIO wake from Suspend-to-RAM
without naming the pin. The domain is proven; the specific pin is not. Moving
to another of the 22 is a one-net edit, which is why the choice came from that
set. A59/A60 are the next candidates and sit on the same symbol unit.

A SECOND SILENT SHORT, and the netlist caught it after the render did not. The
first fix for a +VBUS power symbol colliding with the USB labels dropped a
vertical wire 10.16 mm to clear them -- and that wire ran through the label
anchors four rows below, shorting SOM_IRQ# and SOM_WAKE# to +VBUS. Both nets
simply vanished from the netlist. ERC reported nothing, because nothing was
illegal. Fixed by giving the symbol room horizontally instead, on a row where
it cannot touch anything.
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
Parts:
- added C510, C511: 22u, Capacitor_SMD:C_0805_2012Metric, symbol Device:C
- added C512: 100n, Capacitor_SMD:C_0402_1005Metric, symbol Device:C
- added C513: 10u, Capacitor_SMD:C_0805_2012Metric, symbol Device:C
- added J21: MICRO_SD(TFC-WPAPR-08), footprints:TFC-WPAPR-08, symbol symbols:MICRO_SD(TFC-WPAPR-08)
- added R500, R501, R502, R503, R504: 47k, Resistor_SMD:R_0402_1005Metric, symbol Device:R
- added X2: PCM-071, footprints:PCM-071_2xBTH-060-01-L-D-A-K, symbol r2:PCM-071
Connections:
- new net +3V3_AON: X2.B2 (VBAT)
- new net +3V3_SDIO: C513.1, J21.4 (VDD), R500.1, R501.1, R502.1, R503.1, R504.1, X2.B1 (SoC_VDDSHV5_SDIO)
- new net +5V_SOM: C510.1, C511.1, C512.1, X2.A1 (VIN), X2.A2 (VIN), X2.A3 (VIN)
- new net +VBUS: X2.A40 (X_USB0_VBUS)
- new net FPGA_CS: X2.C40 (X_SPI0_CS0)
- new net FPGA_MISO: X2.D42 (X_SPI0_D1)
- new net FPGA_MOSI: X2.D41 (X_SPI0_D0)
- new net FPGA_SCLK: X2.D40 (X_SPI0_CLK)
- new net GND: C510.2, C511.2, C512.2, C513.2, J21.10, J21.11, J21.12, J21.13, J21.6 (VSS), X2.A14 (GND), X2.A19 (GND), X2.A24 (GND), X2.A29 (GND), X2.A32 (GND), X2.A37 (GND), X2.A4 (GND), X2.A42 (GND), X2.A45 (GND), X2.A50 (GND), X2.A55 (GND), X2.A9 (GND), X2.B13 (GND), X2.B18 (GND), X2.B23 (GND), X2.B28 (GND), X2.B3 (GND), X2.B33 (GND), X2.B38 (GND), X2.B43 (GND), X2.B48 (GND), X2.B53 (GND), X2.B56 (GND), X2.B60 (GND), X2.B8 (GND), X2.C12 (GND), X2.C19 (GND), X2.C24 (GND), X2.C31 (GND), X2.C38 (GND), X2.C43 (GND), X2.C48 (GND), X2.C53 (GND), X2.C59 (GND), X2.C6 (GND), X2.D17 (GND), X2.D22 (GND), X2.D27 (GND), X2.D3 (GND), X2.D34 (GND), X2.D39 (GND), X2.D45 (GND), X2.D52 (GND), X2.D57 (GND), X2.D9 (GND)
- new net MCU_RXD: X2.D38 (X_UART0_TXD)
- new net MCU_TXD: X2.D37 (X_UART0_RXD)
- new net NOR_CS: X2.C41 (X_SPI0_CS1)
- new net PG_SOM: X2.C54 (X_PGOOD)
- new net SD_CD#: J21.9, X2.C23 (X_MMC1_SDCD)
- new net SD_CLK: J21.5 (CLK/SCLK), X2.D26 (X_MMC1_CLK)
- new net SD_CMD: J21.3 (CMD/DI), R500.2, X2.D25 (X_MMC1_CMD)
- new net SD_DAT0: J21.7 (DAT0/DO), R501.2, X2.C25 (X_MMC1_DAT0)
- new net SD_DAT1: J21.8 (DAT1/RES), R502.2, X2.C26 (X_MMC1_DAT1)
- new net SD_DAT2: J21.1 (DAT2/RES), R503.2, X2.D28 (X_MMC1_DAT2)
- new net SD_DAT3: J21.2 (CD/DAT3/CS), R504.2, X2.D29 (X_MMC1_DAT3)
- new net SOM_IRQ#: X2.A57 (X_MCU_MCAN0_TX)
- new net SOM_RESET#: X2.C52 (X_nRESET_IN)
- new net SOM_WAKE#: X2.A58 (X_MCU_MCAN0_RX)
- new net USB_DM: X2.A38 (X_USB0_DM)
- new net USB_DP: X2.A39 (X_USB0_DP)
- no-connect marks 0 -> 147
Other:
- note added: "*** B2 VBAT is the RTC backup, 40 nA. It is NOT this board's +VBAT,"
- note added: "*** PHYTEC showed GPIO wake from Suspend-to-RAM but never named the pin."
- note added: "*** which is the raw Li-ion cell on battery.kicad_sch."
- note added: "1 SOM_RESET# low 2 MCU_EN_5V 3 wait PG_SOM"
- note added: "4 MCU_EN_3V3 + PG_3V3 5 release SOM_RESET#"
- note added: "All three VIN pins and all 45 grounds are connected -- 4.6 requires it."
- note added: "B1 SoC_VDDSHV5_SDIO is an OUTPUT (Table 12), 100 mA: it powers the card."
- note added: "BOOTMODE_8/9 then latch with +3V3 already up."
- note added: "C51 PMIC_EN open: 100K pullup to 5 V on the module, MCU_EN_5V is the"
- note added: "L-1038e.A5 5.4 makes it *mandatory* that nothing drives the SOM's I/O"
- note added: "MCU always-on domain, which survives DeepSleep. *** Confirm at bring-up:"
- note added: "Pin numbers from datasheets/som_pinout.json, which parse_som_pinout.py"
- note added: "SEQUENCING -- power.md 5.1. Getting this wrong risks the module."
- note added: "SOM_WAKE# = A58 (MCU_GPIO0_14), SOM_IRQ# = A57 (MCU_GPIO0_13). Both are"
- note added: "before it is powered, and +3V3 is VCCO for the FPGA bank facing it:"
- note added: "extracts from L-1038e.A5 Tables 7-10. Reasoning: docs/som.md."
- note added: "on/off. C22 MMC1_SDWP open: microSD has no write-protect switch."
- note added: "som -- PCM-071 units 1/3/4. Unit 2, the DPI link, is on dpi_in."
