File: pcb/r2-mainboard/som.kicad_sch (KiCad schematic)
At the start: 14 parts, among them J21 MICRO_SD(TFC-WPAPR-08), J26 BTH-060-01-L-D-A-K-TR, J27 BTH-060-01-L-D-A-K-TR, X2 PCM-071

Commit message: change layout and reduce board size + add second usb host only
Connections:
- net USB1_DM: now reaches J26.B39 (X_USB1_DM)
- net USB1_DP: now reaches J26.B40 (X_USB1_DP)
- net USB1_VBUS: now reaches J26.B41 (X_USB1_VBUS)
- net USB1_DRVVBUS: now reaches J26.B42 (X_USB1_DRVVBUS)
- no-connect marks 145 -> 141
Changed lines of the file:
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@@
-	)
-	(no_connect
-		(at 386.08 72.39)
 	)
 	(no_connect
@@
 	)
 	(no_connect
-		(at 386.08 69.85)
-	)
-	(no_connect
 		(at 314.96 184.15)
 	)
@@
 	)
 	(no_connect
-		(at 386.08 67.31)
-	)
-	(no_connect
 		(at 314.96 153.67)
 	)
@@
 	)
 	(no_connect
-		(at 386.08 64.77)
-	)
-	(no_connect
 		(at 314.96 57.15)
 	)
@@
 	(wire
 		(pts
+			(xy 386.08 67.31) (xy 391.16 67.31)
+		)
+		(stroke
+			(width 0)
+			(type default)
+		)
+	)
+	(wire
+		(pts
 			(xy 104.14 39.37) (xy 114.3 39.37)
 		)
@@
 	(wire
 		(pts
+			(xy 386.08 64.77) (xy 391.16 64.77)
+		)
+		(stroke
+			(width 0)
+			(type default)
+		)
+	)
+	(wire
+		(pts
 			(xy 266.7 214.63) (xy 266.7 218.44)
 		)
@@
 	(wire
 		(pts
+			(xy 386.08 69.85) (xy 391.16 69.85)
+		)
+		(stroke
+			(width 0)
+			(type default)
+		)
+	)
+	(wire
+		(pts
 			(xy 35.56 49.53) (xy 35.56 59.69)
 		)
@@
 		(pts
 			(xy 177.8 100.33) (xy 154.94 100.33)
+		)
+		(stroke
+			(width 0)
+			(type default)
+		)
+	)
+	(wire
+		(pts
+			(xy 386.08 72.39) (xy 391.16 72.39)
 		)
 		(stroke
@@
 			)
 			(justify right bottom)
+		)
+	)
+	(hierarchical_label "USB1_VBUS"
+		(shape input)
+		(at 391.16 69.85 0)
+		(effects
+			(font
+				(size 1.27 1.27)
+			)
+			(justify left)
 		)
 	)
@@
 		)
 	)
+	(hierarchical_label "USB1_DM"
+		(shape bidirectional)
+		(at 391.16 64.77 0)
+		(effects
+			(font
+				(size 1.27 1.27)
+			)
+			(justify left)
+		)
+	)
 	(hierarchical_label "FPGA_MOSI"
 		(shape bidirectional)
@@
 		)
 	)
+	(hierarchical_label "USB1_DRVVBUS"
+		(shape output)
+		(at 391.16 72.39 0)
+		(effects
+			(font
+				(size 1.27 1.27)
+			)
+			(justify left)
+		)
+	)
 	(hierarchical_label "MCU_RXD"
 		(shape bidirectional)
@@
 		)
 	)
+	(hierarchical_label "USB1_DP"
+		(shape bidirectional)
+		(at 391.16 67.31 0)
+		(effects
+			(font
+				(size 1.27 1.27)
+			)
+			(justify left)
+		)
+	)
