File: pcb/r2-mainboard/epd_power.kicad_sch (KiCad schematic)
At the start: 0 parts

Commit message: R2: port epd, epd_power and power_mon from R1
WP4. These three sheets are copied from pcb/mainboard/ rather than redrawn,
because the acceptance criterion is "is it the same as R1" -- copying keeps
every part, value, coordinate and wire, so the two can be diffed directly.
tools/port_r1.py does it and only ever reads R1.

Result: epd and epd_power are provably identical to R1. R1's netlist was
exported from a scratch copy and the partition of each sheet's pins into nets
compared with R2's, undoing the designator renames first: 49/49 and 44/44 net
groups, identical. power_mon differs in exactly four groups, all intended.

103 of 128 parts keep their exact R1 designator; only collisions are renamed,
+200 for R/C and +20 for U/L so the R1 number stays readable inside the new one.
Other transforms: global labels become hierarchical labels (they are different
nets in KiCad, so a mixed project would have failed to connect silently);
I2C1_* becomes *_AON; three transistor symbols moved library in KiCad 10;
SY8120 and MT9700 are lifted into r2.kicad_sym because they are not in
pcb_common at all -- in R1 they survive only as embedded definitions.

power_mon's two video-decoder channels are gone with the ADV7611, so three
shunts are repurposed without any topology change: U22 now measures the SoM's
input current, the always-on domain, and the frontlight from +VSYS. All three
INA3221s move to +3V3_AON -- on a switched rail their I2C pins would clamp the
always-on bus, and power-down IQ is 0.5 uA typ, so the always-on domain finally
becomes measurable.

Two open items closed by reading R1 properly:

- The EPD chain cannot run from +VSYS. LGS5145 is a buck with a 4.5 V minimum,
  used here as an inverting buck-boost; in steady state it sees ~25 V, but at
  startup the negative rail is at 0 V and 3.0 V from a flat cell will not start
  it. power.md §9 closed.
- Negative rails are measured by dividing between the rail and +3V3_DCDC, not
  to ground. Carried over unchanged, with a f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
Parts:
- added C104, C17, C232, C242, C245, C249, C37, C51, C53: 22uF/10V, Capacitor_SMD:C_0805_2012Metric, symbol Device:C
- added C160, C171, C174, C35, C54: 100nF/50V, Capacitor_SMD:C_0402_1005Metric, symbol Device:C
- added C165, C175, C241, C38: 18pF/50V, Capacitor_SMD:C_0402_1005Metric, symbol Device:C
- added C166, C167, C173, C176, C177, C233, C244, C246: 4.7uF/50V, Capacitor_SMD:C_0805_2012Metric, symbol Device:C
- added C172, C178, C52: 470nF/25V, Capacitor_SMD:C_0402_1005Metric, symbol Device:C
- added C56: 4.7uF/6.3V, Capacitor_SMD:C_0402_1005Metric, symbol Device:C
- added D1, D15, D17, D2, D3, D4, D6: 1N5819WS, footprints:D_SOD-323_Alt, symbol Diode:1N5819WS
- added D5: 1N5819WS, footprints:D_SOD-323_Alt, symbol Device:D
- added L30, L32, L5, L6: WPN3012H4R7MT, Inductor_SMD:L_Changjiang_FNR3012S, symbol Device:L
- added Q1, Q7, Q8: AO3401A, Package_TO_SOT_SMD:SOT-23, symbol Transistor_FET:Q_PMOS_GSD
- added Q2: S8050, Package_TO_SOT_SMD:SOT-23, symbol Transistor_BJT:Q_NPN_BEC
- added Q6: AO3400A, Package_TO_SOT_SMD:SOT-23, symbol Transistor_FET:Q_NMOS_GSD
- added R213, R226, R228, R234, R62, R92, R93, R94: 100K/1%, Resistor_SMD:R_0402_1005Metric, symbol Device:R
- added R217, R219, R65: 10K/1%, Resistor_SMD:R_0402_1005Metric, symbol Device:R
- added R218: 240K/1%, Resistor_SMD:R_0402_1005Metric, symbol Device:R
- added R224, R88: 390K/1%, Resistor_SMD:R_0402_1005Metric, symbol Device:R
- added R225, R227, R64, R89: 22K/1%, Resistor_SMD:R_0402_1005Metric, symbol Device:R
- added R229, R230: 5.1K/1%, Resistor_SMD:R_0402_1005Metric, symbol Device:R
- added R63, R66: 33R/1%, Resistor_SMD:R_0402_1005Metric, symbol Device:R
- added R78: 150K/1%, Resistor_SMD:R_0402_1005Metric, symbol Device:R
- added R79: 13K/1%, Resistor_SMD:R_0402_1005Metric, symbol Device:R
- added U23, U24: LGS6302B5, Package_TO_SOT_SMD:SOT-23-5, symbol Regulator_Switching:LGS6302B5
- added U26, U9: LGS5145, Package_TO_SOT_SMD:TSOT-23-6, symbol r2:SY8120
- added U31: LM321, Package_TO_SOT_SMD:SOT-23-5, symbol Amplifier_Operational:LM321
- added U6: MT9700, Package_TO_SOT_SMD:SOT-23-5, symbol r2:MT9700
- added U7, U8: TPS22914BYFPR, Package_BGA:WLP-4_0.83x0.83mm_P0.4mm, symbol Power_Management:AP22913CN4
Connections:
- new net: C241.1, R213.1, R224.1, R225.2, U24.3 (FB)
- new net: C35.2, U9.1 (BS)
- new net: C38.1, R218.1, R219.2, U9.3 (FB)
- new net: C35.1, D3.1 (K), L6.1, U9.6 (SW)
- new net: D4.1 (K), R93.2
- new net: C52.2, R226.2, R227.1, U31.1 (+)
- new net: Q6.2 (S), U31.3 (-), U31.4
- new net: Q2.1 (B), R229.2, R230.2
- new net: Q1.1 (G), Q2.3 (C), R228.1
- new net: D1.2 (A), D4.2 (A), Q1.3 (D)
- new net: C174.1, D17.1 (K), L32.1, U26.6 (SW)
- new net: D2.2 (A), L5.2, U24.1 (SW)
- new net: C174.2, U26.1 (BS)
- new net: C175.1, R88.1, R89.2, U26.3 (FB)
- new net: R217.2, U6.3 (SET)
- new net: Q7.1 (G), R63.2
- new net: D15.2 (A), L30.2, U23.1 (SW)
- new net: Q6.1 (G), Q7.3 (D), R62.1
- new net: D1.1 (K), R92.2
- new net: Q8.3 (D), R64.1
- new net: Q8.1 (G), R66.1
- new net: C165.1, R78.1, R79.2, U23.3 (FB)
- new net +3V3: Q7.2 (S), R65.1
- new net +5V_DCDC: C104.2, U6.5 (VIN)
- new net +5V_EG: C178.1, C233.2, U8.A2 (IN), U9.5 (IN)
- new net +5V_EPD: C160.2, C242.2, C245.2, C249.2, C37.2, C51.2, C53.2, Q1.2 (S), R228.2, R230.1, U31.5 (V+), U6.1 (VOUT)
- new net +5V_ES: C172.1, C173.2, U26.5 (IN), U7.A2 (IN)
- new net +5V_VGH: C232.2, L5.1, U24.4 (EN), U24.5 (IN), U8.A1 (OUT)
- new net +5V_VSH: C17.2, L30.1, U23.4 (EN), U23.5 (IN), U7.A1 (OUT)
- new net +VGH: C241.2, C244.2, D2.1 (K), R224.2
- new net +VP: C165.2, C166.2, C167.2, D15.1 (K), R78.2
- new net -VCOM: C56.2, Q6.3 (D), R64.2
- new net -VGL: C233.1, C246.1, D3.2 (A), D6.2 (A), R219.1, R94.1, U9.2 (GND)
- new net -VN: C173.1, C176.1, C177.1, C54.2, D17.2 (A), D6.1 (K), R226.1, R234.1, R62.2, R89.1, U26.2 (GND), U31.2 (V-)
- new net EN_VGL: R93.1, R94.2, U9.4 (~{SHDN})
- new net EN_VN: R234.2, R92.1, U26.4 (~{SHDN})
- new net EPD_POS_EN: U7.B2 (ON), U8.B2 (ON)
- new net EPD_PWR_EN: U6.4 (EN)
- new net GND: C104.1, C160.1, C166.1, C167.1, C17.1, C171.1, C172.2, C175.2, C176.2, C177.2, C178.2, C232.1, C242.1, C244.1, C245.1, C246.2, C249.1, C37.1, C38.2, C51.1, C52.1, C53.1, C54.1, C56.1, D5.2 (A), L32.2, L6.2, Q2.2 (E), R217.1, R218.2, R225.1, R229.1, R79.1, R88.2, U23.2 (GND), U24.2 (GND), U6.2 (GND), U7.B1 (GND), U8.B1 (GND)
- new net VCOM_DAC: D5.1 (K), R227.2
- new net VCOM_EN: R63.1
- new net VCOM_MEA: C171.2, Q8.2 (S), R65.2
- new net VCOM_MEA_EN: R66.2
- new net VGH_DAC: R213.2
Other:
- note added: "Ilim = 0.68A"
- note added: "Range: 0V ~ -2.7V"
- company: (none) -> Copyright 2025 Modos Tech Inc

Commit message: R2: MPNs into the schematic -- and five caps carry the wrong part number
Sourcing data lived in docs/*.md, not in the schematic, so the BOM the
fab would read had 3 of 96 lines with an MPN. Resolved every LCSC code
already on the board against LCSC's own catalogue and wrote MPN +
Manufacturer back: 53 -> 60 lines, 218 components. Added LCSC codes for
L10-L13, U42 and J22/J23 from the per-sheet docs.

Verified before writing: 321 refs and 519 nets identical before and
after, no duplicated properties, pre-existing MPNs untouched.

Cross-checking each passive value against the part its LCSC code
actually names found five wrong ones, all of them the ADC sense-divider
filter caps on power_mon:

  C91                 1nF/50V  carries C131394  = 100 nF
  C163 C164 C168 C169 1nF/25V  carries C6119801 = 470 nF

Left unwritten rather than cementing the error. C1523 (0402B102K500NT,
1 nF 50 V X7R 0402, JLC Basic, 5.3 M stock) covers both positions.

Also held back: U41, whose C39313 is XC6SLX16-**2**FTG256C while
fpga.md specifies the -3 speed grade.

frontlight.md cites C1848394 as the FPC connector on J22/J23; that code
is TPS22914BYFPR. The 6-pin sibling of J24's C5213749 is C5213748.

Co-Authored-By: Claude Opus 5 <noreply@anthropic.com>
Claude-Session: https://claude.ai/code/session_01MnesETWABbVdbcVnCKfKVs
Parts:
- C104, C17, C232, C242, C245, C249, C37, C51, C53: MPN (none) -> CL21A226MPQNNNE; Manufacturer (none) -> Samsung Electro-Mechanics
- C160, C171, C174, C35, C54: MPN (none) -> CC0402KRX7R9BB104; Manufacturer (none) -> YAGEO
- C165, C175, C241, C38: MPN (none) -> CC0402JRNPO9BN180; Manufacturer (none) -> YAGEO
- C166, C167, C173, C176, C177, C233, C244, C246: MPN (none) -> CGA0805X5R475K500MT; Manufacturer (none) -> HRE
- C172, C178, C52: MPN (none) -> CGA0402X5R474K250GT; Manufacturer (none) -> HRE
- C56: MPN (none) -> CL05A475MQ5NRNC; Manufacturer (none) -> Samsung Electro-Mechanics
- D1, D15, D17, D2, D3, D4, D5, D6: MPN (none) -> B5819WS; Manufacturer (none) -> Slkor
- L30, L32, L5, L6: MPN (none) -> WPN3012H4R7MT
- Q1, Q7, Q8: MPN (none) -> AO3401A; Manufacturer (none) -> UMW
- Q2: MPN (none) -> S8050; Manufacturer (none) -> Slkor
- Q6: MPN (none) -> AO3400A; Manufacturer (none) -> UMW
- R213, R226, R228, R234, R62, R92, R93, R94: MPN (none) -> 0402WGF1003TCE; Manufacturer (none) -> UNI-ROYAL
- R217, R219, R65: MPN (none) -> 0402WGF1002TCE; Manufacturer (none) -> UNI-ROYAL
- R218: MPN (none) -> 0402WGF2403TCE; Manufacturer (none) -> UNI-ROYAL
- R224, R88: MPN (none) -> 0402WGF3903TCE; Manufacturer (none) -> UNI-ROYAL
- R225, R227, R64, R89: MPN (none) -> 0402WGF2202TCE; Manufacturer (none) -> UNI-ROYAL
- R229, R230: MPN (none) -> 0402WGF5101TCE; Manufacturer (none) -> UNI-ROYAL
- R63, R66: MPN (none) -> 0402WGF330JTCE; Manufacturer (none) -> UNI-ROYAL
- R78: MPN (none) -> 0402WGF1503TCE; Manufacturer (none) -> UNI-ROYAL
- R79: MPN (none) -> 0402WGF1302TCE; Manufacturer (none) -> UNI-ROYAL
- U23, U24: MPN (none) -> LGS6302B5; Manufacturer (none) -> Legend-Si
- U26, U9: MPN (none) -> LGS5145; Manufacturer (none) -> Legend-Si
- U31: MPN (none) -> LM321MFX/NOPB; Manufacturer (none) -> TI
- U6: MPN (none) -> MT9700; Manufacturer (none) -> XI'AN Aerosemi Tech
- U7, U8: MPN (none) -> TPS22914BYFPR; Manufacturer (none) -> TI
