File: pcb/r2-mainboard/epd_power.kicad_sch (KiCad schematic)
At the start: 79 parts, among them Q1100 AO3401A, Q1101 S8050, Q1102 AO3400A, Q1103 AO3401A, Q1104 AO3401A, U1100 MT9700, U1101 TPS22914BYFPR, U1102 TPS22914BYFPR, U1103 LGS5145, U1104 LGS6302B5, U1105 LGS6302B5, U1106 LGS5145, U1107 LM321

Commit message: routing
Connections:
- net FB_VGH: now reaches C1124.1, R1112.1, R1116.1, R1117.2, U1105.3 (FB)
- net SW_VGH: now reaches D1101.2 (A), L1100.2, U1105.1 (SW)
- net FB_-VN: now reaches C1118.1, R1107.1, R1108.2, U1106.3 (FB)
- net SW_VP: now reaches D1106.2 (A), L1102.2, U1104.1 (SW)
- net FB_VP: now reaches C1111.1, R1105.1, R1106.2, U1104.3 (FB)

Commit message: changing to osb62x-pm
Parts:
- D1100, D1101, D1102, D1103, D1105, D1106, D1107: footprint footprints:D_SOD-323_Alt -> Diode_SMD:D_SOD-323
- U1101, U1102: footprint Package_BGA:WLP-4_0.83x0.83mm_P0.4mm -> Package_CSP:WLCSP-4_0.89x0.89mm_Layout2x2_P0.5mm

Commit message: Schematics update for new chip.
Parts:
- C1100, C1102, C1104, C1106, C1109, C1122, C1125, C1127, C1129: value 22uF/10V -> 22uF/25V
- C1108: value 4.7uF/6.3V -> 4.7uF/10V
- R1100, R1109, R1110, R1111, R1112, R1118, R1120, R1123: value 100K/1% -> 100k/1%
- R1102, R1108, R1119: value 22K/1% -> 22k/1%
- R1103, R1113: value 10K/1% -> 10k/1%
- R1105: value 150K/1% -> 150k/1%
- R1106: value 13K/1% -> 13k/1%
- R1107, R1116: value 390K/1% -> 390k/1%
- R1114: value 240K/1% -> 240k/1%
- R1115: value 10K/1% -> 10k/1%; footprint Resistor_SMD:R_0402_1005Metric -> Resistor_SMD:R_0603_1608Metric
- R1117: value 20.5K/1% -> 20.5k/1%
- R1121, R1122: value 5.1K/1% -> 5.1k/1%
Changed lines of the file:
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@@
 			)
 		)
-		(property "Value" "22uF/10V"
+		(property "Value" "22uF/25V"
 			(at 96.52 40.64 0)
 			(show_name no)
@@
 			)
 		)
-		(property "Value" "100K/1%"
+		(property "Value" "100k/1%"
 			(at 125.73 134.62 90)
 			(show_name no)
@@
 			)
 		)
-		(property "Value" "100K/1%"
+		(property "Value" "100k/1%"
 			(at 243.84 71.12 90)
 			(show_name no)
@@
 			)
 		)
-		(property "Value" "22uF/10V"
+		(property "Value" "22uF/25V"
 			(at 78.74 68.58 0)
 			(show_name no)
@@
 			)
 		)
-		(property "Value" "22uF/10V"
+		(property "Value" "22uF/25V"
 			(at 63.5 68.58 0)
 			(show_name no)
@@
 			)
 		)
-		(property "Value" "22uF/10V"
+		(property "Value" "22uF/25V"
 			(at 63.5 91.44 0)
 			(show_name no)
@@
 			)
 		)
-		(property "Value" "390K/1%"
+		(property "Value" "390k/1%"
 			(at 144.78 81.28 0)
 			(show_name no)
@@
 			)
 		)
-		(property "Value" "22K/1%"
+		(property "Value" "22k/1%"
 			(at 144.78 88.9 0)
 			(show_name no)
@@
 			)
 		)
-		(property "Value" "5.1K/1%"
+		(property "Value" "5.1k/1%"
 			(at 233.68 78.74 90)
 			(show_name no)
@@
 			)
 		)
-		(property "Value" "22uF/10V"
+		(property "Value" "22uF/25V"
 			(at 78.74 91.44 0)
 			(show_name no)
@@
 			)
 		)
-		(property "Value" "100K/1%"
+		(property "Value" "100k/1%"
 			(at 243.84 55.88 90)
 			(show_name no)
@@
 			)
 		)
-		(property "Value" "10K/1%"
+		(property "Value" "10k/1%"
 			(at 251.46 101.6 90)
 			(show_name no)
@@
 			)
 		)
-		(property "Value" "390K/1%"
+		(property "Value" "390k/1%"
 			(at 142.24 118.11 0)
 			(show_name no)
@@
 			)
 		)
-		(property "Value" "10K/1%"
+		(property "Value" "10k/1%"
 			(at 144.78 170.18 0)
 			(show_name no)
@@
 			)
 		)
-		(property "Footprint" "Resistor_SMD:R_0402_1005Metric"
+		(property "Footprint" "Resistor_SMD:R_0603_1608Metric"
 			(at 141.478 168.91 90)
 			(hide yes)
@@
 			)
 		)
-		(property "Value" "240K/1%"
+		(property "Value" "240k/1%"
 			(at 144.78 162.56 0)
 			(show_name no)
@@
 			)
 		)
-		(property "Value" "22K/1%"
+		(property "Value" "22k/1%"
 			(at 251.46 127 90)
 			(show_name no)
@@
 			)
 		)
-		(property "Value" "4.7uF/6.3V"
+		(property "Value" "4.7uF/10V"
 			(at 254 142.24 0)
 			(show_name no)
@@
 			)
 		)
-		(property "Value" "10K/1%"
+		(property "Value" "10k/1%"
 			(at 83.82 170.18 0)
 			(show_name no)
@@
 			)
 		)
-		(property "Value" "150K/1%"
+		(property "Value" "150k/1%"
 			(at 142.24 39.37 0)
 			(show_name no)
@@
 			)
 		)
-		(property "Value" "22uF/10V"
+		(property "Value" "22uF/25V"
 			(at 48.26 68.58 0)
 			(show_name no)
@@
 			)
 		)
-		(property "Value" "20.5K/1%"
+		(property "Value" "20.5k/1%"
 			(at 142.24 124.46 0)
 			(show_name no)
@@
 			)
 		)
-		(property "Value" "22uF/10V"
+		(property "Value" "22uF/25V"
 			(at 46.99 156.21 90)
 			(show_name no)
@@
 			)
 		)
-		(property "Value" "100K/1%"
+		(property "Value" "100k/1%"
 			(at 264.16 55.88 90)
 			(show_name no)
@@
 			)
 		)
-		(property "Value" "13K/1%"
+		(property "Value" "13k/1%"
 			(at 142.24 45.72 0)
 			(show_name no)
@@
 			)
 		)
-		(property "Value" "5.1K/1%"
+		(property "Value" "5.1k/1%"
 			(at 231.14 86.36 0)
 			(show_name no)
@@
 			)
 		)
-		(property "Value" "22K/1%"
+		(property "Value" "22k/1%"
 			(at 193.04 137.1599 0)
 			(show_name no)
@@
 			)
 		)
-		(property "Value" "100K/1%"
+		(property "Value" "100k/1%"
 			(at 264.16 71.12 90)
 			(show_name no)
@@
 			)
 		)
-		(property "Value" "22uF/10V"
+		(property "Value" "22uF/25V"
 			(at 48.26 91.44 0)
 			(show_name no)
@@
 			)
 		)
-		(property "Value" "100K/1%"
+		(property "Value" "100k/1%"
 			(at 193.04 129.5399 0)
 			(show_name no)
@@
 			)
 		)
-		(property "Value" "22uF/10V"
+		(property "Value" "22uF/25V"
 			(at 96.52 119.38 0)
 			(show_name no)
@@
 			)
 		)
-		(property "Value" "100K/1%"
+		(property "Value" "100k/1%"
 			(at 233.68 119.38 90)
 			(show_name no)
@@
 			)
 		)
-		(property "Value" "100K/1%"
+		(property "Value" "100k/1%"
 			(at 208.28 71.12 0)
 			(show_name no)
