File: pcb/r2-mainboard/fpga_ddr.kicad_sch (KiCad schematic)
At the start: 0 parts

Commit message: R2: WP5 -- fpga_ddr ported, and the FPGA's core rails get a home
fpga_ddr is the last of the three FPGA sheets. The port itself is mechanical:
all 49 local DDR nets come across node-for-node identical to R1 (only U1->U41,
U12->U52, R40->R340, R44->R344 rename), and the five +1V35 power symbols move
to +1V5 with the rest of the bank.

Unit 6 of the FPGA symbol -- 42 pins, 26 GND + 8 VCCAUX + 8 VCCINT -- had no
home in R2 at all. R1 draws it on power.kicad_sch; R2's power sheet is reviewed
and has no FPGA on it. Left as it was, ERC reported missing_unit forever and
eight VCCINT balls would have gone unconnected on the board. It lands here, on
A3, with its 12 decoupling capacitors relocated from R1's power sheet at +300.

One BOM change: C509, a fifth 4.7 uF on VCCINT. UG393 Table 2-1 p.14 row
FT(G)256 LX16 asks for five and R1 fits four. Everything else in that table
either matches or is the 100 uF-vs-more-4.7 uF trade its own note 3 permits,
which R1's working board already settles -- so it is written up, not changed.

tools/check_ucf.py grew the checks this sheet made possible, and they matter:
before, all 48 MCB3 balls fell through to "no expected-name rule", so the one
bank where a single swap is fatal and invisible was verified for nothing.

  - DDR_* name mappings, so those 48 balls are actually compared
  - DDR_RZQ and DDR_ZIO checked by shape instead of by name: RZQ must reach
    exactly one 100R to GND (2x the UCF's UNTUNED_50), ZIO must be left open.
    Both mandatory because s6_ddr3.v sets C3_CALIB_SOFT_IP = "TRUE"
  - all 14 LVDS ports asserted open, which catches a half-finished deletion
  - bank VCCO now read out of the schematic's own VCCO_n balls instead of a
    hand-maintained table -- a stale table is exactly the failure this script
    exists to catch, and it reports a bank split across two nets as a defect

Result: 113 UCF LOC lines, all accounted for -- 97 name-matched, 2 structural,
14 asserted-open, 0 failures, 0 pending, 0 unexplained.

Thre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
Parts:
- added C144, C71, C72, C74, C75, C76, C77, C78, C88: 100nF/50V, Capacitor_SMD:C_0402_1005Metric, symbol Device:C
- added C318, C319, C320, C321, C85, C86, C87: 22uF/6.3V, Capacitor_SMD:C_0603_1608Metric, symbol Device:C
- added C322, C323, C324, C357, C359, C509: 4.7uF/6.3V, Capacitor_SMD:C_0402_1005Metric, symbol Device:C
- added C325, C358, C368, C69, C70, C73, C79, C80, C81, C82, C83, C84: 470nF/25V, Capacitor_SMD:C_0402_1005Metric, symbol Device:C
- added R100, R340: 100R/1%, Resistor_SMD:R_0402_1005Metric, symbol Device:R
- added R101, R103, R344: 5.1K/1%, Resistor_SMD:R_0402_1005Metric, symbol Device:R
- added R102: 240R/1%, Resistor_SMD:R_0402_1005Metric, symbol Device:R
- added R104, R105: 1K/1%, Resistor_SMD:R_0402_1005Metric, symbol Device:R
- added U41: XC6SLX-FTG256, footprints:Xilinx_FTG256, symbol symbols:XC6SLX-FTG256
- added U52: MT41K64M16TW, footprints:BGA-96_9.0x14.0mm_P0.8mm, symbol symbols:MT41K256M16HA
Connections:
- new net: R102.1, U52.L8 (ZQ)
- new net: R340.1, U41.M4 (IO_L1P_3)
- new net +1V2_FPGA: C318.1, C320.1, C322.1, C324.1, C357.1, C359.1, C368.1, C509.1, U41.G7 (VCCINT), U41.G9 (VCCINT), U41.H10 (VCCINT), U41.H8 (VCCINT), U41.J7 (VCCINT), U41.J9 (VCCINT), U41.K10 (VCCINT), U41.K8 (VCCINT)
- new net +1V5: C71.1, C72.1, C74.1, C75.1, C77.1, C78.1, C79.1, C80.1, C81.1, C82.1, C83.1, C84.1, C85.1, C86.1, C87.1, C88.1, R104.1, U41.D2 (VCCO_3), U41.G4 (VCCO_3), U41.J2 (VCCO_3), U41.K4 (VCCO_3), U41.N2 (VCCO_3), U52.A1 (VDDQ), U52.A8 (VDDQ), U52.B2 (VDD), U52.C1 (VDDQ), U52.C9 (VDDQ), U52.D2 (VDDQ), U52.D9 (VDD), U52.E9 (VDDQ), U52.F1 (VDDQ), U52.G7 (VDD), U52.H2 (VDDQ), U52.H9 (VDDQ), U52.K2 (VDD), U52.K8 (VDD), U52.N1 (VDD), U52.N9 (VDD), U52.R1 (VDD), U52.R9 (VDD)
- new net +3V3: C319.1, C321.1, C323.1, C325.1, C358.1, U41.E5 (VCCAUX), U41.F11 (VCCAUX), U41.F8 (VCCAUX), U41.G10 (VCCAUX), U41.H6 (VCCAUX), U41.J10 (VCCAUX), U41.L6 (VCCAUX), U41.L9 (VCCAUX)
- new net +DRAM_VREF: C144.1, C69.1, C70.1, C73.1, C76.1, C88.2, R104.2, R105.1, U41.A3 (IO_L83N_VREF_3), U41.M3 (IO_L1N_VREF_3), U52.H1 (VrefDQ), U52.M8 (VrefCA)
- new net DRAM_ADDR0: U41.K5 (IO_L47P_M3A0_3), U52.N3 (A0)
- new net DRAM_ADDR1: U41.K6 (IO_L47N_M3A1_3), U52.P7 (A1)
- new net DRAM_ADDR10: U41.G6 (IO_L51P_M3A10_3), U52.L7 (A10)
- new net DRAM_ADDR11: U41.E3 (IO_L54N_M3A11_3), U52.R7 (A11)
- new net DRAM_ADDR12: U41.F3 (IO_L53N_M3A12_3), U52.N7 (A12/~{BC})
- new net DRAM_ADDR13: U41.F6 (IO_L55P_M3A13_3), U52.T3 (A13)
- new net DRAM_ADDR14: U41.F5 (IO_L55N_M3A14_3), U52.T7 (A14/NC)
- new net DRAM_ADDR2: U41.D1 (IO_L49N_M3A2_3), U52.P3 (A2)
- new net DRAM_ADDR3: U41.L4 (IO_L45P_M3A3_3), U52.N2 (A3)
- new net DRAM_ADDR4: U41.G5 (IO_L51N_M3A4_3), U52.P8 (A4)
- new net DRAM_ADDR5: U41.H4 (IO_L44P_GCLK21_M3A5_3), U52.P2 (A5)
- new net DRAM_ADDR6: U41.H3 (IO_L44N_GCLK20_M3A6_3), U52.R8 (A6)
- new net DRAM_ADDR7: U41.D3 (IO_L49P_M3A7_3), U52.R2 (A7)
- new net DRAM_ADDR8: U41.B2 (IO_L52P_M3A8_3), U52.T8 (A8)
- new net DRAM_ADDR9: U41.A2 (IO_L52N_M3A9_3), U52.R3 (A9)
- new net DRAM_BA0: U41.C3 (IO_L48P_M3BA0_3), U52.M2 (BA0)
- new net DRAM_BA1: U41.C2 (IO_L48N_M3BA1_3), U52.N8 (BA1)
- new net DRAM_BA2: U41.B1 (IO_L50N_M3BA2_3), U52.M3 (BA2)
- new net DRAM_CASB: U41.H5 (IO_L43N_GCLK22_IRDY2_M3CASN_3), U52.K3 (~{CAS})
- new net DRAM_CKE: R344.1, U41.F4 (IO_L53P_M3CKE_3), U52.K9 (CKE)
- new net DRAM_CKN: R100.1, U41.E1 (IO_L46N_M3CLKN_3), U52.K7 (~{CK})
- new net DRAM_CKP: R100.2, U41.E2 (IO_L46P_M3CLK_3), U52.J7 (CK)
- new net DRAM_CSB: R101.1, U52.L2 (~{CS})
- new net DRAM_DATA0: U41.K2 (IO_L37P_M3DQ0_3), U52.E3 (DQ0)
- new net DRAM_DATA1: U41.K1 (IO_L37N_M3DQ1_3), U52.F7 (DQ1)
- new net DRAM_DATA10: U41.M2 (IO_L35P_M3DQ10_3), U52.C8 (DQ10)
- new net DRAM_DATA11: U41.M1 (IO_L35N_M3DQ11_3), U52.C2 (DQ11)
- new net DRAM_DATA12: U41.P2 (IO_L33P_M3DQ12_3), U52.A7 (DQ12)
- new net DRAM_DATA13: U41.P1 (IO_L33N_M3DQ13_3), U52.A2 (DQ13)
- new net DRAM_DATA14: U41.R2 (IO_L32P_M3DQ14_3), U52.B8 (DQ14)
- new net DRAM_DATA15: U41.R1 (IO_L32N_M3DQ15_3), U52.A3 (DQ15)
- new net DRAM_DATA2: U41.J3 (IO_L38P_M3DQ2_3), U52.F2 (DQ2)
- new net DRAM_DATA3: U41.J1 (IO_L38N_M3DQ3_3), U52.F8 (DQ3)
- new net DRAM_DATA4: U41.F2 (IO_L41P_GCLK27_M3DQ4_3), U52.H3 (DQ4)
- new net DRAM_DATA5: U41.F1 (IO_L41N_GCLK26_M3DQ5_3), U52.H8 (DQ5)
- new net DRAM_DATA6: U41.G3 (IO_L40P_M3DQ6_3), U52.G2 (DQ6)
- new net DRAM_DATA7: U41.G1 (IO_L40N_M3DQ7_3), U52.H7 (DQ7)
- new net DRAM_DATA8: U41.L3 (IO_L36P_M3DQ8_3), U52.D7 (DQ8)
- new net DRAM_DATA9: U41.L1 (IO_L36N_M3DQ9_3), U52.C3 (DQ9)
- new net DRAM_LDM: U41.J4 (IO_L42N_GCLK24_M3LDM_3), U52.E7 (LDM)
- new net DRAM_LDQSN: U41.H1 (IO_L39N_M3LDQSN_3), U52.G3 (~{LDQS})
- new net DRAM_LDQSP: U41.H2 (IO_L39P_M3LDQS_3), U52.F3 (LDQS)
- new net DRAM_ODT: U41.L5 (IO_L45N_M3ODT_3), U52.K1 (ODT)
- new net DRAM_RASB: U41.J6 (IO_L43P_GCLK23_M3RASN_3), U52.J3 (~{RAS})
- new net DRAM_RST: R103.1, U41.E4 (IO_L54P_M3RESET_3), U52.T2 (~{RESET})
- new net DRAM_UDM: U41.K3 (IO_L42P_GCLK25_TRDY2_M3UDM_3), U52.D3 (UDM)
- new net DRAM_UDQSN: U41.N1 (IO_L34N_M3UDQSN_3), U52.B7 (~{UDQS})
- new net DRAM_UDQSP: U41.N3 (IO_L34P_M3UDQS_3), U52.C7 (UDQS)
- new net DRAM_WEB: U41.C1 (IO_L50P_M3WE_3), U52.L3 (~{WE})
- new net GND: C144.2, C318.2, C319.2, C320.2, C321.2, C322.2, C323.2, C324.2, C325.2, C357.2, C358.2, C359.2, C368.2, C509.2, C69.2, C70.2, C71.2, C72.2, C73.2, C74.2, C75.2, C76.2, C77.2, C78.2, C79.2, C80.2, C81.2, C82.2, C83.2, C84.2, C85.2, C86.2, C87.2, R101.2, R102.2, R103.2, R105.2, R340.2, R344.2, U41.A1 (GND), U41.A16 (GND), U41.B11 (GND), U41.B7 (GND), U41.D13 (GND), U41.D4 (GND), U41.E9 (GND), U41.G15 (GND), U41.G2 (GND), U41.G8 (GND), U41.H12 (GND), U41.H7 (GND), U41.H9 (GND), U41.J5 (GND), U41.J8 (GND), U41.K7 (GND), U41.K9 (GND), U41.L15 (GND), U41.L2 (GND), U41.M8 (GND), U41.N13 (GND), U41.P3 (GND), U41.R10 (GND), U41.R6 (GND), U41.T1 (GND), U41.T16 (GND), U52.A9 (VSS), U52.B1 (VSSQ), U52.B3 (VSS), U52.B9 (VSSQ), U52.D1 (VSSQ), U52.D8 (VSSQ), U52.E1 (VSS), U52.E2 (VSSQ), U52.E8 (VSSQ), U52.F9 (VSSQ), U52.G1 (VSSQ), U52.G8 (VSS), U52.G9 (VSSQ), U52.J1 (VSS), U52.J2 (VSS), U52.J8 (VSS), U52.J9 (VSS), U52.L1 (VSS), U52.L9 (VSS), U52.M1 (VSS), U52.M9 (VSS), U52.P1 (VSS), U52.P9 (VSS), U52.T1 (VSS), U52.T9 (VSS)
- no-connect marks 0 -> 4
Other:
- note added: "(DDR_A is [12:0]). Kept routed: T3/T7 are the density-expansion balls, so"
- note added: "Bank 3 VCCO is 1.5 V, not R1's 1.35 V: the UCF constrains DDR_RESET_N as"
- note added: "CAP for DRAM0"
- note added: "DRAM_ADDR13/14 reach U52 balls T3/T7, which the fitted 1 Gb MT41K64M16"
- note added: "DRAM_CSB is tied low by R101 and reaches no FPGA pin: the MCB has no chip"
- note added: "FPGA core rails. Unit 6 of U41 is 26 GND + 8 VCCAUX + 8 VCCINT; R1 draws"
- note added: "LVCMOS15 and the rest of the bank SSTL15_II, and DS162 Table 7 specifies"
- note added: "M5 (DDR_ZIO) is reserved for MCB calibration, not spare -- leave it open."
- note added: "SSTL15 over 1.425-1.575 V only. VREF = R104/R105 = 1.500/2 = 0.750 V."
- note added: "ZIO"
- note added: "a 2 Gb or 4 Gb part stays a gateware-only change."
- note added: "does not bond (Micron 1Gb_DDR3L Rev L Fig 7 p.18) and top.v never drives"
- note added: "it on power.kicad_sch, which in R2 has no FPGA. C509 is the fifth 4.7uF"
- note added: "on VCCINT that UG393 Table 2-1 (FTG256 LX16) wants and R1 does not fit."
- note added: "select (no DDR_CS_N in constraint.ucf, no such port in top.v)."
- company: (none) -> Copyright 2025 Modos Tech Inc

Commit message: R2: MPNs into the schematic -- and five caps carry the wrong part number
Sourcing data lived in docs/*.md, not in the schematic, so the BOM the
fab would read had 3 of 96 lines with an MPN. Resolved every LCSC code
already on the board against LCSC's own catalogue and wrote MPN +
Manufacturer back: 53 -> 60 lines, 218 components. Added LCSC codes for
L10-L13, U42 and J22/J23 from the per-sheet docs.

Verified before writing: 321 refs and 519 nets identical before and
after, no duplicated properties, pre-existing MPNs untouched.

Cross-checking each passive value against the part its LCSC code
actually names found five wrong ones, all of them the ADC sense-divider
filter caps on power_mon:

  C91                 1nF/50V  carries C131394  = 100 nF
  C163 C164 C168 C169 1nF/25V  carries C6119801 = 470 nF

Left unwritten rather than cementing the error. C1523 (0402B102K500NT,
1 nF 50 V X7R 0402, JLC Basic, 5.3 M stock) covers both positions.

Also held back: U41, whose C39313 is XC6SLX16-**2**FTG256C while
fpga.md specifies the -3 speed grade.

frontlight.md cites C1848394 as the FPC connector on J22/J23; that code
is TPS22914BYFPR. The 6-pin sibling of J24's C5213749 is C5213748.

Co-Authored-By: Claude Opus 5 <noreply@anthropic.com>
Claude-Session: https://claude.ai/code/session_01MnesETWABbVdbcVnCKfKVs
Parts:
- C144, C71, C72, C74, C75, C76, C77, C78, C88: MPN (none) -> CC0402KRX7R9BB104; Manufacturer (none) -> YAGEO
- C318, C319, C320, C321, C85, C86, C87: MPN (none) -> CL10A226MQ8NRNC; Manufacturer (none) -> Samsung Electro-Mechanics
- C322, C323, C324, C357, C359, C509: MPN (none) -> CL05A475MQ5NRNC; Manufacturer (none) -> Samsung Electro-Mechanics
- C325, C358, C368, C69, C70, C73, C79, C80, C81, C82, C83, C84: MPN (none) -> CGA0402X5R474K250GT; Manufacturer (none) -> HRE
- R100, R340: MPN (none) -> 0402WGF1000TCE; Manufacturer (none) -> UNI-ROYAL
- R101, R103, R344: MPN (none) -> 0402WGF5101TCE; Manufacturer (none) -> UNI-ROYAL
- R102: MPN (none) -> 0402WGF2400TCE; Manufacturer (none) -> UNI-ROYAL
- R104, R105: MPN (none) -> 0402WGF1001TCE; Manufacturer (none) -> UNI-ROYAL
- U52: MPN (none) -> MT41K64M16TW-107 IT:J; Manufacturer (none) -> micron
