File: pcb/r2-mainboard/fpga_ddr.kicad_sch (KiCad schematic)
At the start: 44 parts, among them U41 XC6SLX-FTG256, U52 MT41K64M16TW

Commit message: change layout and reduce board size + add second usb host only
Other:
- note added: "VCCAUX"
- note added: "VCCINT"
Changed lines of the file:
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@@
+		)
+	)
+	(text "VCCINT"
+		(exclude_from_sim no)
+		(at 397.764 144.272 0)
+		(effects
+			(font
+				(size 1.27 1.27)
+			)
 		)
 	)
@@
 		)
 	)
+	(text "VCCAUX"
+		(exclude_from_sim no)
+		(at 362.458 172.212 0)
+		(effects
+			(font
+				(size 1.27 1.27)
+			)
+		)
+	)
