File: pcb/r2-mainboard/fpga_ddr.kicad_sch (KiCad schematic)
At the start: 44 parts, among them U41 XC6SLX-FTG256, U52 MT41K64M16TW

Commit message: R2: renumber every sheet to the page-based designator scheme
The owner's scheme is classifier + sheet page + two-digit part from 00. Four
sheets already used it; this converts the remaining nine, so all thirteen now
agree: pages 2-9 take three digits, pages 10-14 four. 292 of 333 designators
changed. A part shared by several sheets takes its lowest page, so the FPGA is
U700 (pages 7-9) and the two SoM connectors are J501/J502 (pages 5-6).

The whole risk here is silently rewiring the board, so the netlist was diffed
rather than eyeballed:

  nets 519 -> 519, total pin connections 1563 -> 1563
  named nets present in both whose pin multiset changed: 0
  ERC unchanged at 14 errors / 20 warnings
  check_ucf.py: 99 balls matched, 0 failures

That last one matters most: it resolves the gateware's 113 UCF constraints to
board nets *by ball name*, so it is the sharpest detector of the corruption
this change could cause.

Two earlier attempts did cause exactly that. A bare quoted-string substitution
also rewrites FPGA ball names (C1, D2, N11, T1) and BTH-060 pin names (A1-D60),
which are spelled exactly like designators; one run left ERC identical while 40
nets came back with a different pin multiset. The tool now substitutes only at
the two positions that store an instance's designator, and excludes every pin
name everywhere else. docs/layout.md 9.5 records the hazard and how to prove a
renumber was clean.

Only the three scripts that read the design are updated. The gen_*/patch_*/
port_r1.py scripts keep the old names deliberately: each wrote a sheet once and
has not been re-runnable since it was hand-edited in Eeschema, so they are a
historical record -- and port_r1.py's dict keys are R1 designators that were
never renumbered at all.

Co-Authored-By: Claude Opus 5 <noreply@anthropic.com>
Claude-Session: https://claude.ai/code/session_01MHTAe6ZnhogTEgtyPcLhwG
Parts:
- renumbered C69 to C800, C70 to C801, C71 to C802, C72 to C803, C73 to C804, C74 to C805, C75 to C806, C76 to C807, C77 to C808, C78 to C809, C79 to C810, C80 to C811, C81 to C812, C82 to C813, C83 to C814, C84 to C815, C85 to C816, C86 to C817, C87 to C818, C88 to C819, C144 to C820, C318 to C821, C319 to C822, C320 to C823, C321 to C824, C322 to C825, C323 to C826, C324 to C827, C325 to C828, C357 to C829, C358 to C830, C359 to C831, C368 to C832, C509 to C833, R100 to R800, R101 to R801, R102 to R802, R103 to R803, R104 to R804, R105 to R805, R340 to R806, R344 to R807, U41 to U700, U52 to U800
