File: pcb/r2-mainboard/fpga_ddr.kicad_sch (KiCad schematic)
At the start: 44 parts, among them U700 XC6SLX-FTG256, U800 MT41K64M16TW

Commit message: routing
Connections:
- net DRAM_DATA10: now also U800.A2 (DQ13); no longer U800.C8 (DQ10)
- net DRAM_DATA11: now also U800.A3 (DQ15); no longer U800.C2 (DQ11)
- net DRAM_DATA12: now also U800.C3 (DQ9); no longer U800.A7 (DQ12)
- net DRAM_DATA13: now also U800.C8 (DQ10); no longer U800.A2 (DQ13)
- net DRAM_DATA15: now also U800.A7 (DQ12); no longer U800.A3 (DQ15)
- net DRAM_DATA9: now also U800.C2 (DQ11); no longer U800.C3 (DQ9)
Other:
- moved on the sheet: C804
Changed lines of the file:
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@@
 	)
 	(junction
+		(at 185.42 33.02)
+		(diameter 0)
+		(color 0 0 0 0)
+	)
+	(junction
 		(at 299.72 87.63)
 		(diameter 0)
@@
 	)
 	(junction
-		(at 185.42 33.02)
-		(diameter 0.9144)
-		(color 0 0 0 0)
-	)
-	(junction
 		(at 353.06 161.29)
 		(diameter 0)
@@
 	)
 	(junction
-		(at 175.26 33.02)
+		(at 167.64 33.02)
 		(diameter 0)
 		(color 0 0 0 0)
@@
 	)
 	(junction
-		(at 175.26 40.64)
+		(at 167.64 40.64)
 		(diameter 0.9144)
 		(color 0 0 0 0)
@@
 	(wire
 		(pts
-			(xy 175.26 33.02) (xy 185.42 33.02)
+			(xy 167.64 33.02) (xy 185.42 33.02)
 		)
 		(stroke
@@
 	(wire
 		(pts
+			(xy 248.92 40.64) (xy 233.68 40.64)
+		)
+		(stroke
+			(width 0)
+			(type default)
+		)
+	)
+	(wire
+		(pts
 			(xy 193.04 66.04) (xy 208.28 66.04)
 		)
@@
 	(wire
 		(pts
-			(xy 233.68 40.64) (xy 248.92 40.64)
-		)
-		(stroke
-			(width 0)
-			(type default)
-		)
-	)
-	(wire
-		(pts
 			(xy 170.18 162.56) (xy 180.34 162.56)
 		)
@@
 	(wire
 		(pts
-			(xy 185.42 40.64) (xy 175.26 40.64)
+			(xy 167.64 40.64) (xy 185.42 40.64)
 		)
 		(stroke
@@
 	)
 	(label "DRAM_DATA11"
-		(at 248.92 43.18 180)
+		(at 248.92 33.02 180)
 		(effects
 			(font
@@
 	)
 	(label "DRAM_DATA15"
-		(at 248.92 33.02 180)
+		(at 248.92 40.64 180)
 		(effects
 			(font
@@
 	)
 	(label "DRAM_DATA13"
-		(at 248.92 38.1 180)
+		(at 248.92 45.72 180)
 		(effects
 			(font
@@
 	)
 	(label "DRAM_DATA12"
-		(at 248.92 40.64 180)
+		(at 248.92 48.26 180)
 		(effects
 			(font
@@
 	)
 	(label "DRAM_DATA10"
-		(at 248.92 45.72 180)
+		(at 248.92 38.1 180)
 		(effects
 			(font
@@
 	)
 	(label "DRAM_DATA9"
-		(at 248.92 48.26 180)
+		(at 248.92 43.18 180)
 		(effects
 			(font
@@
 	(symbol
 		(lib_id "Device:C")
-		(at 175.26 36.83 0)
+		(at 167.64 36.83 0)
 		(unit 1)
 		(body_style 1)
@@
 		(dnp no)
 		(property "Reference" "C804"
-			(at 178.181 35.6616 0)
+			(at 170.561 35.6616 0)
 			(show_name no)
 			(do_not_autoplace no)
@@
 		)
 		(property "Value" "470nF/25V"
-			(at 178.181 37.973 0)
+			(at 170.561 37.973 0)
 			(show_name no)
 			(do_not_autoplace no)
@@
 		)
 		(property "Footprint" "Capacitor_SMD:C_0402_1005Metric"
-			(at 176.2252 40.64 0)
+			(at 168.6052 40.64 0)
 			(hide yes)
 			(show_name no)
@@
 		)
 		(property "Datasheet" ""
-			(at 175.26 36.83 0)
+			(at 167.64 36.83 0)
 			(hide yes)
 			(show_name no)
@@
 		)
 		(property "Description" ""
-			(at 175.26 36.83 0)
+			(at 167.64 36.83 0)
 			(hide yes)
 			(show_name no)
@@
 		)
 		(property "Ref.Price" "0.0036"
-			(at 175.26 36.83 0)
+			(at 167.64 36.83 0)
 			(hide yes)
 			(show_name no)
@@
 		)
 		(property "desc" ""
-			(at 175.26 36.83 0)
+			(at 167.64 36.83 0)
 			(hide yes)
 			(show_name no)
@@
 		)
 		(property "LCSC" "C6119801"
-			(at 175.26 36.83 0)
+			(at 167.64 36.83 0)
 			(hide yes)
 			(show_name no)
@@
 		)
 		(property "Manufacturer" "HRE"
-			(at 0 0 0)
+			(at -7.62 0 0)
 			(hide yes)
 			(show_name no)
@@
 		)
 		(property "MPN" "CGA0402X5R474K250GT"
-			(at 0 0 0)
+			(at -7.62 0 0)
 			(hide yes)
 			(show_name no)
@@
 	(symbol
 		(lib_id "power:GND")
-		(at 175.26 40.64 0)
+		(at 167.64 40.64 0)
 		(unit 1)
 		(body_style 1)
@@
 		(dnp no)
 		(property "Reference" "#PWR0234"
-			(at 175.26 46.99 0)
+			(at 167.64 46.99 0)
 			(hide yes)
 			(show_name no)
@@
 		)
 		(property "Value" "GND"
-			(at 175.387 45.0342 0)
+			(at 167.767 45.0342 0)
 			(show_name no)
 			(do_not_autoplace no)
@@
 		)
 		(property "Footprint" ""
-			(at 175.26 40.64 0)
+			(at 167.64 40.64 0)
 			(hide yes)
 			(show_name no)
@@
 		)
 		(property "Datasheet" ""
-			(at 175.26 40.64 0)
+			(at 167.64 40.64 0)
 			(hide yes)
 			(show_name no)
@@
 		)
 		(property "Description" ""
-			(at 175.26 40.64 0)
+			(at 167.64 40.64 0)
 			(hide yes)
 			(show_name no)
@@
 	(symbol
 		(lib_id "symbols:+V")
-		(at 175.26 33.02 0)
+		(at 167.64 33.02 0)
 		(unit 1)
 		(body_style 1)
@@
 		(dnp no)
 		(property "Reference" "#PWR0100"
-			(at 175.26 36.83 0)
+			(at 167.64 36.83 0)
 			(hide yes)
 			(show_name no)
@@
 		)
 		(property "Value" "+DRAM_VREF"
-			(at 175.26 27.94 0)
+			(at 167.64 27.94 0)
 			(show_name no)
 			(do_not_autoplace no)
@@
 		)
 		(property "Footprint" ""
-			(at 175.26 33.02 0)
+			(at 167.64 33.02 0)
 			(hide yes)
 			(show_name no)
@@
 		)
 		(property "Datasheet" ""
-			(at 175.26 33.02 0)
+			(at 167.64 33.02 0)
 			(hide yes)
 			(show_name no)
@@
 		)
 		(property "Description" ""
-			(at 175.26 33.02 0)
+			(at 167.64 33.02 0)
 			(hide yes)
 			(show_name no)

Commit message: changing to osb62x-pm
Parts:
- U800: footprint footprints:BGA-96_9.0x14.0mm_P0.8mm -> Package_BGA:BGA-96_9.0x13.0mm_Layout2x3x16_P0.8mm
Connections:
- net DRAM_DATA1: now also U800.F8 (DQ3); no longer U800.F7 (DQ1)
- net DRAM_DATA12: now also U800.C8 (DQ10); no longer U800.C3 (DQ9)
- net DRAM_DATA13: now also U800.D7 (DQ8); no longer U800.C8 (DQ10)
- net DRAM_DATA3: now also U800.G2 (DQ6); no longer U800.F8 (DQ3)
- net DRAM_DATA4: now also U800.H8 (DQ5); no longer U800.H3 (DQ4)
- net DRAM_DATA5: now also U800.H7 (DQ7); no longer U800.H8 (DQ5)
- net DRAM_DATA6: now also U800.H3 (DQ4); no longer U800.G2 (DQ6)
- net DRAM_DATA7: now also U800.F7 (DQ1); no longer U800.H7 (DQ7)
- net DRAM_DATA8: now also U800.C3 (DQ9); no longer U800.D7 (DQ8)

Commit message: Schematics update for new chip.
Parts:
- C816, C817, C818, C821, C822, C823, C824: value 22uF/6.3V -> 22uF/25V; footprint Capacitor_SMD:C_0603_1608Metric -> Capacitor_SMD:C_0805_2012Metric
- C825, C826, C827, C829, C831, C833: value 4.7uF/6.3V -> 4.7uF/10V
- R801, R803, R807: value 5.1K/1% -> 5.1k/1%
- R804, R805: value 1K/1% -> 1k/1%
Changed lines of the file:
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@@
 			)
 		)
-		(property "Value" "1K/1%"
+		(property "Value" "1k/1%"
 			(at 250.698 142.113 0)
 			(show_name no)
@@
 			)
 		)
-		(property "Value" "4.7uF/6.3V"
+		(property "Value" "4.7uF/10V"
 			(at 342.9 156.21 0)
 			(show_name no)
@@
 			)
 		)
-		(property "Value" "5.1K/1%"
+		(property "Value" "5.1k/1%"
 			(at 179.578 119.253 0)
 			(show_name no)
@@
 			)
 		)
-		(property "Value" "4.7uF/6.3V"
+		(property "Value" "4.7uF/10V"
 			(at 381 156.21 0)
 			(show_name no)
@@
 			)
 		)
-		(property "Value" "5.1K/1%"
+		(property "Value" "5.1k/1%"
 			(at 189.738 119.253 0)
 			(show_name no)
@@
 			)
 		)
-		(property "Value" "4.7uF/6.3V"
+		(property "Value" "4.7uF/10V"
 			(at 330.2 182.88 0)
 			(show_name no)
@@
 			)
 		)
-		(property "Value" "22uF/6.3V"
+		(property "Value" "22uF/25V"
 			(at 223.901 159.893 0)
 			(show_name no)
@@
 			)
 		)
-		(property "Footprint" "Capacitor_SMD:C_0603_1608Metric"
+		(property "Footprint" "Capacitor_SMD:C_0805_2012Metric"
 			(at 221.9452 162.56 0)
 			(hide yes)
@@
 			)
 		)
-		(property "Value" "22uF/6.3V"
+		(property "Value" "22uF/25V"
 			(at 317.5 156.21 0)
 			(show_name no)
@@
 			)
 		)
-		(property "Footprint" "Capacitor_SMD:C_0603_1608Metric"
+		(property "Footprint" "Capacitor_SMD:C_0805_2012Metric"
 			(at 314.96 152.4 0)
 			(hide yes)
@@
 			)
 		)
-		(property "Value" "22uF/6.3V"
+		(property "Value" "22uF/25V"
 			(at 317.5 182.88 0)
 			(show_name no)
@@
 			)
 		)
-		(property "Footprint" "Capacitor_SMD:C_0603_1608Metric"
+		(property "Footprint" "Capacitor_SMD:C_0805_2012Metric"
 			(at 314.96 179.07 0)
 			(hide yes)
@@
 			)
 		)
-		(property "Value" "4.7uF/6.3V"
+		(property "Value" "4.7uF/10V"
 			(at 368.3 156.21 0)
 			(show_name no)
@@
 			)
 		)
-		(property "Value" "22uF/6.3V"
+		(property "Value" "22uF/25V"
 			(at 304.8 182.88 0)
 			(show_name no)
@@
 			)
 		)
-		(property "Footprint" "Capacitor_SMD:C_0603_1608Metric"
+		(property "Footprint" "Capacitor_SMD:C_0805_2012Metric"
 			(at 302.26 179.07 0)
 			(hide yes)
@@
 			)
 		)
-		(property "Value" "5.1K/1%"
+		(property "Value" "5.1k/1%"
 			(at 253.238 119.253 0)
 			(show_name no)
@@
 			)
 		)
-		(property "Value" "22uF/6.3V"
+		(property "Value" "22uF/25V"
 			(at 223.901 139.573 0)
 			(show_name no)
@@
 			)
 		)
-		(property "Footprint" "Capacitor_SMD:C_0603_1608Metric"
+		(property "Footprint" "Capacitor_SMD:C_0805_2012Metric"
 			(at 221.9452 142.24 0)
 			(hide yes)
@@
 			)
 		)
-		(property "Value" "22uF/6.3V"
+		(property "Value" "22uF/25V"
 			(at 304.8 156.21 0)
 			(show_name no)
@@
 			)
 		)
-		(property "Footprint" "Capacitor_SMD:C_0603_1608Metric"
+		(property "Footprint" "Capacitor_SMD:C_0805_2012Metric"
 			(at 302.26 152.4 0)
 			(hide yes)
@@
 			)
 		)
-		(property "Value" "1K/1%"
+		(property "Value" "1k/1%"
 			(at 250.698 154.813 0)
 			(show_name no)
@@
 			)
 		)
-		(property "Value" "4.7uF/6.3V"
+		(property "Value" "4.7uF/10V"
 			(at 330.2 156.21 0)
 			(show_name no)
@@
 			)
 		)
-		(property "Value" "4.7uF/6.3V"
+		(property "Value" "4.7uF/10V"
 			(at 355.6 156.21 0)
 			(show_name no)
@@
 			)
 		)
-		(property "Value" "22uF/6.3V"
+		(property "Value" "22uF/25V"
 			(at 241.681 147.193 0)
 			(show_name no)
@@
 			)
 		)
-		(property "Footprint" "Capacitor_SMD:C_0603_1608Metric"
+		(property "Footprint" "Capacitor_SMD:C_0805_2012Metric"
 			(at 239.7252 149.86 0)
 			(hide yes)
