File: pcb/r2-mainboard/fpga_io.kicad_sch (KiCad schematic)
At the start: 0 parts

Commit message: R2: WP5 -- fpga_io ported, verified pin-for-pin against R1
Banks 0 and 1 of the XC6SLX16: the EPD panel bus out, DPI in. Ported from R1 by
an extended tools/port_r1.py rather than redrawn, so the pinout the gateware
depends on cannot drift -- Caster's constraint.ucf fixes almost all of it and
ISE 14.7 is the only toolchain that still targets Spartan-6.

RESULT
69 signal nets identical to R1, zero mismatches: every EPDC_*, DPI_*, LED,
EPD_THROT and VCCO ball lands on exactly the pin R1 used. All 33 EPDC_*
hierarchical labels on epd.kicad_sch have exactly one source here, no more and
no fewer. ERC on /fpga_io/ is 4, all of them "units C/D/E/F of U41 are not
placed yet" (missing_unit, missing_power_pin, missing_bidi_pin,
power_pin_not_driven) which resolve as fpga_ddr, fpga_config and unit 6 land.

THE 12 FMC SIGNALS ARE DELETED
R1 wires a 12-signal parallel bus between the H750's FMC and the FPGA --
FMC_A16, FMC_D0-D7, FMC_NE1, FMC_NOE, FMC_NWE -- but no .ucf in Caster assigns
any of it, so the gateware has never used that bus. R2 has no MCU-side parallel
bus at all. The labels and their stubs go and the freed bank-1 pins get
no-connect flags.

A CROSS-SHEET SHORT, CAUGHT ONLY BY THE PIN-MAP CHECK
The first run reported 7 mismatches: U41.D14 on VCOM_MEA_EN, J14 on SHDN, and
five more. Adding 57 sheet pins grew fpga_io's box on the root to y 68.6-221.0
and epd_power was sitting at y 106.7-132.1 in the same column, so their sheet
pins overlapped and the nets shorted. This is the hazard docs/epd-port.md §8
records; tools/layout_root.py moved epd_power to y 233.68 and the check now
asserts no two sheet boxes on the root overlap.

Worth recording because it is the argument for the check: ERC did not catch
this, and neither did anything else. Only comparing every ball against R1 did.
tools/check_ucf.py should exist before fpga_ddr, where one swapped MCB3 pin is
fatal and invisible.

R1 LEAVES 12 OF ITS 24 SPARE BALLS UNFLAGGED
Those arrived as pin_not_connected. docs/mcu.md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
Parts:
- added D308: LED GREEN, LED_SMD:LED_0603_1608Metric, symbol Device:LED
- added R311: 10K/1%, Resistor_SMD:R_0402_1005Metric, symbol Device:R
- added U41: XC6SLX-FTG256, footprints:Xilinx_FTG256, symbol symbols:XC6SLX-FTG256
Connections:
- new net: D308.2 (A), R311.2
- new net +3V3: U41.B13 (VCCO_0), U41.B4 (VCCO_0), U41.B9 (VCCO_0), U41.D10 (VCCO_0), U41.D15 (VCCO_1), U41.D7 (VCCO_0), U41.G13 (VCCO_1), U41.J15 (VCCO_1), U41.K13 (VCCO_1), U41.N15 (VCCO_1), U41.R13 (VCCO_1)
- new net DPI_B2: U41.T14 (IO_L51P_M1DQ12_1)
- new net DPI_B3: U41.R14 (IO_L50P_M1UDQS_1)
- new net DPI_B4: U41.N14 (IO_L45P_A1_M1LDQS_1)
- new net DPI_B5: U41.P15 (IO_L48P_HDC_M1DQ8_1)
- new net DPI_B6: U41.M13 (IO_L74P_AWAKE_1)
- new net DPI_B7: U41.M14 (IO_L74N_DOUT_BUSY_1)
- new net DPI_DE: U41.T13 (IO_L51N_M1DQ13_1)
- new net DPI_G2: U41.L12 (IO_L53P_1)
- new net DPI_G3: U41.L13 (IO_L53N_VREF_1)
- new net DPI_G4: U41.L14 (IO_L47P_FWE_B_M1DQ0_1)
- new net DPI_G5: U41.K12 (IO_L42P_GCLK7_M1UDM_1)
- new net DPI_G6: U41.K14 (IO_L41N_GCLK8_M1CASN_1)
- new net DPI_G7: U41.J12 (IO_L40N_GCLK10_M1A6_1)
- new net DPI_HS: U41.R12 (IO_L52P_M1DQ14_1)
- new net DPI_PCLK: U41.J13 (IO_L41P_GCLK9_IRDY1_M1RASN_1)
- new net DPI_R2: U41.J14 (IO_L43P_GCLK5_M1DQ4_1)
- new net DPI_R3: U41.H14 (IO_L39N_M1ODT_1)
- new net DPI_R4: U41.H13 (IO_L39P_M1A3_1)
- new net DPI_R5: U41.G12 (IO_L38P_A5_M1CLK_1)
- new net DPI_R6: U41.G14 (IO_L36P_A9_M1BA0_1)
- new net DPI_R7: U41.D14 (IO_L31P_A19_M1CKE_1)
- new net DPI_VS: U41.T12 (IO_L52N_M1DQ15_1)
- new net EPDC_CLKN: U41.D8 (IO_L38P_0)
- new net EPDC_CLKP: U41.C8 (IO_L38N_VREF_0)
- new net EPDC_D0N: U41.C10 (IO_L37N_GCLK12_0)
- new net EPDC_D0P: U41.E10 (IO_L37P_GCLK13_0)
- new net EPDC_D10N: U41.B8 (IO_L33P_0)
- new net EPDC_D10P: U41.A8 (IO_L33N_0)
- new net EPDC_D11N: U41.C9 (IO_L34P_GCLK19_0)
- new net EPDC_D11P: U41.A9 (IO_L34N_GCLK18_0)
- new net EPDC_D1N: U41.B10 (IO_L35P_GCLK17_0)
- new net EPDC_D1P: U41.A10 (IO_L35N_GCLK16_0)
- new net EPDC_D2N: U41.E11 (IO_L64N_SCP4_0)
- new net EPDC_D2P: U41.F10 (IO_L64P_SCP5_0)
- new net EPDC_D3N: U41.D12 (IO_L66N_SCP0_0)
- new net EPDC_D3P: U41.D11 (IO_L66P_SCP1_0)
- new net EPDC_D4N: U41.C11 (IO_L39P_0)
- new net EPDC_D4P: U41.A11 (IO_L39N_0)
- new net EPDC_D5N: U41.B12 (IO_L62P_0)
- new net EPDC_D5P: U41.A12 (IO_L62N_VREF_0)
- new net EPDC_D6N: U41.C13 (IO_L63P_SCP7_0)
- new net EPDC_D6P: U41.A13 (IO_L63N_SCP6_0)
- new net EPDC_D7N: U41.B14 (IO_L65P_SCP3_0)
- new net EPDC_D7P: U41.A14 (IO_L65N_SCP2_0)
- new net EPDC_D8N: U41.A7 (IO_L6N_0)
- new net EPDC_D8P: U41.C7 (IO_L6P_0)
- new net EPDC_D9N: U41.E8 (IO_L36N_GCLK14_0)
- new net EPDC_D9P: U41.E7 (IO_L36P_GCLK15_0)
- new net EPDC_GDCLK: U41.B16 (IO_L29N_A22_M1A14_1)
- new net EPDC_GDOE: U41.D16 (IO_L31N_A18_M1A12_1)
- new net EPDC_GDSP: U41.C16 (IO_L33N_A14_M1A4_1)
- new net EPDC_SDCE0: U41.E15 (IO_L34P_A13_M1WE_1)
- new net EPDC_SDLE: U41.E16 (IO_L34N_A12_M1BA2_1)
- new net EPDC_SDOE: U41.F15 (IO_L35P_A11_M1A7_1)
- new net EPDC_SE_CLK: U41.B15 (IO_L29P_A23_M1A13_1)
- new net EPD_THROT: U41.M16 (IO_L46N_FOE_B_M1DQ3_1)
- new net FPGA_CLK33: U41.K11 (IO_L42N_GCLK6_TRDY1_M1LDM_1)
- new net GND: D308.1 (K)
- new net LED: R311.1, U41.C15 (IO_L33P_A15_M1A10_1)
- no-connect marks 0 -> 36
Other:
- company: (none) -> Copyright 2025 Modos Tech Inc

Commit message: R2: WP5 review answer 2 -- J3 is deleted, and with it ten dead nets
Owner's decision, manual-analysis/Analysis_fpga.md: "Yes, delete J3 connector."

J3 was the 16-pin panel connector. It carried nothing but EPDC_D8-D11 (eight
nets), EPDC_CLKP/CLKN and six grounds, and check_ucf.py had already shown that
no LOC line in Caster's constraint.ucf assigns any of the ten -- EPD_SD is 16
bits in every build variant and the UCF maps those 16 to panel pairs D0-D7, and
there is no EPD_CLK port in top.v at all. So this is not an unpopulated option;
nothing in the gateware could drive it.

Why it existed upstream, which the owner also asked: Glider is a general-purpose
EPD monitor. README "Screen Adapters" -- "A single 50pin connector is enough for
8/16-bit screens, the 16 pin connector additionally adds support for LVDS
screens and 32-bit/64-bit screens." In the screen list every MiniLVDS panel is
8" 1920x1440 or larger; every 6" 1448x1072 panel is TTL on 34 pins. R2 is a 6"
reader, so J3 is the large-panel option and J6 alone is the reader's connector.

tools/patch_drop_j3.py does it surgically -- both sheets are frozen. On epd:
J3, #PWR0201, ten hierarchical labels, ten signal wires, the thirteen-wire
ground comb and its six junctions. On fpga_io: ten labels and wires, and ten
no-connect flags on C7 A7 B8 A8 C9 A9 E7 E8 D8 C8. port_r1.py keeps the ten
names in HIER so a --force re-port still reproduces R1, and subtracts a new
DEAD_ON_R2 set from the sheet-pin list instead.

Verified: netlist before/after is 351 nets either way -- exactly the ten dead
nets gone, exactly seven J3 nodes off GND, ten new one-pin unconnected- nets on
the expected balls, and every other net byte-identical. check_ucf.py still 113
constrained balls / 0 failures, and its "reserved but not driven" list falls
from 11 balls to 1 (EPD_THROT). ERC unchanged at 105 excluding library links.
Both pages and the root rendered and read.

The r2.kicad_sch diff is large because removing ten sheet pins moves every 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
Connections:
- net EPDC_CLKN: no longer names the net of U41.D8 (IO_L38P_0)
- net EPDC_CLKP: no longer names the net of U41.C8 (IO_L38N_VREF_0)
- net EPDC_D10N: no longer names the net of U41.B8 (IO_L33P_0)
- net EPDC_D10P: no longer names the net of U41.A8 (IO_L33N_0)
- net EPDC_D11N: no longer names the net of U41.C9 (IO_L34P_GCLK19_0)
- net EPDC_D11P: no longer names the net of U41.A9 (IO_L34N_GCLK18_0)
- net EPDC_D8N: no longer names the net of U41.A7 (IO_L6N_0)
- net EPDC_D8P: no longer names the net of U41.C7 (IO_L6P_0)
- net EPDC_D9N: no longer names the net of U41.E8 (IO_L36N_GCLK14_0)
- net EPDC_D9P: no longer names the net of U41.E7 (IO_L36P_GCLK15_0)
- no-connect marks 36 -> 46
Changed lines of the file:
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@@
-	(wire
-		(pts
-			(xy 218.44 76.2) (xy 213.36 76.2)
-		)
-		(stroke
-			(width 0)
-			(type default)
-		)
-	)
 	(wire
 		(pts
@@
 	(wire
 		(pts
-			(xy 218.44 111.76) (xy 213.36 111.76)
-		)
-		(stroke
-			(width 0)
-			(type default)
-		)
-	)
-	(wire
-		(pts
 			(xy 119.38 175.26) (xy 114.3 175.26)
 		)
@@
 	(wire
 		(pts
-			(xy 218.44 86.36) (xy 213.36 86.36)
-		)
-		(stroke
-			(width 0)
-			(type default)
-		)
-	)
-	(wire
-		(pts
 			(xy 119.38 78.74) (xy 114.3 78.74)
 		)
@@
 	(wire
 		(pts
-			(xy 218.44 73.66) (xy 213.36 73.66)
-		)
-		(stroke
-			(width 0)
-			(type default)
-		)
-	)
-	(wire
-		(pts
 			(xy 218.44 93.98) (xy 213.36 93.98)
 		)
@@
 	(wire
 		(pts
-			(xy 218.44 99.06) (xy 213.36 99.06)
-		)
-		(stroke
-			(width 0)
-			(type default)
-		)
-	)
-	(wire
-		(pts
 			(xy 119.38 147.32) (xy 114.3 147.32)
 		)
@@
 	(wire
 		(pts
-			(xy 218.44 91.44) (xy 213.36 91.44)
-		)
-		(stroke
-			(width 0)
-			(type default)
-		)
-	)
-	(wire
-		(pts
 			(xy 218.44 137.16) (xy 213.36 137.16)
 		)
@@
 	(wire
 		(pts
-			(xy 218.44 83.82) (xy 213.36 83.82)
-		)
-		(stroke
-			(width 0)
-			(type default)
-		)
-	)
-	(wire
-		(pts
 			(xy 218.44 142.24) (xy 213.36 142.24)
 		)
@@
 	(wire
 		(pts
-			(xy 218.44 109.22) (xy 213.36 109.22)
-		)
-		(stroke
-			(width 0)
-			(type default)
-		)
-	)
-	(wire
-		(pts
 			(xy 101.6 25.4) (xy 104.14 25.4)
 		)
@@
 	(wire
 		(pts
-			(xy 218.44 101.6) (xy 213.36 101.6)
-		)
-		(stroke
-			(width 0)
-			(type default)
-		)
-	)
-	(wire
-		(pts
 			(xy 119.38 101.6) (xy 114.3 101.6)
 		)
@@
 		(pts
 			(xy 119.38 142.24) (xy 114.3 142.24)
-		)
-		(stroke
-			(width 0)
-			(type default)
-		)
-	)
-	(wire
-		(pts
-			(xy 218.44 88.9) (xy 213.36 88.9)
 		)
 		(stroke
@@
 		)
 	)
-	(hierarchical_label "EPDC_D11P"
-		(shape output)
-		(at 218.44 91.44 0)
-		(effects
-			(font
-				(size 1.27 1.27)
-			)
-			(justify left)
-		)
-	)
 	(hierarchical_label "DPI_HS"
 		(shape input)
@@
 		)
 	)
-	(hierarchical_label "EPDC_D10P"
-		(shape output)
-		(at 218.44 86.36 0)
-		(effects
-			(font
-				(size 1.27 1.27)
-			)
-			(justify left)
-		)
-	)
 	(hierarchical_label "DPI_G3"
 		(shape input)
@@
 		)
 	)
-	(hierarchical_label "EPDC_D9N"
-		(shape output)
-		(at 218.44 101.6 0)
-		(effects
-			(font
-				(size 1.27 1.27)
-			)
-			(justify left)
-		)
-	)
 	(hierarchical_label "FPGA_CLK33"
 		(shape input)
@@
 		)
 	)
-	(hierarchical_label "EPDC_D10N"
-		(shape output)
-		(at 218.44 83.82 0)
-		(effects
-			(font
-				(size 1.27 1.27)
-			)
-			(justify left)
-		)
-	)
 	(hierarchical_label "DPI_PCLK"
 		(shape input)
@@
 		)
 	)
-	(hierarchical_label "EPDC_D9P"
-		(shape output)
-		(at 218.44 99.06 0)
-		(effects
-			(font
-				(size 1.27 1.27)
-			)
-			(justify left)
-		)
-	)
 	(hierarchical_label "EPDC_D6N"
 		(shape output)
@@
 		)
 	)
-	(hierarchical_label "EPDC_D8N"
-		(shape output)
-		(at 218.44 76.2 0)
-		(effects
-			(font
-				(size 1.27 1.27)
-			)
-			(justify left)
-		)
-	)
 	(hierarchical_label "DPI_B7"
 		(shape input)
@@
 		)
 	)
-	(hierarchical_label "EPDC_CLKN"
-		(shape output)
-		(at 218.44 109.22 0)
-		(effects
-			(font
-				(size 1.27 1.27)
-			)
-			(justify left)
-		)
-	)
 	(hierarchical_label "DPI_G7"
 		(shape input)
@@
 		)
 	)
-	(hierarchical_label "EPDC_D11N"
-		(shape output)
-		(at 218.44 88.9 0)
-		(effects
-			(font
-				(size 1.27 1.27)
-			)
-			(justify left)
-		)
-	)
 	(hierarchical_label "DPI_R5"
 		(shape input)
@@
 		)
 	)
-	(hierarchical_label "EPDC_D8P"
-		(shape output)
-		(at 218.44 73.66 0)
-		(effects
-			(font
-				(size 1.27 1.27)
-			)
-			(justify left)
-		)
-	)
 	(hierarchical_label "EPD_THROT"
 		(shape input)
@@
 		(shape input)
 		(at 119.38 101.6 0)
-		(effects
-			(font
-				(size 1.27 1.27)
-			)
-			(justify left)
-		)
-	)
-	(hierarchical_label "EPDC_CLKP"
-		(shape output)
-		(at 218.44 111.76 0)
 		(effects
 			(font
@@
 		)
 	)
+	(no_connect
+		(at 213.36 73.66)
+	)
+	(no_connect
+		(at 213.36 76.2)
+	)
+	(no_connect
+		(at 213.36 83.82)
+	)
+	(no_connect
+		(at 213.36 86.36)
+	)
+	(no_connect
+		(at 213.36 88.9)
+	)
+	(no_connect
+		(at 213.36 91.44)
+	)
+	(no_connect
+		(at 213.36 99.06)
+	)
+	(no_connect
+		(at 213.36 101.6)
+	)
+	(no_connect
+		(at 213.36 109.22)
+	)
+	(no_connect
+		(at 213.36 111.76)
+	)
 )

Commit message: R2: MPNs into the schematic -- and five caps carry the wrong part number
Sourcing data lived in docs/*.md, not in the schematic, so the BOM the
fab would read had 3 of 96 lines with an MPN. Resolved every LCSC code
already on the board against LCSC's own catalogue and wrote MPN +
Manufacturer back: 53 -> 60 lines, 218 components. Added LCSC codes for
L10-L13, U42 and J22/J23 from the per-sheet docs.

Verified before writing: 321 refs and 519 nets identical before and
after, no duplicated properties, pre-existing MPNs untouched.

Cross-checking each passive value against the part its LCSC code
actually names found five wrong ones, all of them the ADC sense-divider
filter caps on power_mon:

  C91                 1nF/50V  carries C131394  = 100 nF
  C163 C164 C168 C169 1nF/25V  carries C6119801 = 470 nF

Left unwritten rather than cementing the error. C1523 (0402B102K500NT,
1 nF 50 V X7R 0402, JLC Basic, 5.3 M stock) covers both positions.

Also held back: U41, whose C39313 is XC6SLX16-**2**FTG256C while
fpga.md specifies the -3 speed grade.

frontlight.md cites C1848394 as the FPC connector on J22/J23; that code
is TPS22914BYFPR. The 6-pin sibling of J24's C5213749 is C5213748.

Co-Authored-By: Claude Opus 5 <noreply@anthropic.com>
Claude-Session: https://claude.ai/code/session_01MnesETWABbVdbcVnCKfKVs
Parts:
- D308: MPN (none) -> XL-1608UGC-04; Manufacturer (none) -> XINGLIGHT
- R311: MPN (none) -> 0402WGF1002TCE; Manufacturer (none) -> UNI-ROYAL
Changed lines of the file:
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@@
+			)
+		)
+		(property "Manufacturer" "XINGLIGHT" (at 0 0 0)
+			(effects
+				(font
+					(size 1.27 1.27)
+				)
+				(hide yes)
+			)
+		)
+		(property "MPN" "XL-1608UGC-04" (at 0 0 0)
+			(effects
+				(font
+					(size 1.27 1.27)
+				)
+				(hide yes)
 			)
 		)
@@
 			)
 		)
+		(property "Manufacturer" "UNI-ROYAL" (at 0 0 0)
+			(effects
+				(font
+					(size 1.27 1.27)
+				)
+				(hide yes)
+			)
+		)
+		(property "MPN" "0402WGF1002TCE" (at 0 0 0)
+			(effects
+				(font
+					(size 1.27 1.27)
+				)
+				(hide yes)
+			)
+		)
