File: pcb/r2-mainboard/fpga_io.kicad_sch (KiCad schematic)
At the start: 3 parts, among them U41 XC6SLX-FTG256

Commit message: R2: the six approved edits, and one of them was already done
Owner-approved 2026-08-19, KiCad closed for the pass.

1. R225 22k -> 20.5K/1%, LCSC C57105 (0402WGF2052TCE, UNI-ROYAL, the
   family the rest of the board already uses). Rendered and checked:
   R224 390k over R225 20.5k with R213 100k injecting VGH_DAC, so
   20.5||100 = 17.01k and VGH = 1.2 x (1 + 390/17.01) = 28.71 V at
   DAC = 0 -- exactly epd-port.md 10.3's target.
2. The five sense-divider caps that carried codes for the wrong
   capacitance -> C1523 (0402B102K500NT, 1 nF 50 V X7R, JLC Basic,
   5.3 M stock). One part covers both the 25 V and 50 V positions.
2b. R88/R224 -> C54920667 (HRC0402F3903DNTO, 390k 1%, 20 k stock).
   C25782 had 14 units against two per board. The owner found this one;
   both obvious alternatives were traps -- C23150 is 0603, and C44937
   is 3.9 ohm despite "390K" in its part number.
3. C147 set DNP rather than deleted. panel.md 7 had already ruled that
   J6.7/J6.44 stay; that covered the pins but not the capacitor on the
   dead net. DNP drops it from placement, keeps the topology of a frozen
   sheet untouched, and leaves the footprint if a future panel drives
   the rail. in_bom stays yes -- that is this board's convention for all
   13 DNP parts, so they show up flagged rather than vanishing.
4. Ten duplicate #PWR references renumbered to #PWR1112-1121 on the
   battery sheet, which was the colliding side in every case.
5. J3 was already deleted on 2026-08-15. No work needed.
6. Specter -> Reflow across 22 files: 14 sheets, 7 generators, the
   project file. .history/ deliberately untouched.

Verified as one change: netlist before and after has 518 nets with
identical pin membership, and epd_power and epd were rendered to PNG and
inspected.

Docs updated to match: epd-port.md 10 is applied rather than designed,
frontlight.md 1 loses the "9 in series is inferred" hedge (the vendor
listing confirms 2 x 9), and io-expansion.md 4's "only guess on this
sheet" is resolved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
Other:
- title: Glider-R2 / Specter mainboard -> Glider-R2 / Reflow mainboard
Changed lines of the file:
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@@
 	(paper "A4")
 	(title_block
-		(title "Glider-R2 / Specter mainboard")
+		(title "Glider-R2 / Reflow mainboard")
 		(date "2026-08-07")
 		(rev "A")

Commit message: R2: two interrupts that could never fire, and the SoM footprint
The EXTI collisions mcu.md §3.4 found are applied. An EXTI line is picked
by the pin's *number*, so TOUCH_INT# on PC3 was fighting PD3 GAUGE_ALRT#
and PEN_INT# on PC6 was fighting PD6 QON_SNS -- as drawn neither touch nor
pen could raise an interrupt at all. Each swaps with an output, which needs
no line, so it costs nothing. FL_INT# gets PB12 at the same time, which was
frontlight.md §10.3's own first suggestion; §9's later push for PB7 was
wrong, because PC7 KEY_PREV# holds EXTI7.

518 -> 517 nets, the drop being the PB12 unconnected- pseudo-net, and
exactly five membership changes. Every hierarchical label in the project
now has a counterpart -- DANGLING_OK is empty and ERC excluding
footprint_link_issues is 32, down from 105.

The PCM-071 footprint is built rather than downloaded, because two drawings
have landed that over-determine it: Samtec's own vector land pattern (parsed
from the content stream, every measurement agreeing with a printed dimension
to under 1 um) and L-1038e.A5 Figure 7, which is a carrier-board drawing.
The trap it contains is that the alignment hole is NOT on the connector's
centreline -- it is 1.054 mm from one row and 5.118 from the other, and
Figure 7 dimensions the holes, so assuming a centred hole puts both
connectors 2.06 mm out. The check worth trusting is the one nothing forces:
the B and C rows land 0.982 and 0.998 mm inside the module's edges.

Also: U41's speed grade is settled -2 -- LCSC has no -3 in FTG256 at all,
and caster.xise's -3 is ISE's untouched default (valueState="default"), not
a choice anyone made. But -2's MCB is rated 667 Mb/s against the 666.67 this
design runs, so fpga.md §1.1 asks for one free ISE build before the order.

And a bring-up landmine: epd_pos_rails_good() accepts VGH <= 28.0 V while
R2's own R225 change puts it at 28.41 V nominal. A correctly built board
would fatal() at every EPD power-up. epd-port.md §10.5.

Co-Authored-By: Claude Op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
Parts:
- U41: MPN (none) -> XC6SLX16-2FTG256C; Manufacturer (none) -> AMD/XILINX
Changed lines of the file:
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@@
+			)
+		)
+		(property "MPN" "XC6SLX16-2FTG256C"
+			(at 91.44 109.22 0)
+			(hide yes)
+			(show_name no)
+			(do_not_autoplace no)
+			(effects
+				(font
+					(size 1.27 1.27)
+				)
+			)
+		)
+		(property "Manufacturer" "AMD/XILINX"
+			(at 91.44 111.76 0)
+			(hide yes)
+			(show_name no)
+			(do_not_autoplace no)
+			(effects
+				(font
+					(size 1.27 1.27)
+				)
 			)
 		)

Commit message: R2: renumber every sheet to the page-based designator scheme
The owner's scheme is classifier + sheet page + two-digit part from 00. Four
sheets already used it; this converts the remaining nine, so all thirteen now
agree: pages 2-9 take three digits, pages 10-14 four. 292 of 333 designators
changed. A part shared by several sheets takes its lowest page, so the FPGA is
U700 (pages 7-9) and the two SoM connectors are J501/J502 (pages 5-6).

The whole risk here is silently rewiring the board, so the netlist was diffed
rather than eyeballed:

  nets 519 -> 519, total pin connections 1563 -> 1563
  named nets present in both whose pin multiset changed: 0
  ERC unchanged at 14 errors / 20 warnings
  check_ucf.py: 99 balls matched, 0 failures

That last one matters most: it resolves the gateware's 113 UCF constraints to
board nets *by ball name*, so it is the sharpest detector of the corruption
this change could cause.

Two earlier attempts did cause exactly that. A bare quoted-string substitution
also rewrites FPGA ball names (C1, D2, N11, T1) and BTH-060 pin names (A1-D60),
which are spelled exactly like designators; one run left ERC identical while 40
nets came back with a different pin multiset. The tool now substitutes only at
the two positions that store an instance's designator, and excludes every pin
name everywhere else. docs/layout.md 9.5 records the hazard and how to prove a
renumber was clean.

Only the three scripts that read the design are updated. The gen_*/patch_*/
port_r1.py scripts keep the old names deliberately: each wrote a sheet once and
has not been re-runnable since it was hand-edited in Eeschema, so they are a
historical record -- and port_r1.py's dict keys are R1 designators that were
never renumbered at all.

Co-Authored-By: Claude Opus 5 <noreply@anthropic.com>
Claude-Session: https://claude.ai/code/session_01MHTAe6ZnhogTEgtyPcLhwG
Parts:
- renumbered D308 to D700, R311 to R700, U41 to U700
Changed lines of the file:
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@@
 		(dnp no)
 		(fields_autoplaced yes)
-		(property "Reference" "U41"
+		(property "Reference" "U700"
 			(at 69.85 106.6799 0)
 			(show_name no)
@@
 			(project "r2"
 				(path "/dee825bf-c2f1-415d-afdf-cf702072a6e8/42cafb44-c4a2-4885-8a35-a2a05165e7e7"
-					(reference "U41")
+					(reference "U700")
 					(unit 2)
 				)
@@
 		(dnp no)
 		(fields_autoplaced yes)
-		(property "Reference" "U41"
+		(property "Reference" "U700"
 			(at 179.07 91.4399 0)
 			(show_name no)
@@
 			(project "r2"
 				(path "/dee825bf-c2f1-415d-afdf-cf702072a6e8/42cafb44-c4a2-4885-8a35-a2a05165e7e7"
-					(reference "U41")
+					(reference "U700")
 					(unit 1)
 				)
@@
 		(in_pos_files yes)
 		(dnp no)
-		(property "Reference" "D308"
+		(property "Reference" "D700"
 			(at 203.2 160.02 0)
 			(show_name no)
@@
 			(project "r2"
 				(path "/dee825bf-c2f1-415d-afdf-cf702072a6e8/42cafb44-c4a2-4885-8a35-a2a05165e7e7"
-					(reference "D308")
+					(reference "D700")
 					(unit 1)
 				)
@@
 		(in_pos_files yes)
 		(dnp no)
-		(property "Reference" "R311"
+		(property "Reference" "R700"
 			(at 194.31 160.02 90)
 			(show_name no)
@@
 			(project "r2"
 				(path "/dee825bf-c2f1-415d-afdf-cf702072a6e8/42cafb44-c4a2-4885-8a35-a2a05165e7e7"
-					(reference "R311")
+					(reference "R700")
 					(unit 1)
 				)
