File: pcb/r2-mainboard/fpga_io.kicad_sch (KiCad schematic)
At the start: 3 parts, among them U700 XC6SLX-FTG256

Commit message: Schematics update for new chip.
Parts:
- R700: value 10K/1% -> 10k/1%
Changed lines of the file:
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@@
 			)
 		)
-		(property "Value" "10K/1%"
+		(property "Value" "10k/1%"
 			(at 194.31 165.1 90)
 			(show_name no)
