File: pcb/r2-mainboard/io_expansion.kicad_sch (KiCad schematic)
At the start: 0 parts

Commit message: R2: WP6b -- io_expansion drawn; Stage C capture is complete
Two FPC connectors, two gated rails, seven MCU pins, everything DNP.
NOTES-R2-plan.md constraint 3 wants touch and pen "addable without a respin";
this sheet is that provision, and it is honest about which half of the promise
is certain:

  certain  -- the seven MCU pins exist and are routed, and +3V3_TOUCH /
              +3V3_PEN exist. Those are what would otherwise force a
              whole-board respin.
  a guess  -- the FPC pad order, because neither the touch controller nor the
              digitizer is chosen and the panel is not either.

docs/io-expansion.md 5 puts that in front of the owner as the last open
decision in Stage C, with three ways to close it, rather than burying it.

PC4/PC5 are USART3_TX/RX at AF0 -- verified in stm32g0b1.pdf's
alternate-function table, both free, and the one allocation here that is not
interchangeable. The other five are ordinary GPIO. Touch adds no I2C pins: it
joins the existing always-on bus, and SCL_AON/SDA_AON now carry J22.3/J22.4
alongside the charger, gauge and three INA3221s. Two spares remain, and which
two was deliberate -- PA12 (USB-DP capable) and PB12 (ADC-capable) are the two
with a capability the rest lack.

Everything DNP is coherent, not lazy: with no connector fitted there is no
load, so a fitted load switch would be two parts powering nothing. It also
means these two TPS22914s consume none of the thin LCSC stock epd-port.md 7
flags, so that stays a two-part problem.

A FOURTH SILENT SHORT, and this time the tooling caught it before the netlist
did. The connectors' GND pins dropped from their own label column and ran
straight through the two anchors below -- putting SCL_AON, SDA_AON, PEN_TXD
and PEN_RXD on GND. The entire always-on I2C bus was shorted to ground and ERC
said nothing.

So schgen.Sheet.check_label_crossings() now runs inside render() for every
generator: no wire may pass *through* a label anchor it does not end at. Ending
at an a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
Parts:
- added C517, C518: 1uF/16V, Capacitor_SMD:C_0402_1005Metric, symbol Device:C
- added J22, J23: HC-FPC-05-09-6RLTAG, footprints:HC-FPC-05-09-6RLTAG, symbol Connector_Generic:Conn_01x06
- added U54, U55: TPS22914BYFPR, Package_BGA:WLP-4_0.83x0.83mm_P0.4mm, symbol Power_Management:AP22913CN4
Connections:
- new net +3V3: U54.A2 (IN), U55.A2 (IN)
- new net +3V3_PEN: C518.1, J23.1 (Pin_1), U55.A1 (OUT)
- new net +3V3_TOUCH: C517.1, J22.1 (Pin_1), U54.A1 (OUT)
- new net GND: C517.2, C518.2, J22.2 (Pin_2), J23.2 (Pin_2), J23.6 (Pin_6), U54.B1 (GND), U55.B1 (GND)
- new net MCU_EN_PEN: U55.B2 (ON)
- new net MCU_EN_TOUCH: U54.B2 (ON)
- new net PEN_INT#: J23.5 (Pin_5)
- new net PEN_RXD: J23.4 (Pin_4)
- new net PEN_TXD: J23.3 (Pin_3)
- new net SCL_AON: J22.3 (Pin_3)
- new net SDA_AON: J22.4 (Pin_4)
- new net TOUCH_INT#: J22.5 (Pin_5)
- new net TOUCH_RST#: J22.6 (Pin_6)
Other:
- note added: "*** EVERYTHING ON THIS SHEET IS DNP -- both connectors, both load"
- note added: "*** THE FPC PIN ORDER IS PROVISIONAL. Neither the touch controller nor"
- note added: "*** accept that this group alone may need a respin. io-expansion.md 5."
- note added: "*** consume none of the thin stock epd-port.md 7 flags."
- note added: "*** fitted switch would power nothing. It also means these two TPS22914s"
- note added: "*** is the one guess here. Confirm against the real parts before fab, or"
- note added: "*** switches, their capacitors. No connector fitted means no load, so a"
- note added: "*** the digitizer is chosen -- the panel is not either -- so the pad order"
- note added: "Certain, and what stops a whole-board respin: the seven MCU pins exist and"
- note added: "See docs/io-expansion.md. Plan constraint 3: the first board is compute +"
- note added: "are routed, and both gated rails exist. PC4/PC5 are USART3_TX/RX at AF0 --"
- note added: "display + power only, and these get pads so they can be added later."
- note added: "io_expansion -- touch and pen, provisioned but NOT FITTED."
- note added: "sits on the existing always-on bus with the charger, gauge and INA3221s."
- note added: "the one allocation that is not interchangeable. Touch adds no I2C pins; it"

Commit message: R2: MPNs into the schematic -- and five caps carry the wrong part number
Sourcing data lived in docs/*.md, not in the schematic, so the BOM the
fab would read had 3 of 96 lines with an MPN. Resolved every LCSC code
already on the board against LCSC's own catalogue and wrote MPN +
Manufacturer back: 53 -> 60 lines, 218 components. Added LCSC codes for
L10-L13, U42 and J22/J23 from the per-sheet docs.

Verified before writing: 321 refs and 519 nets identical before and
after, no duplicated properties, pre-existing MPNs untouched.

Cross-checking each passive value against the part its LCSC code
actually names found five wrong ones, all of them the ADC sense-divider
filter caps on power_mon:

  C91                 1nF/50V  carries C131394  = 100 nF
  C163 C164 C168 C169 1nF/25V  carries C6119801 = 470 nF

Left unwritten rather than cementing the error. C1523 (0402B102K500NT,
1 nF 50 V X7R 0402, JLC Basic, 5.3 M stock) covers both positions.

Also held back: U41, whose C39313 is XC6SLX16-**2**FTG256C while
fpga.md specifies the -3 speed grade.

frontlight.md cites C1848394 as the FPC connector on J22/J23; that code
is TPS22914BYFPR. The 6-pin sibling of J24's C5213749 is C5213748.

Co-Authored-By: Claude Opus 5 <noreply@anthropic.com>
Claude-Session: https://claude.ai/code/session_01MnesETWABbVdbcVnCKfKVs
Parts:
- J22, J23: LCSC (none) -> C5213748; MPN (none) -> HC-FPC-05-09-6RLTAG; Manufacturer (none) -> HCTL
- U54, U55: MPN (none) -> TPS22914BYFPR; Manufacturer (none) -> TI
Changed lines of the file:
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@@
+			)
+		)
+		(property "Manufacturer" "TI" (at 0 0 0)
+			(effects
+				(font
+					(size 1.27 1.27)
+				)
+				(hide yes)
+			)
+		)
+		(property "MPN" "TPS22914BYFPR" (at 0 0 0)
+			(effects
+				(font
+					(size 1.27 1.27)
+				)
+				(hide yes)
 			)
 		)
@@
 			)
 		)
+		(property "Manufacturer" "HCTL" (at 0 0 0)
+			(effects
+				(font
+					(size 1.27 1.27)
+				)
+				(hide yes)
+			)
+		)
+		(property "LCSC" "C5213748" (at 0 0 0)
+			(effects
+				(font
+					(size 1.27 1.27)
+				)
+				(hide yes)
+			)
+		)
+		(property "MPN" "HC-FPC-05-09-6RLTAG" (at 0 0 0)
+			(effects
+				(font
+					(size 1.27 1.27)
+				)
+				(hide yes)
+			)
+		)
 		(pin "5"
 		)
@@
 			)
 		)
+		(property "Manufacturer" "HCTL" (at 0 0 0)
+			(effects
+				(font
+					(size 1.27 1.27)
+				)
+				(hide yes)
+			)
+		)
+		(property "LCSC" "C5213748" (at 0 0 0)
+			(effects
+				(font
+					(size 1.27 1.27)
+				)
+				(hide yes)
+			)
+		)
+		(property "MPN" "HC-FPC-05-09-6RLTAG" (at 0 0 0)
+			(effects
+				(font
+					(size 1.27 1.27)
+				)
+				(hide yes)
+			)
+		)
 		(pin "4"
 		)
@@
 			)
 		)
+		(property "Manufacturer" "TI" (at 0 0 0)
+			(effects
+				(font
+					(size 1.27 1.27)
+				)
+				(hide yes)
+			)
+		)
+		(property "MPN" "TPS22914BYFPR" (at 0 0 0)
+			(effects
+				(font
+					(size 1.27 1.27)
+				)
+				(hide yes)
+			)
+		)
