File: pcb/r2-mainboard/io_expansion.kicad_sch (KiCad schematic)
At the start: 6 parts, among them J22 HC-FPC-05-09-6RLTAG, J23 HC-FPC-05-09-6RLTAG, U54 TPS22914BYFPR, U55 TPS22914BYFPR

Commit message: R2: the six approved edits, and one of them was already done
Owner-approved 2026-08-19, KiCad closed for the pass.

1. R225 22k -> 20.5K/1%, LCSC C57105 (0402WGF2052TCE, UNI-ROYAL, the
   family the rest of the board already uses). Rendered and checked:
   R224 390k over R225 20.5k with R213 100k injecting VGH_DAC, so
   20.5||100 = 17.01k and VGH = 1.2 x (1 + 390/17.01) = 28.71 V at
   DAC = 0 -- exactly epd-port.md 10.3's target.
2. The five sense-divider caps that carried codes for the wrong
   capacitance -> C1523 (0402B102K500NT, 1 nF 50 V X7R, JLC Basic,
   5.3 M stock). One part covers both the 25 V and 50 V positions.
2b. R88/R224 -> C54920667 (HRC0402F3903DNTO, 390k 1%, 20 k stock).
   C25782 had 14 units against two per board. The owner found this one;
   both obvious alternatives were traps -- C23150 is 0603, and C44937
   is 3.9 ohm despite "390K" in its part number.
3. C147 set DNP rather than deleted. panel.md 7 had already ruled that
   J6.7/J6.44 stay; that covered the pins but not the capacitor on the
   dead net. DNP drops it from placement, keeps the topology of a frozen
   sheet untouched, and leaves the footprint if a future panel drives
   the rail. in_bom stays yes -- that is this board's convention for all
   13 DNP parts, so they show up flagged rather than vanishing.
4. Ten duplicate #PWR references renumbered to #PWR1112-1121 on the
   battery sheet, which was the colliding side in every case.
5. J3 was already deleted on 2026-08-15. No work needed.
6. Specter -> Reflow across 22 files: 14 sheets, 7 generators, the
   project file. .history/ deliberately untouched.

Verified as one change: netlist before and after has 518 nets with
identical pin membership, and epd_power and epd were rendered to PNG and
inspected.

Docs updated to match: epd-port.md 10 is applied rather than designed,
frontlight.md 1 loses the "9 in series is inferred" hedge (the vendor
listing confirms 2 x 9), and io-expansion.md 4's "only guess on this
sheet" is resolved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
Other:
- title: Glider-R2 / Specter mainboard -> Glider-R2 / Reflow mainboard
Changed lines of the file:
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@@
 	(paper "A3")
 	(title_block
-		(title "Glider-R2 / Specter mainboard")
+		(title "Glider-R2 / Reflow mainboard")
 		(date "2026-08-15")
 		(rev "A")
