File: pcb/r2-mainboard/power.kicad_sch (KiCad schematic)
At the start: 39 parts, among them U10 TPS7A0233DBVR, U12 TPS61022RWUR, U13 TPS63802DLAR, U14 TPS62A02DRLR, U15 TPS62A02DRLR

Commit message: R2: WP5 groundwork -- Xilinx/Micron datasheets, LX16 fix, DDR bank to 1.5 V
Steps 1-3 of the WP5 plan. No FPGA sheet is drawn yet; this is the evidence base
and the one power change that had to land before fpga_ddr can be.

DATASHEETS
AMD's documentation portal no longer serves PDFs at any of the old xilinx.com
paths -- every URL returns the same 2.5 KB JavaScript shell -- so these came from
the Wayback Machine: ds162 (DC & Switching), ug380 (Configuration), ug381
(SelectIO), ug393 (PCB Design). The hardware owner supplied mt41k64m16 from
DigiKey after micron.com proved unreachable. UG385 Packaging was deliberately
skipped at 15.8 MB, since pcb_common's XC6SLX-FTG256 symbol already encodes bank
membership in its pin names.

THE FPGA IS AN LX16, NOT AN LX9
NOTES-R2-plan.md's architecture diagram said XC6SLX9 and
NOTES-R2-hardware-facts.md carried a BOM row for XC6SLX9-2FTG256C at $6.10 --
stock and price for the wrong device. The gateware targets xc6slx16-ftg256-3 in
four places (caster.xise Device/Package/Speed Grade, par/ise_flow.sh,
par/ise_run.txt, mig.prj TargetFPGA) and R1's own schematic says
XC6SLX16-FTG256. An LX9 is not a drop-in: the MIG's C3_SMALL_DEVICE parameter
exists specifically for xc6slx9 packages, so it would need the memory controller
regenerated. LCSC stock and price for the LX16 are marked for re-query rather
than guessed.

DDR BANK 1.35 V -> 1.5 V
Caster's UCF constrains all 48 DDR pins as SSTL15_II / DIFF_SSTL15_II /
LVCMOS15, and ds162.pdf Table 7 specifies SSTL15_II only over VCCO
1.425-1.575 V with VREF 0.69-0.81 V. The committed rail was 1.344 V -- 81 mV
below the VCCO minimum, with a half-rail VREF of 0.672 V below its minimum too.
Spartan-6 has no 1.35 V I/O standard to relabel the gateware to: SSTL135 appears
nowhere in ds162.pdf or ug381.pdf, and LVCMOS15 and the HSTL standards still
stop at 1.4 V. R1 runs the same way and works, but on a different layout, and
neither board can be tested from here.

mt41k64m16.pdf p.1 makes the fix fr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
Parts:
- R33: value 124k/1% -> 150k/1%
Connections:
- net +1V35_DCDC renamed +1V5_DCDC
- net PG_1V35 renamed PG_1V5
Other:
- note added: "+1V5_DCDC — DDR3L at 1.5 V and the FPGA's DDR bank VCCO"
- note removed: "+1V35_DCDC — DDR3L and the FPGA's DDR bank VCCO"
Changed lines of the file:
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@@
 		)
 	)
-	(text "+1V35_DCDC  —  DDR3L and the FPGA's DDR bank VCCO"
+	(text "+1V5_DCDC  —  DDR3L at 1.5 V and the FPGA's DDR bank VCCO"
 		(exclude_from_sim no)
 		(at 275.59 140.97 0)
@@
 		)
 	)
-	(label "PG_1V35"
+	(label "PG_1V5"
 		(at 370.84 191.77 0)
 		(effects
@@
 		)
 	)
-	(label "PG_1V35"
+	(label "PG_1V5"
 		(at 372.11 99.06 180)
 		(effects
@@
 		)
 	)
-	(hierarchical_label "PG_1V35"
+	(hierarchical_label "PG_1V5"
 		(shape output)
 		(at 379.73 99.06 0)
@@
 			)
 		)
-		(property "Value" "124k/1%"
+		(property "Value" "150k/1%"
 			(at 350.52 165.862 0)
 			(show_name no)
@@
 			)
 		)
-		(property "Value" "+1V35_DCDC"
+		(property "Value" "+1V5_DCDC"
 			(at 370.84 147.32 0)
 			(show_name no)
@@
 			)
 		)
-		(property "Value" "+1V35_DCDC"
+		(property "Value" "+1V5_DCDC"
 			(at 260.35 246.38 0)
 			(show_name no)

Commit message: R2: MPNs into the schematic -- and five caps carry the wrong part number
Sourcing data lived in docs/*.md, not in the schematic, so the BOM the
fab would read had 3 of 96 lines with an MPN. Resolved every LCSC code
already on the board against LCSC's own catalogue and wrote MPN +
Manufacturer back: 53 -> 60 lines, 218 components. Added LCSC codes for
L10-L13, U42 and J22/J23 from the per-sheet docs.

Verified before writing: 321 refs and 519 nets identical before and
after, no duplicated properties, pre-existing MPNs untouched.

Cross-checking each passive value against the part its LCSC code
actually names found five wrong ones, all of them the ADC sense-divider
filter caps on power_mon:

  C91                 1nF/50V  carries C131394  = 100 nF
  C163 C164 C168 C169 1nF/25V  carries C6119801 = 470 nF

Left unwritten rather than cementing the error. C1523 (0402B102K500NT,
1 nF 50 V X7R 0402, JLC Basic, 5.3 M stock) covers both positions.

Also held back: U41, whose C39313 is XC6SLX16-**2**FTG256C while
fpga.md specifies the -3 speed grade.

frontlight.md cites C1848394 as the FPC connector on J22/J23; that code
is TPS22914BYFPR. The 6-pin sibling of J24's C5213749 is C5213748.

Co-Authored-By: Claude Opus 5 <noreply@anthropic.com>
Claude-Session: https://claude.ai/code/session_01MnesETWABbVdbcVnCKfKVs
Parts:
- C22, C25, C26, C27, C30, C32, C34: MPN (none) -> CL21A226MPQNNNE; Manufacturer (none) -> Samsung Electro-Mechanics
- L10, L12, L13: LCSC (none) -> C3224227; MPN (none) -> DFE322512F-1R0M; Manufacturer (none) -> muRata
- L11: LCSC (none) -> C703140; MPN (none) -> DFE252012F-R47M; Manufacturer (none) -> muRata
- U10: MPN (none) -> TPS7A0233DBVR; Manufacturer (none) -> TI
- U12: MPN (none) -> TPS61022RWUR; Manufacturer (none) -> TI
- U13: MPN (none) -> TPS63802DLAR; Manufacturer (none) -> TI
- U14, U15: MPN (none) -> TPS62A02DRLR; Manufacturer (none) -> TI
