File: pcb/r2-mainboard/power.kicad_sch (KiCad schematic)
At the start: 39 parts, among them U10 TPS7A0233DBVR, U12 TPS61022RWUR, U13 TPS63802DLAR, U14 TPS62A02DRLR, U15 TPS62A02DRLR

Commit message: routing and board layout
Connections:
- net OSCIL_2: now reaches L11.2, U13.7 (L2)
- net OSCIL_1: now reaches L11.1, U13.9 (L1)
- net 1V5_SW: now reaches L13.1, U15.2 (SW)
- net 1V2_SW: now reaches L12.1, U14.2 (SW)
Other:
- moved on the sheet: L12, L13
Changed lines of the file:
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@@
 	(wire
 		(pts
-			(xy 342.9 156.21) (xy 370.84 156.21)
+			(xy 346.71 156.21) (xy 370.84 156.21)
 		)
 		(stroke
@@
 	(wire
 		(pts
-			(xy 330.2 156.21) (xy 335.28 156.21)
+			(xy 330.2 156.21) (xy 339.09 156.21)
 		)
 		(stroke
@@
 	(wire
 		(pts
-			(xy 218.44 156.21) (xy 223.52 156.21)
+			(xy 218.44 156.21) (xy 227.33 156.21)
 		)
 		(stroke
@@
 	(wire
 		(pts
-			(xy 231.14 156.21) (xy 259.08 156.21)
+			(xy 234.95 156.21) (xy 259.08 156.21)
 		)
 		(stroke
@@
 		)
 	)
+	(label "1V2_SW"
+		(at 219.71 156.21 0)
+		(effects
+			(font
+				(size 1.27 1.27)
+			)
+			(justify left bottom)
+		)
+	)
 	(label "MCU_EN_5V"
 		(at 372.11 68.58 180)
@@
 		)
 	)
+	(label "OSCIL_2"
+		(at 80.01 144.78 0)
+		(effects
+			(font
+				(size 1.27 1.27)
+			)
+			(justify left bottom)
+		)
+	)
 	(label "MCU_EN_3V3"
 		(at 46.99 161.29 180)
@@
 		)
 	)
+	(label "OSCIL_1"
+		(at 72.39 144.78 0)
+		(effects
+			(font
+				(size 1.27 1.27)
+			)
+			(justify left bottom)
+		)
+	)
 	(label "MCU_EN_FPGA_CORE"
 		(at 372.11 78.74 180)
@@
 		)
 	)
+	(label "1V5_SW"
+		(at 331.47 156.21 0)
+		(effects
+			(font
+				(size 1.27 1.27)
+			)
+			(justify left bottom)
+		)
+	)
 	(label "PG_3V3"
 		(at 372.11 88.9 180)
@@
 	(symbol
 		(lib_id "Device:L")
-		(at 227.33 156.21 90)
+		(at 231.14 156.21 90)
 		(unit 1)
 		(body_style 1)
@@
 		(dnp no)
 		(property "Reference" "L12"
-			(at 227.33 151.765 270)
+			(at 233.934 148.336 270)
 			(show_name no)
 			(do_not_autoplace no)
@@
 		)
 		(property "Value" "1uH/3.8A"
-			(at 227.584 153.67 270)
+			(at 234.188 150.241 270)
 			(show_name no)
 			(do_not_autoplace no)
@@
 		)
 		(property "Footprint" "Inductor_SMD:L_1210_3225Metric"
-			(at 227.33 156.21 270)
+			(at 231.14 156.21 270)
 			(hide yes)
 			(show_name no)
@@
 		)
 		(property "Datasheet" ""
-			(at 227.33 156.21 270)
+			(at 231.14 156.21 270)
 			(hide yes)
 			(show_name no)
@@
 		)
 		(property "Description" "1 µH power inductor, 1210 — Isat 4.8 A / Irms 3.8 A / 32 mΩ (Murata DFE322512F-1R0M, LCSC C3224227)"
-			(at 227.33 156.21 270)
+			(at 231.14 156.21 270)
 			(hide yes)
 			(show_name no)
@@
 		)
 		(property "Manufacturer" "muRata"
-			(at 0 0 0)
+			(at 3.81 0 0)
 			(hide yes)
 			(show_name no)
@@
 		)
 		(property "LCSC" "C3224227"
-			(at 0 0 0)
+			(at 3.81 0 0)
 			(hide yes)
 			(show_name no)
@@
 		)
 		(property "MPN" "DFE322512F-1R0M"
-			(at 0 0 0)
+			(at 3.81 0 0)
 			(hide yes)
 			(show_name no)
@@
 	(symbol
 		(lib_id "Device:L")
-		(at 339.09 156.21 90)
+		(at 342.9 156.21 90)
 		(unit 1)
 		(body_style 1)
@@
 		(dnp no)
 		(property "Reference" "L13"
-			(at 339.09 151.765 270)
+			(at 342.9 151.765 270)
 			(show_name no)
 			(do_not_autoplace no)
@@
 		)
 		(property "Value" "1uH/3.8A"
-			(at 339.344 153.924 270)
+			(at 343.154 153.924 270)
 			(show_name no)
 			(do_not_autoplace no)
@@
 		)
 		(property "Footprint" "Inductor_SMD:L_1210_3225Metric"
-			(at 339.09 156.21 270)
+			(at 342.9 156.21 270)
 			(hide yes)
 			(show_name no)
@@
 		)
 		(property "Datasheet" ""
-			(at 339.09 156.21 270)
+			(at 342.9 156.21 270)
 			(hide yes)
 			(show_name no)
@@
 		)
 		(property "Description" "1 µH power inductor, 1210 — Isat 4.8 A / Irms 3.8 A / 32 mΩ (Murata DFE322512F-1R0M, LCSC C3224227)"
-			(at 339.09 156.21 270)
+			(at 342.9 156.21 270)
 			(hide yes)
 			(show_name no)
@@
 		)
 		(property "Manufacturer" "muRata"
-			(at 0 0 0)
+			(at 3.81 0 0)
 			(hide yes)
 			(show_name no)
@@
 		)
 		(property "LCSC" "C3224227"
-			(at 0 0 0)
+			(at 3.81 0 0)
 			(hide yes)
 			(show_name no)
@@
 		)
 		(property "MPN" "DFE322512F-1R0M"
-			(at 0 0 0)
+			(at 3.81 0 0)
 			(hide yes)
 			(show_name no)
@@
 		)
 		(property "Value" "0.47uH/4.9A"
-			(at 76.2 140.97 270)
+			(at 76.2 133.35 270)
 			(show_name no)
 			(do_not_autoplace no)
