File: pcb/r2-mainboard/power.kicad_sch (KiCad schematic)
At the start: 39 parts, among them U10 TPS7A0233DBVR, U12 TPS61022RWUR, U13 TPS63802DLAR, U14 TPS62A02DRLR, U15 TPS62A02DRLR

Commit message: Docs: library audit list and a first production costing
libraries.md -- every symbol in r2.kicad_sym and every footprint in
r2.pretty, with what it was derived from, which tools/ script emits it,
and what was actually checked. Written for the owner's audit before the
libraries get rehomed. Notes that pcb_common has never been modified,
and calls out the three newest entries (TPS2553DBV and the two
_Mirrored FPC land patterns) as the least reviewed.

NOTES-production-costing.md -- what 1000 units costs and what a campaign
would have to raise, prompted by Good Display's US$750 / MOQ 1000 quote.
Central estimate EUR 340/unit COGS and a EUR ~548k goal, but the honest
finding is the sensitivity: the PCM-071 at EUR 250 @1-9 costs more than
the display, and the sibling quote says ~EUR 190 of that is a memory-
shortage surcharge. A 1000-piece quote moves the goal by EUR 290k, so it
is the single highest-value thing to chase. Also states plainly that at
the central estimate the margin is thin to negative against market
comparables, and what to do about it.

Both indexed in CLAUDE.md.

Co-Authored-By: Claude Opus 5 <noreply@anthropic.com>
Claude-Session: https://claude.ai/code/session_01MHTAe6ZnhogTEgtyPcLhwG
Parts:
- renumbered U10 to U300, U12 to U301, U13 to U302, U14 to U303, U15 to U304
Changed lines of the file:
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@@
 		(in_pos_files yes)
 		(dnp no)
-		(property "Reference" "U13"
+		(property "Reference" "U302"
 			(at 85.09 176.53 0)
 			(show_name no)
@@
 			(project "r2"
 				(path "/dee825bf-c2f1-415d-afdf-cf702072a6e8/3c7f0f04-b337-4425-b9f6-94d0a6934c0f"
-					(reference "U13")
+					(reference "U302")
 					(unit 1)
 				)
@@
 		(in_pos_files yes)
 		(dnp no)
-		(property "Reference" "U15"
+		(property "Reference" "U304"
 			(at 312.42 149.86 0)
 			(show_name no)
@@
 			(project "r2"
 				(path "/dee825bf-c2f1-415d-afdf-cf702072a6e8/3c7f0f04-b337-4425-b9f6-94d0a6934c0f"
-					(reference "U15")
+					(reference "U304")
 					(unit 1)
 				)
@@
 		(in_pos_files yes)
 		(dnp no)
-		(property "Reference" "U14"
+		(property "Reference" "U303"
 			(at 200.66 149.86 0)
 			(show_name no)
@@
 			(project "r2"
 				(path "/dee825bf-c2f1-415d-afdf-cf702072a6e8/3c7f0f04-b337-4425-b9f6-94d0a6934c0f"
-					(reference "U14")
+					(reference "U303")
 					(unit 1)
 				)
@@
 		(in_pos_files yes)
 		(dnp no)
-		(property "Reference" "U12"
+		(property "Reference" "U301"
 			(at 233.68 96.52 0)
 			(show_name no)
@@
 			(project "r2"
 				(path "/dee825bf-c2f1-415d-afdf-cf702072a6e8/3c7f0f04-b337-4425-b9f6-94d0a6934c0f"
-					(reference "U12")
+					(reference "U301")
 					(unit 1)
 				)
@@
 		(in_pos_files yes)
 		(dnp no)
-		(property "Reference" "U10"
+		(property "Reference" "U300"
 			(at 62.23 52.07 0)
 			(show_name no)
@@
 			(project "r2"
 				(path "/dee825bf-c2f1-415d-afdf-cf702072a6e8/3c7f0f04-b337-4425-b9f6-94d0a6934c0f"
-					(reference "U10")
+					(reference "U300")
 					(unit 1)
 				)

Commit message: R2: renumber every sheet to the page-based designator scheme
The owner's scheme is classifier + sheet page + two-digit part from 00. Four
sheets already used it; this converts the remaining nine, so all thirteen now
agree: pages 2-9 take three digits, pages 10-14 four. 292 of 333 designators
changed. A part shared by several sheets takes its lowest page, so the FPGA is
U700 (pages 7-9) and the two SoM connectors are J501/J502 (pages 5-6).

The whole risk here is silently rewiring the board, so the netlist was diffed
rather than eyeballed:

  nets 519 -> 519, total pin connections 1563 -> 1563
  named nets present in both whose pin multiset changed: 0
  ERC unchanged at 14 errors / 20 warnings
  check_ucf.py: 99 balls matched, 0 failures

That last one matters most: it resolves the gateware's 113 UCF constraints to
board nets *by ball name*, so it is the sharpest detector of the corruption
this change could cause.

Two earlier attempts did cause exactly that. A bare quoted-string substitution
also rewrites FPGA ball names (C1, D2, N11, T1) and BTH-060 pin names (A1-D60),
which are spelled exactly like designators; one run left ERC identical while 40
nets came back with a different pin multiset. The tool now substitutes only at
the two positions that store an instance's designator, and excludes every pin
name everywhere else. docs/layout.md 9.5 records the hazard and how to prove a
renumber was clean.

Only the three scripts that read the design are updated. The gen_*/patch_*/
port_r1.py scripts keep the old names deliberately: each wrote a sheet once and
has not been re-runnable since it was hand-edited in Eeschema, so they are a
historical record -- and port_r1.py's dict keys are R1 designators that were
never renumbered at all.

Co-Authored-By: Claude Opus 5 <noreply@anthropic.com>
Claude-Session: https://claude.ai/code/session_01MHTAe6ZnhogTEgtyPcLhwG
Parts:
- renumbered C20 to C300, C21 to C301, C22 to C302, C25 to C303, C26 to C304, C27 to C305, C28 to C306, C29 to C307, C30 to C308, C31 to C309, C32 to C310, C33 to C311, C34 to C312, L10 to L300, L11 to L301, L12 to L302, L13 to L303, R20 to R300, R21 to R301, R22 to R302, R23 to R303, R24 to R304, R25 to R305, R26 to R306, R27 to R307, R28 to R308, R29 to R309, R30 to R310, R31 to R311, R32 to R312, R33 to R313, R34 to R314, R35 to R315, R36 to R316
