File: pcb/r2-mainboard/power.kicad_sch (KiCad schematic)
At the start: 39 parts, among them U300 TPS7A0233DBVR, U301 TPS61022RWUR, U302 TPS63802DLAR, U303 TPS62A02DRLR, U304 TPS62A02DRLR

Commit message: routing
Parts:
- renumbered L300 to L301, L301 to L302, L302 to L303, L303 to L304
Changed lines of the file:
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@@
 		(in_pos_files yes)
 		(dnp no)
-		(property "Reference" "L300"
+		(property "Reference" "L301"
 			(at 241.3 43.815 270)
 			(show_name no)
@@
 			(project "r2"
 				(path "/dee825bf-c2f1-415d-afdf-cf702072a6e8/3c7f0f04-b337-4425-b9f6-94d0a6934c0f"
-					(reference "L300")
+					(reference "L301")
 					(unit 1)
 				)
@@
 		(in_pos_files yes)
 		(dnp no)
-		(property "Reference" "L302"
-			(at 233.934 148.336 270)
+		(property "Reference" "L303"
+			(at 233.934 148.336 90)
 			(show_name no)
 			(do_not_autoplace no)
@@
 			(project "r2"
 				(path "/dee825bf-c2f1-415d-afdf-cf702072a6e8/3c7f0f04-b337-4425-b9f6-94d0a6934c0f"
-					(reference "L302")
+					(reference "L303")
 					(unit 1)
 				)
@@
 		(in_pos_files yes)
 		(dnp no)
-		(property "Reference" "L303"
-			(at 342.9 151.765 270)
+		(property "Reference" "L304"
+			(at 342.9 151.765 90)
 			(show_name no)
 			(do_not_autoplace no)
@@
 			(project "r2"
 				(path "/dee825bf-c2f1-415d-afdf-cf702072a6e8/3c7f0f04-b337-4425-b9f6-94d0a6934c0f"
-					(reference "L303")
+					(reference "L304")
 					(unit 1)
 				)
@@
 		(in_pos_files yes)
 		(dnp no)
-		(property "Reference" "L301"
-			(at 76.2 131.445 270)
+		(property "Reference" "L302"
+			(at 76.2 131.445 90)
 			(show_name no)
 			(do_not_autoplace no)
@@
 			(project "r2"
 				(path "/dee825bf-c2f1-415d-afdf-cf702072a6e8/3c7f0f04-b337-4425-b9f6-94d0a6934c0f"
-					(reference "L301")
+					(reference "L302")
 					(unit 1)
 				)

Commit message: Schematics update for new chip.
Parts:
- C300, C301: value 1uF/16V -> 1uF/25V
- C302, C303, C304, C305, C308, C310, C312: value 22uF/10V -> 22uF/25V
- C307: value 10uF/10V -> 10uF/25V
- C309, C311: value 4.7uF/10V -> 4.7uF/25V
- R300, R306, R311, R315: value 100k -> 100k/1%
- R308, R312, R316: value 470k -> 470k/1%
Other:
- moved on the sheet: C302, C303, C304, C305, C306, L301, R300, R301, R302, R303, U301
