File: pcb/r2-mainboard/power_mon.kicad_sch (KiCad schematic)
At the start: 0 parts

Commit message: R2: port epd, epd_power and power_mon from R1
WP4. These three sheets are copied from pcb/mainboard/ rather than redrawn,
because the acceptance criterion is "is it the same as R1" -- copying keeps
every part, value, coordinate and wire, so the two can be diffed directly.
tools/port_r1.py does it and only ever reads R1.

Result: epd and epd_power are provably identical to R1. R1's netlist was
exported from a scratch copy and the partition of each sheet's pins into nets
compared with R2's, undoing the designator renames first: 49/49 and 44/44 net
groups, identical. power_mon differs in exactly four groups, all intended.

103 of 128 parts keep their exact R1 designator; only collisions are renamed,
+200 for R/C and +20 for U/L so the R1 number stays readable inside the new one.
Other transforms: global labels become hierarchical labels (they are different
nets in KiCad, so a mixed project would have failed to connect silently);
I2C1_* becomes *_AON; three transistor symbols moved library in KiCad 10;
SY8120 and MT9700 are lifted into r2.kicad_sym because they are not in
pcb_common at all -- in R1 they survive only as embedded definitions.

power_mon's two video-decoder channels are gone with the ADV7611, so three
shunts are repurposed without any topology change: U22 now measures the SoM's
input current, the always-on domain, and the frontlight from +VSYS. All three
INA3221s move to +3V3_AON -- on a switched rail their I2C pins would clamp the
always-on bus, and power-down IQ is 0.5 uA typ, so the always-on domain finally
becomes measurable.

Two open items closed by reading R1 properly:

- The EPD chain cannot run from +VSYS. LGS5145 is a buck with a 4.5 V minimum,
  used here as an inverting buck-boost; in steady state it sees ~25 V, but at
  startup the negative rail is at 0 V and 3.0 V from a flat cell will not start
  it. power.md §9 closed.
- Negative rails are measured by dividing between the rail and +3V3_DCDC, not
  to ground. Carried over unchanged, with a f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
Parts:
- added C141, C142, C143: 100nF/50V, Capacitor_SMD:C_0402_1005Metric, symbol Device:C
- added C163, C164, C168, C169: 1nF/25V, Capacitor_SMD:C_0402_1005Metric, symbol Device:C
- added C91: 1nF/50V, Capacitor_SMD:C_0402_1005Metric, symbol Device:C
- added R115, R117, R50, R96, R98: 1M/1%, Resistor_SMD:R_0402_1005Metric, symbol Device:R
- added R116, R118, R51, R87, R97: 100K/1%, Resistor_SMD:R_0402_1005Metric, symbol Device:R
- added R207, R208, R53, R54, R56, R60, R61, R72: 20mR, Resistor_SMD:R_0805_2012Metric, symbol Device:R
- added U21, U22, U27: INA3221, Package_DFN_QFN:Texas_RGV0016A_VQFN-16-1EP_4x4mm_P0.65mm_EP2.1x2.1mm, symbol Power_Management:INA3221
Connections:
- new net +1V2_DCDC: R60.2, U27.15 (IN+2)
- new net +1V2_FPGA: R60.1, U27.14 (IN-2)
- new net +1V35: R56.1, U27.11 (IN-1)
- new net +1V35_DCDC: R56.2, U27.12 (IN+1)
- new net +3V3: R61.1, U21.1 (IN-3)
- new net +3V3_AON: C141.1, C142.1, C143.1, R208.1, U21.16 (VPU), U21.4 (VS), U22.14 (IN-2), U22.16 (VPU), U22.4 (VS), U22.5 (A0), U27.16 (VPU), U27.4 (VS)
- new net +3V3_AON_DCDC: R208.2, U22.15 (IN+2)
- new net +3V3_DCDC: R116.2, R118.2, R61.2, U21.2 (IN+3)
- new net +5V_DCDC: R207.2, U22.12 (IN+1)
- new net +5V_EG: R54.2, U21.14 (IN-2)
- new net +5V_EPD: R53.1, R54.1, U21.12 (IN+1), U21.15 (IN+2)
- new net +5V_ES: R53.2, U21.11 (IN-1)
- new net +5V_SOM: R207.1, U22.11 (IN-1)
- new net +VBUS: R50.1
- new net +VGH: R98.2
- new net +VP: R96.2
- new net +VSYS: R72.2, U22.2 (IN+3)
- new net +VSYS_FL: R72.1, U22.1 (IN-3)
- new net -VGL: R117.1
- new net -VN: R115.1
- new net EPD_PWR_EN: U21.9 (CRITICAL)
- new net GND: C141.2, C142.2, C143.2, C163.1, C164.1, C168.1, C169.1, C91.2, R51.2, R87.1, R97.1, U21.17 (EP), U21.3 (GND), U21.5 (A0), U22.17 (EP), U22.3 (GND), U27.1 (IN-3), U27.17 (EP), U27.2 (IN+3), U27.3 (GND)
- new net SCL_AON: U21.6 (SCL), U22.6 (SCL), U27.6 (SCL)
- new net SDA_AON: U21.7 (SDA), U22.7 (SDA), U27.5 (A0), U27.7 (SDA)
- new net VBUS_MEA: C91.1, R50.2, R51.1
- new net VGH_MEA: C164.2, R97.2, R98.1
- new net VGL_MEA: C169.2, R117.2, R118.1
- new net VN_MEA: C168.2, R115.2, R116.1
- new net VP_MEA: C163.2, R87.2, R96.1
- no-connect marks 0 -> 11
Other:
- company: (none) -> Copyright 2025 Modos Tech Inc

Commit message: R2: WP5 groundwork -- Xilinx/Micron datasheets, LX16 fix, DDR bank to 1.5 V
Steps 1-3 of the WP5 plan. No FPGA sheet is drawn yet; this is the evidence base
and the one power change that had to land before fpga_ddr can be.

DATASHEETS
AMD's documentation portal no longer serves PDFs at any of the old xilinx.com
paths -- every URL returns the same 2.5 KB JavaScript shell -- so these came from
the Wayback Machine: ds162 (DC & Switching), ug380 (Configuration), ug381
(SelectIO), ug393 (PCB Design). The hardware owner supplied mt41k64m16 from
DigiKey after micron.com proved unreachable. UG385 Packaging was deliberately
skipped at 15.8 MB, since pcb_common's XC6SLX-FTG256 symbol already encodes bank
membership in its pin names.

THE FPGA IS AN LX16, NOT AN LX9
NOTES-R2-plan.md's architecture diagram said XC6SLX9 and
NOTES-R2-hardware-facts.md carried a BOM row for XC6SLX9-2FTG256C at $6.10 --
stock and price for the wrong device. The gateware targets xc6slx16-ftg256-3 in
four places (caster.xise Device/Package/Speed Grade, par/ise_flow.sh,
par/ise_run.txt, mig.prj TargetFPGA) and R1's own schematic says
XC6SLX16-FTG256. An LX9 is not a drop-in: the MIG's C3_SMALL_DEVICE parameter
exists specifically for xc6slx9 packages, so it would need the memory controller
regenerated. LCSC stock and price for the LX16 are marked for re-query rather
than guessed.

DDR BANK 1.35 V -> 1.5 V
Caster's UCF constrains all 48 DDR pins as SSTL15_II / DIFF_SSTL15_II /
LVCMOS15, and ds162.pdf Table 7 specifies SSTL15_II only over VCCO
1.425-1.575 V with VREF 0.69-0.81 V. The committed rail was 1.344 V -- 81 mV
below the VCCO minimum, with a half-rail VREF of 0.672 V below its minimum too.
Spartan-6 has no 1.35 V I/O standard to relabel the gateware to: SSTL135 appears
nowhere in ds162.pdf or ug381.pdf, and LVCMOS15 and the HSTL standards still
stop at 1.4 V. R1 runs the same way and works, but on a different layout, and
neither board can be tested from here.

mt41k64m16.pdf p.1 makes the fix fr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
Connections:
- net +1V35 renamed +1V5
- net +1V35_DCDC renamed +1V5_DCDC
Changed lines of the file:
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@@
 			)
 		)
-		(property "Value" "+1V35"
+		(property "Value" "+1V5"
 			(at 58.42 147.32 0)
 			(show_name no)
@@
 			)
 		)
-		(property "Value" "+1V35_DCDC"
+		(property "Value" "+1V5_DCDC"
 			(at 87.63 147.32 0)
 			(show_name no)

Commit message: R2: MPNs into the schematic -- and five caps carry the wrong part number
Sourcing data lived in docs/*.md, not in the schematic, so the BOM the
fab would read had 3 of 96 lines with an MPN. Resolved every LCSC code
already on the board against LCSC's own catalogue and wrote MPN +
Manufacturer back: 53 -> 60 lines, 218 components. Added LCSC codes for
L10-L13, U42 and J22/J23 from the per-sheet docs.

Verified before writing: 321 refs and 519 nets identical before and
after, no duplicated properties, pre-existing MPNs untouched.

Cross-checking each passive value against the part its LCSC code
actually names found five wrong ones, all of them the ADC sense-divider
filter caps on power_mon:

  C91                 1nF/50V  carries C131394  = 100 nF
  C163 C164 C168 C169 1nF/25V  carries C6119801 = 470 nF

Left unwritten rather than cementing the error. C1523 (0402B102K500NT,
1 nF 50 V X7R 0402, JLC Basic, 5.3 M stock) covers both positions.

Also held back: U41, whose C39313 is XC6SLX16-**2**FTG256C while
fpga.md specifies the -3 speed grade.

frontlight.md cites C1848394 as the FPC connector on J22/J23; that code
is TPS22914BYFPR. The 6-pin sibling of J24's C5213749 is C5213748.

Co-Authored-By: Claude Opus 5 <noreply@anthropic.com>
Claude-Session: https://claude.ai/code/session_01MnesETWABbVdbcVnCKfKVs
Parts:
- C141, C142, C143: MPN (none) -> CC0402KRX7R9BB104; Manufacturer (none) -> YAGEO
- R115, R117, R50, R96, R98: MPN (none) -> 0402WGF1004TCE; Manufacturer (none) -> UNI-ROYAL
- R116, R118, R51, R87, R97: MPN (none) -> 0402WGF1003TCE; Manufacturer (none) -> UNI-ROYAL
- R207, R208, R53, R54, R56, R60, R61, R72: MPN (none) -> FRL0805FR020TS; Manufacturer (none) -> FOJAN
- U21, U22, U27: MPN (none) -> INA3221AIRGVR; Manufacturer (none) -> TI
