File: pcb/r2-mainboard/power_mon.kicad_sch (KiCad schematic)
At the start: 29 parts, among them U21 INA3221, U22 INA3221, U27 INA3221

Commit message: R2: the six approved edits, and one of them was already done
Owner-approved 2026-08-19, KiCad closed for the pass.

1. R225 22k -> 20.5K/1%, LCSC C57105 (0402WGF2052TCE, UNI-ROYAL, the
   family the rest of the board already uses). Rendered and checked:
   R224 390k over R225 20.5k with R213 100k injecting VGH_DAC, so
   20.5||100 = 17.01k and VGH = 1.2 x (1 + 390/17.01) = 28.71 V at
   DAC = 0 -- exactly epd-port.md 10.3's target.
2. The five sense-divider caps that carried codes for the wrong
   capacitance -> C1523 (0402B102K500NT, 1 nF 50 V X7R, JLC Basic,
   5.3 M stock). One part covers both the 25 V and 50 V positions.
2b. R88/R224 -> C54920667 (HRC0402F3903DNTO, 390k 1%, 20 k stock).
   C25782 had 14 units against two per board. The owner found this one;
   both obvious alternatives were traps -- C23150 is 0603, and C44937
   is 3.9 ohm despite "390K" in its part number.
3. C147 set DNP rather than deleted. panel.md 7 had already ruled that
   J6.7/J6.44 stay; that covered the pins but not the capacitor on the
   dead net. DNP drops it from placement, keeps the topology of a frozen
   sheet untouched, and leaves the footprint if a future panel drives
   the rail. in_bom stays yes -- that is this board's convention for all
   13 DNP parts, so they show up flagged rather than vanishing.
4. Ten duplicate #PWR references renumbered to #PWR1112-1121 on the
   battery sheet, which was the colliding side in every case.
5. J3 was already deleted on 2026-08-15. No work needed.
6. Specter -> Reflow across 22 files: 14 sheets, 7 generators, the
   project file. .history/ deliberately untouched.

Verified as one change: netlist before and after has 518 nets with
identical pin membership, and epd_power and epd were rendered to PNG and
inspected.

Docs updated to match: epd-port.md 10 is applied rather than designed,
frontlight.md 1 loses the "9 in series is inferred" hedge (the vendor
listing confirms 2 x 9), and io-expansion.md 4's "only guess on this
sheet" is resolved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
Parts:
- C163, C164, C168, C169: LCSC C6119801 -> C1523; MPN (none) -> 0402B102K500NT; Manufacturer (none) -> FH
- C91: LCSC C131394 -> C1523; MPN (none) -> 0402B102K500NT; Manufacturer (none) -> FH
Other:
- title: Glider-R2 / Specter mainboard -> Glider-R2 / Reflow mainboard
Changed lines of the file:
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@@
 	(paper "A4")
 	(title_block
-		(title "Glider-R2 / Specter mainboard")
+		(title "Glider-R2 / Reflow mainboard")
 		(date "2026-08-07")
 		(rev "A")
@@
 			)
 		)
+		(property "MPN" "0402B102K500NT" (at 0 0 0)
+			(effects
+				(font
+					(size 1.27 1.27)
+				)
+				(hide yes)
+			)
+		)
+		(property "Manufacturer" "FH" (at 0 0 0)
+			(effects
+				(font
+					(size 1.27 1.27)
+				)
+				(hide yes)
+			)
+		)
 		(property "Value" "1nF/25V"
 			(at 210.82 69.85 90)
@@
 			)
 		)
-		(property "LCSC" "C6119801"
+		(property "LCSC" "C1523"
 			(at 217.17 68.58 0)
 			(hide yes)
@@
 			)
 		)
+		(property "MPN" "0402B102K500NT" (at 0 0 0)
+			(effects
+				(font
+					(size 1.27 1.27)
+				)
+				(hide yes)
+			)
+		)
+		(property "Manufacturer" "FH" (at 0 0 0)
+			(effects
+				(font
+					(size 1.27 1.27)
+				)
+				(hide yes)
+			)
+		)
 		(property "Value" "1nF/25V"
 			(at 210.82 54.61 90)
@@
 			)
 		)
-		(property "LCSC" "C6119801"
+		(property "LCSC" "C1523"
 			(at 217.17 53.34 0)
 			(hide yes)
@@
 			)
 		)
+		(property "MPN" "0402B102K500NT" (at 0 0 0)
+			(effects
+				(font
+					(size 1.27 1.27)
+				)
+				(hide yes)
+			)
+		)
+		(property "Manufacturer" "FH" (at 0 0 0)
+			(effects
+				(font
+					(size 1.27 1.27)
+				)
+				(hide yes)
+			)
+		)
 		(property "Value" "1nF/25V"
 			(at 210.82 85.09 90)
@@
 			)
 		)
-		(property "LCSC" "C6119801"
+		(property "LCSC" "C1523"
 			(at 217.17 83.82 0)
 			(hide yes)
@@
 			)
 		)
+		(property "MPN" "0402B102K500NT" (at 0 0 0)
+			(effects
+				(font
+					(size 1.27 1.27)
+				)
+				(hide yes)
+			)
+		)
+		(property "Manufacturer" "FH" (at 0 0 0)
+			(effects
+				(font
+					(size 1.27 1.27)
+				)
+				(hide yes)
+			)
+		)
 		(property "Value" "1nF/50V"
 			(at 205.74 115.57 90)
@@
 			)
 		)
-		(property "LCSC" "C131394"
+		(property "LCSC" "C1523"
 			(at 217.17 114.3 0)
 			(hide yes)
@@
 			)
 		)
+		(property "MPN" "0402B102K500NT" (at 0 0 0)
+			(effects
+				(font
+					(size 1.27 1.27)
+				)
+				(hide yes)
+			)
+		)
+		(property "Manufacturer" "FH" (at 0 0 0)
+			(effects
+				(font
+					(size 1.27 1.27)
+				)
+				(hide yes)
+			)
+		)
 		(property "Value" "1nF/25V"
 			(at 210.82 100.33 90)
@@
 			)
 		)
-		(property "LCSC" "C6119801"
+		(property "LCSC" "C1523"
 			(at 217.17 99.06 0)
 			(hide yes)

Commit message: R2: renumber every sheet to the page-based designator scheme
The owner's scheme is classifier + sheet page + two-digit part from 00. Four
sheets already used it; this converts the remaining nine, so all thirteen now
agree: pages 2-9 take three digits, pages 10-14 four. 292 of 333 designators
changed. A part shared by several sheets takes its lowest page, so the FPGA is
U700 (pages 7-9) and the two SoM connectors are J501/J502 (pages 5-6).

The whole risk here is silently rewiring the board, so the netlist was diffed
rather than eyeballed:

  nets 519 -> 519, total pin connections 1563 -> 1563
  named nets present in both whose pin multiset changed: 0
  ERC unchanged at 14 errors / 20 warnings
  check_ucf.py: 99 balls matched, 0 failures

That last one matters most: it resolves the gateware's 113 UCF constraints to
board nets *by ball name*, so it is the sharpest detector of the corruption
this change could cause.

Two earlier attempts did cause exactly that. A bare quoted-string substitution
also rewrites FPGA ball names (C1, D2, N11, T1) and BTH-060 pin names (A1-D60),
which are spelled exactly like designators; one run left ERC identical while 40
nets came back with a different pin multiset. The tool now substitutes only at
the two positions that store an instance's designator, and excludes every pin
name everywhere else. docs/layout.md 9.5 records the hazard and how to prove a
renumber was clean.

Only the three scripts that read the design are updated. The gen_*/patch_*/
port_r1.py scripts keep the old names deliberately: each wrote a sheet once and
has not been re-runnable since it was hand-edited in Eeschema, so they are a
historical record -- and port_r1.py's dict keys are R1 designators that were
never renumbered at all.

Co-Authored-By: Claude Opus 5 <noreply@anthropic.com>
Claude-Session: https://claude.ai/code/session_01MHTAe6ZnhogTEgtyPcLhwG
Parts:
- renumbered C91 to C1200, C141 to C1201, C142 to C1202, C143 to C1203, C163 to C1204, C164 to C1205, C168 to C1206, C169 to C1207, R50 to R1200, R51 to R1201, R53 to R1202, R54 to R1203, R56 to R1204, R60 to R1205, R61 to R1206, R72 to R1207, R87 to R1208, R96 to R1209, R97 to R1210, R98 to R1211, R115 to R1212, R116 to R1213, R117 to R1214, R118 to R1215, R207 to R1216, R208 to R1217, U21 to U1200, U22 to U1201, U27 to U1202
Changed lines of the file:
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@@
 		(in_pos_files yes)
 		(dnp no)
-		(property "Reference" "R116"
+		(property "Reference" "R1213"
 			(at 227.33 76.2 90)
 			(show_name no)
@@
 			(project "r2"
 				(path "/dee825bf-c2f1-415d-afdf-cf702072a6e8/ba07d81a-25ab-477b-a3a6-9eea9be2fd08"
-					(reference "R116")
+					(reference "R1213")
 					(unit 1)
 				)
@@
 		(dnp no)
 		(fields_autoplaced yes)
-		(property "Reference" "U21"
+		(property "Reference" "U1200"
 			(at 111.4141 33.02 0)
 			(show_name no)
@@
 			(project "r2"
 				(path "/dee825bf-c2f1-415d-afdf-cf702072a6e8/ba07d81a-25ab-477b-a3a6-9eea9be2fd08"
-					(reference "U21")
+					(reference "U1200")
 					(unit 1)
 				)
@@
 		(in_pos_files yes)
 		(dnp no)
-		(property "Reference" "C164"
+		(property "Reference" "C1205"
 			(at 223.52 69.85 90)
 			(show_name no)
@@
 			(project "r2"
 				(path "/dee825bf-c2f1-415d-afdf-cf702072a6e8/ba07d81a-25ab-477b-a3a6-9eea9be2fd08"
-					(reference "C164")
+					(reference "C1205")
 					(unit 1)
 				)
@@
 		(in_pos_files yes)
 		(dnp no)
-		(property "Reference" "C163"
+		(property "Reference" "C1204"
 			(at 223.52 54.61 90)
 			(show_name no)
@@
 			(project "r2"
 				(path "/dee825bf-c2f1-415d-afdf-cf702072a6e8/ba07d81a-25ab-477b-a3a6-9eea9be2fd08"
-					(reference "C163")
+					(reference "C1204")
 					(unit 1)
 				)
@@
 		(dnp no)
 		(fields_autoplaced yes)
-		(property "Reference" "U22"
+		(property "Reference" "U1201"
 			(at 111.4141 86.36 0)
 			(show_name no)
@@
 			(project "r2"
 				(path "/dee825bf-c2f1-415d-afdf-cf702072a6e8/ba07d81a-25ab-477b-a3a6-9eea9be2fd08"
-					(reference "U22")
+					(reference "U1201")
 					(unit 1)
 				)
@@
 		(in_pos_files yes)
 		(dnp no)
-		(property "Reference" "R96"
+		(property "Reference" "R1209"
 			(at 227.33 45.72 90)
 			(show_name no)
@@
 			(project "r2"
 				(path "/dee825bf-c2f1-415d-afdf-cf702072a6e8/ba07d81a-25ab-477b-a3a6-9eea9be2fd08"
-					(reference "R96")
+					(reference "R1209")
 					(unit 1)
 				)
@@
 		(in_pos_files yes)
 		(dnp no)
-		(property "Reference" "R87"
+		(property "Reference" "R1208"
 			(at 220.98 45.72 90)
 			(show_name no)
@@
 			(project "r2"
 				(path "/dee825bf-c2f1-415d-afdf-cf702072a6e8/ba07d81a-25ab-477b-a3a6-9eea9be2fd08"
-					(reference "R87")
+					(reference "R1208")
 					(unit 1)
 				)
@@
 		(in_pos_files yes)
 		(dnp no)
-		(property "Reference" "R56"
+		(property "Reference" "R1204"
 			(at 68.58 147.32 90)
 			(show_name no)
@@
 			(project "r2"
 				(path "/dee825bf-c2f1-415d-afdf-cf702072a6e8/ba07d81a-25ab-477b-a3a6-9eea9be2fd08"
-					(reference "R56")
+					(reference "R1204")
 					(unit 1)
 				)
@@
 		(in_pos_files yes)
 		(dnp no)
-		(property "Reference" "C142"
+		(property "Reference" "C1202"
 			(at 132.461 89.0016 0)
 			(show_name no)
@@
 			(project "r2"
 				(path "/dee825bf-c2f1-415d-afdf-cf702072a6e8/ba07d81a-25ab-477b-a3a6-9eea9be2fd08"
-					(reference "C142")
+					(reference "C1202")
 					(unit 1)
 				)
@@
 		(dnp no)
 		(fields_autoplaced yes)
-		(property "Reference" "U27"
+		(property "Reference" "U1202"
 			(at 111.4141 139.7 0)
 			(show_name no)
@@
 			(project "r2"
 				(path "/dee825bf-c2f1-415d-afdf-cf702072a6e8/ba07d81a-25ab-477b-a3a6-9eea9be2fd08"
-					(reference "U27")
+					(reference "U1202")
 					(unit 1)
 				)
@@
 		(in_pos_files yes)
 		(dnp no)
-		(property "Reference" "C168"
+		(property "Reference" "C1206"
 			(at 223.52 85.09 90)
 			(show_name no)
@@
 			(project "r2"
 				(path "/dee825bf-c2f1-415d-afdf-cf702072a6e8/ba07d81a-25ab-477b-a3a6-9eea9be2fd08"
-					(reference "C168")
+					(reference "C1206")
 					(unit 1)
 				)
@@
 		(in_pos_files yes)
 		(dnp no)
-		(property "Reference" "R208"
+		(property "Reference" "R1217"
 			(at 68.58 101.6 90)
 			(show_name no)
@@
 			(project "r2"
 				(path "/dee825bf-c2f1-415d-afdf-cf702072a6e8/ba07d81a-25ab-477b-a3a6-9eea9be2fd08"
-					(reference "R208")
+					(reference "R1217")
 					(unit 1)
 				)
@@
 		(in_pos_files yes)
 		(dnp no)
-		(property "Reference" "C141"
+		(property "Reference" "C1201"
 			(at 132.461 142.3416 0)
 			(show_name no)
@@
 			(project "r2"
 				(path "/dee825bf-c2f1-415d-afdf-cf702072a6e8/ba07d81a-25ab-477b-a3a6-9eea9be2fd08"
-					(reference "C141")
+					(reference "C1201")
 					(unit 1)
 				)
@@
 		(in_pos_files yes)
 		(dnp no)
-		(property "Reference" "R118"
+		(property "Reference" "R1215"
 			(at 227.33 91.44 90)
 			(show_name no)
@@
 			(project "r2"
 				(path "/dee825bf-c2f1-415d-afdf-cf702072a6e8/ba07d81a-25ab-477b-a3a6-9eea9be2fd08"
-					(reference "R118")
+					(reference "R1215")
 					(unit 1)
 				)
@@
 		(in_pos_files yes)
 		(dnp no)
-		(property "Reference" "R50"
+		(property "Reference" "R1200"
 			(at 227.33 106.68 90)
 			(show_name no)
@@
 			(project "r2"
 				(path "/dee825bf-c2f1-415d-afdf-cf702072a6e8/ba07d81a-25ab-477b-a3a6-9eea9be2fd08"
-					(reference "R50")
+					(reference "R1200")
 					(unit 1)
 				)
@@
 		(in_pos_files yes)
 		(dnp no)
-		(property "Reference" "R51"
+		(property "Reference" "R1201"
 			(at 220.98 106.68 90)
 			(show_name no)
@@
 			(project "r2"
 				(path "/dee825bf-c2f1-415d-afdf-cf702072a6e8/ba07d81a-25ab-477b-a3a6-9eea9be2fd08"
-					(reference "R51")
+					(reference "R1201")
 					(unit 1)
 				)
@@
 		(in_pos_files yes)
 		(dnp no)
-		(property "Reference" "R72"
+		(property "Reference" "R1207"
 			(at 68.58 109.22 90)
 			(show_name no)
@@
 			(project "r2"
 				(path "/dee825bf-c2f1-415d-afdf-cf702072a6e8/ba07d81a-25ab-477b-a3a6-9eea9be2fd08"
-					(reference "R72")
+					(reference "R1207")
 					(unit 1)
 				)
@@
 		(in_pos_files yes)
 		(dnp no)
-		(property "Reference" "R60"
+		(property "Reference" "R1205"
 			(at 68.58 154.94 90)
 			(show_name no)
@@
 			(project "r2"
 				(path "/dee825bf-c2f1-415d-afdf-cf702072a6e8/ba07d81a-25ab-477b-a3a6-9eea9be2fd08"
-					(reference "R60")
+					(reference "R1205")
 					(unit 1)
 				)
@@
 		(in_pos_files yes)
 		(dnp no)
-		(property "Reference" "R115"
+		(property "Reference" "R1212"
 			(at 220.98 76.2 90)
 			(show_name no)
@@
 			(project "r2"
 				(path "/dee825bf-c2f1-415d-afdf-cf702072a6e8/ba07d81a-25ab-477b-a3a6-9eea9be2fd08"
-					(reference "R115")
+					(reference "R1212")
 					(unit 1)
 				)
@@
 		(in_pos_files yes)
 		(dnp no)
-		(property "Reference" "R98"
+		(property "Reference" "R1211"
 			(at 227.33 60.96 90)
 			(show_name no)
@@
 			(project "r2"
 				(path "/dee825bf-c2f1-415d-afdf-cf702072a6e8/ba07d81a-25ab-477b-a3a6-9eea9be2fd08"
-					(reference "R98")
+					(reference "R1211")
 					(unit 1)
 				)
@@
 		(in_pos_files yes)
 		(dnp no)
-		(property "Reference" "R54"
+		(property "Reference" "R1203"
 			(at 68.58 48.26 90)
 			(show_name no)
@@
 			(project "r2"
 				(path "/dee825bf-c2f1-415d-afdf-cf702072a6e8/ba07d81a-25ab-477b-a3a6-9eea9be2fd08"
-					(reference "R54")
+					(reference "R1203")
 					(unit 1)
 				)
@@
 		(in_pos_files yes)
 		(dnp no)
-		(property "Reference" "C91"
+		(property "Reference" "C1200"
 			(at 218.44 115.57 90)
 			(show_name no)
@@
 			(project "r2"
 				(path "/dee825bf-c2f1-415d-afdf-cf702072a6e8/ba07d81a-25ab-477b-a3a6-9eea9be2fd08"
-					(reference "C91")
+					(reference "C1200")
 					(unit 1)
 				)
@@
 		(in_pos_files yes)
 		(dnp no)
-		(property "Reference" "R53"
+		(property "Reference" "R1202"
 			(at 68.58 40.64 90)
 			(show_name no)
@@
 			(project "r2"
 				(path "/dee825bf-c2f1-415d-afdf-cf702072a6e8/ba07d81a-25ab-477b-a3a6-9eea9be2fd08"
-					(reference "R53")
+					(reference "R1202")
 					(unit 1)
 				)
@@
 		(in_pos_files yes)
 		(dnp no)
-		(property "Reference" "R207"
+		(property "Reference" "R1216"
 			(at 68.58 93.98 90)
 			(show_name no)
@@
 			(project "r2"
 				(path "/dee825bf-c2f1-415d-afdf-cf702072a6e8/ba07d81a-25ab-477b-a3a6-9eea9be2fd08"
-					(reference "R207")
+					(reference "R1216")
 					(unit 1)
 				)
@@
 		(in_pos_files yes)
 		(dnp no)
-		(property "Reference" "C169"
+		(property "Reference" "C1207"
 			(at 223.52 100.33 90)
 			(show_name no)
@@
 			(project "r2"
 				(path "/dee825bf-c2f1-415d-afdf-cf702072a6e8/ba07d81a-25ab-477b-a3a6-9eea9be2fd08"
-					(reference "C169")
+					(reference "C1207")
 					(unit 1)
 				)
@@
 		(in_pos_files yes)
 		(dnp no)
-		(property "Reference" "R97"
+		(property "Reference" "R1210"
 			(at 220.98 60.96 90)
 			(show_name no)
@@
 			(project "r2"
 				(path "/dee825bf-c2f1-415d-afdf-cf702072a6e8/ba07d81a-25ab-477b-a3a6-9eea9be2fd08"
-					(reference "R97")
+					(reference "R1210")
 					(unit 1)
 				)
@@
 		(in_pos_files yes)
 		(dnp no)
-		(property "Reference" "R61"
+		(property "Reference" "R1206"
 			(at 68.58 55.88 90)
 			(show_name no)
@@
 			(project "r2"
 				(path "/dee825bf-c2f1-415d-afdf-cf702072a6e8/ba07d81a-25ab-477b-a3a6-9eea9be2fd08"
-					(reference "R61")
+					(reference "R1206")
 					(unit 1)
 				)
@@
 		(in_pos_files yes)
 		(dnp no)
-		(property "Reference" "C143"
+		(property "Reference" "C1203"
 			(at 132.461 35.6616 0)
 			(show_name no)
@@
 			(project "r2"
 				(path "/dee825bf-c2f1-415d-afdf-cf702072a6e8/ba07d81a-25ab-477b-a3a6-9eea9be2fd08"
-					(reference "C143")
+					(reference "C1203")
 					(unit 1)
 				)
@@
 		(in_pos_files yes)
 		(dnp no)
-		(property "Reference" "R117"
+		(property "Reference" "R1214"
 			(at 220.98 91.44 90)
 			(show_name no)
@@
 			(project "r2"
 				(path "/dee825bf-c2f1-415d-afdf-cf702072a6e8/ba07d81a-25ab-477b-a3a6-9eea9be2fd08"
-					(reference "R117")
+					(reference "R1214")
 					(unit 1)
 				)
