File: pcb/r2-mainboard/r2_claude.kicad_pcb (KiCad board)
At the start: 4 copper layers, 90 x 80 mm, 324 parts, among them J1 USB-C 16P, J2 Pico-Lock 504050-0391, J20 SWD+JTAG (DNP), J21 MICRO_SD(TFC-WPAPR-08), J22 HC-FPC-05-09-6RLTAG, J23 HC-FPC-05-09-6RLTAG, J24 HC-FPC-05-09-8RLTAG, J25 SolderPads 3x, J26 BTH-060-01-L-D-A-K-TR, J27 BTH-060-01-L-D-A-K-TR, J6 FPC-05F-50PH20, Q1 AO3401A, Q2 S8050, Q6 AO3400A, Q7 AO3401A, Q8 AO3401A, Q9 AO3400A, SW20 SW, SW21 SW, SW22 SW, U1 BQ25892RTW, U10 TPS7A0233DBVR, U12 TPS61022RWUR, U13 TPS63802DLAR, U14 TPS62A02DRLR, U15 TPS62A02DRLR, U2 MAX17048G+T10, U20 STM32G0B1RCT6, U21 INA3221, U22 INA3221, U23 LGS6302B5, U24 LGS6302B5, U26 LGS5145, U27 INA3221, U3 USBLC6-2SC6, U31 LM321, U41 XC6SLX-FTG256, U42 W25Q128JVSIQ, U52 MT41K64M16TW, U53 LM3630A, U54 TPS22914BYFPR, U55 TPS22914BYFPR, U6 MT9700, U7 TPS22914BYFPR, U8 TPS22914BYFPR, U9 LGS5145, X1 33.33MHz, X2 PCM-071, Y20 32.768kHz

Commit message: R2: withdraw the RWU0007A thermal-pad concern -- it was wrong
power.md §7 item 2 said KiCad's Texas_RWU0007A_VQFN-7_2x2mm_P0.5mm leaves the
thermal-pad segments unnumbered, so U12's heat path is not tied to GND, and to
copy the footprint into r2.pretty and renumber those pads 1 before layout.

Reading the placed footprint with the layer field visible: the six unnumbered
pads are F.Paste ONLY. They are stencil apertures -- each large pad split into
two openings to control solder volume, the standard idiom at that size. Pads
1/2/3 are F.Cu + F.Mask, numbered, and netted GND / SW / +5V_DCDC. Pin 1 is the
thermal path per Table 5-1 and it is on GND already.

Acting on the note would have renumbered paste apertures into copper and
shorted GND, SW and VOUT together -- creating the failure it was meant to
prevent. Found because the owner is routing U12 right now.

§11.2 item 5 amended to a plain layout instruction, and §8's open-items list
no longer carries it.

Co-Authored-By: Claude Opus 5 <noreply@anthropic.com>
Claude-Session: https://claude.ai/code/session_01MnesETWABbVdbcVnCKfKVs
Routing:
- net GND: vias 0 -> 77
- added copper zone on B.Cu, net GND
- added copper zone on F.Cu, net GND
- added copper zone on In1.Cu, net GND

Commit message: R2 claude: ground planes, the two HV islands, and a maze router
Planes first, because GND is 344 of the 1047 ratsnest edges and layout.md
7.2 wants the DDR3 bus over one continuous In1.Cu -- which only exists if
In1.Cu is a plane rather than 344 tracks.

  F.Cu    GND pour, so SMD ground pads connect where they sit
  In1.Cu  the solid plane, the continuous reference
  In2.Cu  R1 calls this "mixed"; the third routing layer here
  B.Cu    GND pour
  + 76 stitching vias tying the outer pours to the plane

GND ratsnest 666 -> 44 pads. Board DRC 11 violations, all silkscreen: no
copper errors, no shorts, no dangling copper.

layout.md 7.1 / epd-port.md 11.1, the item the docs call the single most
dangerous in the project: U9 and U26 are inverting buck-boosts whose pin 2 is
labelled GND but sits at -VGL (about -20 V) and -VN (about -15 V). Each now has
a rule area over its courtyard + 1.5 mm that forbids copper pour on every
layer while still allowing tracks and vias, so the plane is cut away beneath
the part but its own signals can still reach it. check_pcb.py already refuses
a zone on -VGL/-VN; check_hv_islands.py is the other half, sampling a grid
across each island against the filled polygons KiCad actually produced. Both
islands: 0 of 700 sample points carry GND copper.

route.py is an A* maze router on a 0.1 mm grid over F.Cu/In2.Cu/B.Cu (0.1 mm
divides every pad pitch in the design, so pads land on grid nodes). Occupancy
is a net id per cell; a cell is usable when empty or already ours.

Four things it took to make it correct, each found by DRC and each worth
keeping:

- Pad halos overwrote each other. U14 is a SOT-563 whose pads are 0.35 mm tall
  on a 0.5 mm pitch, so a 0.19 mm halo reaches into the next pad; whichever was
  stamped last owned the overlap and tracks drove straight across a neighbour.
  Bodies are stamped first now, then halos, and a halo cell already owned by a
  different net becomes BLOCKED rather than changing hands.

- Pad dimensions were tra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
Routing:
- net GND: vias 77 -> 76

Commit message: R2: GND does not belong in a width class, and a check that says why
The owner, mid-route: "I can't always have a 0.6 mm GND trace. Sometimes for
signals it's just not necessary." Correct, and the class was at fault.

GND was in PWR, whose track width is 0.6 mm. But GND's current path is the
In1.Cu plane; a GND segment is almost always a short stub from a pad to a
stitching via, where 0.6 mm buys nothing and gets overridden by hand every
time. On Default it routes at 0.2 mm and takes a 0.6/0.3 via, which is also the
more useful stitching via -- PWR's 0.8/0.35 is clumsy under a BGA. Clearance is
0.11 either way. +VSYS stays in PWR: unlike GND it has real routed runs to the
four converters that should start wide.

The first idea for a check was "every segment must meet its net class width".
GND is exactly why that is wrong: it would have flagged dozens of correct 0.2 mm
stubs, and a noisy check gets switched off, taking the real findings with it. So
check 7 is inverted -- only nets where a document states a current, each entry
carrying that current and its source, with the width from IPC-2152 at 1 oz and
20 C rise rounded DOWN to a floor. A net absent from the table is not unimportant;
it is a net nobody has put a number on yet.

It finds 8 of the 10 listed nets routed and all 8 too thin, the worst being
Net-(U12-SW) at 0.13 mm on a node carrying ~2.8 A average and 3.4 A peak.

Also fixes a trap in import_r1_settings.py: it assigned the class list wholesale,
so a second run would have silently deleted the owner's hand-made Signals_NET
class. It now keeps any class it did not create, and their patterns with them.

Co-Authored-By: Claude Opus 5 <noreply@anthropic.com>
Claude-Session: https://claude.ai/code/session_01MnesETWABbVdbcVnCKfKVs
Routing:
- net GND: vias 76 -> 77
