File: pcb/r2-mainboard/r2_claude.kicad_pcb (KiCad board)
At the start: 4 copper layers, 185.5 x 95 mm, 327 parts, among them J1 USB-C 16P, J2 Pico-Lock 504050-0391, J20 SWD+JTAG (DNP), J21 MICRO_SD(TFC-WPAPR-08), J22 HC-FPC-05-09-6RLTAG, J23 HC-FPC-05-09-6RLTAG, J24 HC-FPC-05-09-8RLTAG, J25 SolderPads 3x, J26 BTH-060-01-L-D-A-K-TR, J27 BTH-060-01-L-D-A-K-TR, J6 FPC-05F-50PH20, Q1 AO3401A, Q2 S8050, Q6 AO3400A, Q7 AO3401A, Q8 AO3401A, Q9 AO3400A, SW20 SW, SW21 SW, SW22 SW, U1 BQ25892RTW, U10 TPS7A0233DBVR, U12 TPS61022RWUR, U13 TPS63802DLAR, U14 TPS62A02DRLR, U15 TPS62A02DRLR, U2 MAX17048G+T10, U20 STM32G0B1RCT6, U21 INA3221, U22 INA3221, U23 LGS6302B5, U24 LGS6302B5, U26 LGS5145, U27 INA3221, U3 USBLC6-2SC6, U31 LM321, U41 XC6SLX-FTG256, U42 W25Q128JVSIQ, U52 MT41K64M16TW, U53 LM3630A, U54 TPS22914BYFPR, U55 TPS22914BYFPR, U6 MT9700, U7 TPS22914BYFPR, U8 TPS22914BYFPR, U9 LGS5145, X1 33.33MHz, X2 PCM-071, Y20 32.768kHz

Commit message: Recover from the KiCad crash; finish the USB1_D+/D- rename
KiCad crashed and deleted 150 tracked files plus 19 untracked ones.
Recovery, in the order that matters:

  1. copied _restore_backup_2026-08-31T20-57-08-688 aside (261 MB)
  2. rescued the 4 untracked files that existed only there -- the
     PHYTEC PCM-071 STEP/x_t/Basic models and the library/3dmodels copy.
     The other 15 were __pycache__, .lck and .bak.
  3. git checkout of the 150 deletions (deletions only, so the six
     modified files were never touched)
  4. three files the crash had *rolled back* rather than deleted, and
     which git checkout therefore missed, restored from HEAD:
       r2.kicad_sym    -- was 11 symbols, missing TPS2553DBV,
                          BTH-060_AB/CD and BOM_ITEM, and carrying the
                          superseded PCM-071 symbol: the pre-2026-08-20
                          state, before the SoM was split in two
       sym-lib-table   -- had lost the Reflow declaration
       fp-lib-table    -- had lost Reflow and (version 7)

r2.kicad_pcb was not damaged -- 328 footprints, 471 segments, same as
HEAD. Rescuing PCM-071_1573-1.STEP also repairs X2's 3D model path,
which an earlier restore had broken.

Separately, the USB1 net rename is finished at the owner's request:
som.kicad_sch USB1_DM/DP -> USB1_D-/D+ (the J26 X_USB1_* pin names are
PHYTEC's and are untouched), and a USB1_+ typo on U57's second ESD stub
in io_expansion corrected to USB1_D+. sheet_pins + wire_root re-run:
113 names on 233 sheet pins, 113 joined, 0 one-sided. All five USB1
nets verified node-for-node.

⚠ The tree is mid-renumber (J200/U200/U300... appearing) and carries one
severed net: +3V3_TOUCH reaches only J22.1, while U54.A1 and C517.1 sit
on an unnamed Net-(U54-OUT). Committed as-is so the recovery is not at
risk from another crash; the break is called out rather than hidden.

Co-Authored-By: Claude Opus 5 <noreply@anthropic.com>
Claude-Session: https://claude.ai/code/session_01MHTAe6Znh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
Parts:
- removed R14, R15: 0R, Resistor_SMD:R_0402_1005Metric
- removed R16: 10k, Resistor_SMD:R_0402_1005Metric
- C4, C5, C7: footprint Capacitor_SMD:C_0805_2012Metric -> Capacitor_SMD:C_0402_1005Metric
- moved J1 165.9 mm to (183.5, 63.0), turned to 180 degrees
- moved Q9 160.1 mm to (128.6, 26.9), turned to -90 degrees
- moved SW22 160.0 mm to (133.6, 24.5), turned to 90 degrees
- moved U3 155.8 mm to (186.2, 55.9), turned to 90 degrees
- moved R43 155.4 mm to (128.3, 23.1)
- moved F1 148.6 mm to (176.9, 63.0), turned to -90 degrees
- moved R512 147.7 mm to (127.3, 29.9), turned to 90 degrees
- moved R510 147.1 mm to (136.4, 30.0), turned to 90 degrees
- moved FB20 145.0 mm to (116.2, 22.2), turned to -90 degrees
- moved R504 143.2 mm to (165.0, 38.2), turned to -90 degrees
- moved C518 143.0 mm to (107.7, 35.2), turned to -90 degrees
- moved U12 142.6 mm to (144.2, 22.7), turned to 90 degrees
- moved U55 142.5 mm to (116.3, 38.3), turned to 90 degrees
- moved Y20 140.8 mm to (120.0, 38.0)
- moved U54 140.8 mm to (111.7, 36.1), turned to 180 degrees
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Routing:
- net /battery/CHG_TS: track 25.1 -> 0.00 mm, vias 3 -> 0
- net GND: track 19.9 -> 0.00 mm, vias 0 -> 77
- net +VBAT: track 17.5 -> 0.00 mm
- net +VSYS: track 7.16 -> 0.00 mm
- net Net-(C3-Pad2): track 6.15 -> 0.00 mm
- net Net-(U1-BTST): track 4.46 -> 0.00 mm
- net /battery/REGN: track 1.67 -> 0.00 mm
- net Net-(U1-PMID): track 1.56 -> 0.00 mm
- net +VBUS: track 1.55 -> 0.00 mm
- net Net-(U1-ILIM): track 1.33 -> 0.00 mm
- added copper zone on B.Cu, net GND
- added copper zone on F.Cu, net GND
Other:
- board size 185.5 x 95 mm -> 90 x 80 mm
