File: pcb/r2-mainboard/r2_claude.kicad_pcb (KiCad board)
At the start: 4 copper layers, 90 x 80 mm, 324 parts, among them J1 USB-C 16P, J2 Pico-Lock 504050-0391, J20 SWD+JTAG (DNP), J21 MICRO_SD(TFC-WPAPR-08), J22 HC-FPC-05-09-6RLTAG, J23 HC-FPC-05-09-6RLTAG, J24 HC-FPC-05-09-8RLTAG, J25 SolderPads 3x, J26 BTH-060-01-L-D-A-K-TR, J27 BTH-060-01-L-D-A-K-TR, J6 FPC-05F-50PH20, Q1 AO3401A, Q2 S8050, Q6 AO3400A, Q7 AO3401A, Q8 AO3401A, Q9 AO3400A, SW20 SW, SW21 SW, SW22 SW, U1 BQ25892RTW, U10 TPS7A0233DBVR, U12 TPS61022RWUR, U13 TPS63802DLAR, U14 TPS62A02DRLR, U15 TPS62A02DRLR, U2 MAX17048G+T10, U20 STM32G0B1RCT6, U21 INA3221, U22 INA3221, U23 LGS6302B5, U24 LGS6302B5, U26 LGS5145, U27 INA3221, U3 USBLC6-2SC6, U31 LM321, U41 XC6SLX-FTG256, U42 W25Q128JVSIQ, U52 MT41K64M16TW, U53 LM3630A, U54 TPS22914BYFPR, U55 TPS22914BYFPR, U6 MT9700, U7 TPS22914BYFPR, U8 TPS22914BYFPR, U9 LGS5145, X1 33.33MHz, X2 PCM-071, Y20 32.768kHz

Commit message: routing
Parts:
- added R14: 0R, Resistor_SMD:R_0402_1005Metric, F.Cu at (100.6, 124.9)
- added R15: 0R, Resistor_SMD:R_0402_1005Metric, F.Cu at (103.5, 113.0)
- added R16: 10k, Resistor_SMD:R_0402_1005Metric, F.Cu at (103.5, 115.0)
- C4, C5, C7: footprint Capacitor_SMD:C_0402_1005Metric -> Capacitor_SMD:C_0805_2012Metric
- moved J1 165.9 mm to (19.7, 36.6), turned to 0 degrees
- moved Q9 160.1 mm to (62.0, 172.5), turned to 0 degrees
- moved SW22 160.0 mm to (71.0, 171.8), turned to 0 degrees
- moved U3 155.8 mm to (31.5, 37.0), turned to 0 degrees
- moved R43 155.4 mm to (76.3, 169.5)
- moved F1 148.6 mm to (29.6, 43.0), turned to 0 degrees
- moved R512 147.7 mm to (79.2, 169.5), turned to 0 degrees
- moved R510 147.1 mm to (79.2, 165.6), turned to 0 degrees
- moved FB20 145.0 mm to (76.3, 161.6), turned to 0 degrees
- moved R504 143.2 mm to (113.7, 171.9), turned to 0 degrees
- moved C518 143.0 mm to (117.5, 177.8), turned to 0 degrees
- moved U12 142.6 mm to (103.0, 159.2), turned to 0 degrees
- moved U55 142.5 mm to (114.2, 180.7), turned to 0 degrees
- moved Y20 140.8 mm to (77.3, 172.2)
- moved U54 140.8 mm to (114.2, 176.8), turned to 0 degrees
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Routing:
- net /battery/CHG_TS: track 0.00 -> 25.1 mm, vias 0 -> 3
- net GND: track 0.00 -> 19.9 mm, vias 77 -> 0
- net +VBAT: track 0.00 -> 17.5 mm
- net +VSYS: track 0.00 -> 7.16 mm
- net Net-(C3-Pad2): track 0.00 -> 6.15 mm
- net Net-(U1-BTST): track 0.00 -> 4.46 mm
- net /battery/REGN: track 0.00 -> 1.67 mm
- net Net-(U1-PMID): track 0.00 -> 1.56 mm
- net +VBUS: track 0.00 -> 1.55 mm
- net Net-(U1-ILIM): track 0.00 -> 1.33 mm
- removed copper zone on B.Cu, net GND
- removed copper zone on F.Cu, net GND
Other:
- board size 90 x 80 mm -> 185.5 x 95 mm
