File: pcb/r2-mainboard/battery.kicad_sch (KiCad schematic)
At the start: 35 parts, among them J1 USB-C 16P, J2 Pico-Lock 504050-0391, J25 SolderPads 3x, U1 BQ25892RTW, U2 MAX17048G+T10, U3 USBLC6-2SC6

Commit message: routing and board layout
Connections:
- net USBD+: now also J1.A6 (USBD+), J1.B6 (USBD+), U3.3 (I/O2)
- net USBD-: now also J1.A7 (USBD-), J1.B7 (USBD-), U3.1 (I/O1)
- net +VBUS_PRE: now reaches F1.1, J1.A4 (VBUS), J1.A9 (VBUS), J1.B4 (VBUS), J1.B9 (VBUS)
- net CHG_SW: now reaches C3.2, L1.1, U1.19 (SW), U1.20 (SW)
- net CHG_DSEL: no longer names the net of U1.24 (NC/DSEL)
- no-connect marks 2 -> 3
Other:
- note removed: "Second-source option field — fit ONLY for the BQ25890/95 (D+/D-/DSEL variant). Not fitted for the BQ25892/96."
- moved on the sheet: C7, C8, F1, J1, J2, R1, R11, R12, R13, R17, R18, R19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
