File: pcb/r2-mainboard/battery.kicad_sch (KiCad schematic)
At the start: 35 parts, among them J200 USB-C 16P, J201 Pico-Lock 504050-0391, J202 SolderPads 3x, U200 BQ25892RTW, U201 MAX17048G+T10, U202 USBLC6-2SC6

Commit message: changing to osb62x-pm
Parts:
- U200: footprint Package_DFN_QFN:WQFN-24-1EP_4x4mm_P0.5mm_EP2.6x2.6mm -> Package_DFN_QFN:Texas_RTW_WQFN-24-1EP_4x4mm_P0.5mm_EP2.7x2.7mm_ThermalVias

Commit message: Schematics update for new chip.
Parts:
- C205: value 4.7uF/16V -> 4.7uF/25V; footprint Capacitor_SMD:C_0603_1608Metric -> Capacitor_SMD:C_0805_2012Metric
- C207: value 100nF/16V -> 100nF/50V
- R200, R201: value 5.1k -> 5.1k/1%
- R202, R203, R204, R215, R217: value 10k -> 10k/1%
- R205, R206: value 2.2k -> 2.2k/1%
- R213, R214: value 100k -> 100k/1%
- R216: value 1k -> 1k/1%
Changed lines of the file:
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@@
 			)
 		)
-		(property "Value" "10k"
+		(property "Value" "10k/1%"
 			(at 130.81 179.832 0)
 			(show_name no)
@@
 			)
 		)
-		(property "Value" "5.1k"
+		(property "Value" "5.1k/1%"
 			(at 77.47 103.632 0)
 			(show_name no)
@@
 			)
 		)
-		(property "Value" "10k"
+		(property "Value" "10k/1%"
 			(at 151.13 179.832 0)
 			(show_name no)
@@
 			)
 		)
-		(property "Value" "1k"
+		(property "Value" "1k/1%"
 			(at 210.82 227.3299 0)
 			(show_name no)
@@
 			)
 		)
-		(property "Value" "100k"
+		(property "Value" "100k/1%"
 			(at 129.54 207.772 0)
 			(show_name no)
@@
 			)
 		)
-		(property "Value" "10k"
+		(property "Value" "10k/1%"
 			(at 110.49 179.832 0)
 			(show_name no)
@@
 			)
 		)
-		(property "Value" "100nF/16V"
+		(property "Value" "100nF/50V"
 			(at 328.93 80.772 0)
 			(show_name no)
@@
 			)
 		)
-		(property "Value" "5.1k"
+		(property "Value" "5.1k/1%"
 			(at 97.79 103.632 0)
 			(show_name no)
@@
 			)
 		)
-		(property "Value" "4.7uF/16V"
+		(property "Value" "4.7uF/25V"
 			(at 217.17 145.542 0)
 			(show_name no)
@@
 			)
 		)
-		(property "Footprint" "Capacitor_SMD:C_0603_1608Metric"
+		(property "Footprint" "Capacitor_SMD:C_0805_2012Metric"
 			(at 214.63 143.51 0)
 			(hide yes)
@@
 			)
 		)
-		(property "Value" "2.2k"
+		(property "Value" "2.2k/1%"
 			(at 191.77 179.832 0)
 			(show_name no)
@@
 			)
 		)
-		(property "Value" "10k"
+		(property "Value" "10k/1%"
 			(at 325.12 137.922 0)
 			(show_name no)
@@
 			)
 		)
-		(property "Value" "100k"
+		(property "Value" "100k/1%"
 			(at 109.22 207.772 0)
 			(show_name no)
@@
 			)
 		)
-		(property "Value" "10k"
+		(property "Value" "10k/1%"
 			(at 361.95 137.922 0)
 			(show_name no)
@@
 			)
 		)
-		(property "Value" "2.2k"
+		(property "Value" "2.2k/1%"
 			(at 171.45 179.832 0)
 			(show_name no)
