File: pcb/r2-mainboard/frontlight.kicad_sch (KiCad schematic)
At the start: 10 parts, among them J24 HC-FPC-05-09-8RLTAG, U53 LM3630A

Commit message: routing and board layout
Parts:
- removed R509: 0R, Resistor_SMD:R_0402_1005Metric, symbol Device:R
- R508: now not fitted
Connections:
- net +VSYS_FL: now also U53.C2 (SEL)
- net FL_INT#: no longer names the net of U53.B2 (~{INTN})
- net FL_INT#: no longer R508.1
- no-connect marks 4 -> 6
Changed lines of the file:
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@@
-	)
-	(junction
-		(at 177.8 90.17)
-		(diameter 0)
-		(color 0 0 0 0)
 	)
 	(junction
@@
 	)
 	(no_connect
+		(at 177.8 95.25)
+	)
+	(no_connect
+		(at 162.56 90.17)
+	)
+	(no_connect
 		(at 195.58 121.92)
 	)
@@
 	(wire
 		(pts
+			(xy 137.16 57.15) (xy 137.16 67.31)
+		)
+		(stroke
+			(width 0)
+			(type default)
+		)
+	)
+	(wire
+		(pts
 			(xy 127 57.15) (xy 127 72.39)
 		)
@@
 	(wire
 		(pts
-			(xy 162.56 90.17) (xy 182.88 90.17)
-		)
-		(stroke
-			(width 0)
-			(type default)
-		)
-	)
-	(wire
-		(pts
 			(xy 137.16 57.15) (xy 140.97 57.15)
 		)
@@
 	(wire
 		(pts
-			(xy 137.16 74.93) (xy 133.35 74.93)
-		)
-		(stroke
-			(width 0)
-			(type default)
-		)
-	)
-	(wire
-		(pts
 			(xy 137.16 87.63) (xy 116.84 87.63)
 		)
@@
 	(wire
 		(pts
-			(xy 125.73 74.93) (xy 121.92 74.93)
-		)
-		(stroke
-			(width 0)
-			(type default)
-		)
-	)
-	(wire
-		(pts
-			(xy 177.8 90.17) (xy 177.8 95.25)
+			(xy 121.92 74.93) (xy 137.16 74.93)
 		)
 		(stroke
@@
 		(pts
 			(xy 92.71 50.8) (xy 92.71 57.15)
-		)
-		(stroke
-			(width 0)
-			(type default)
-		)
-	)
-	(wire
-		(pts
-			(xy 137.16 57.15) (xy 137.16 67.31)
 		)
 		(stroke
@@
 			)
 			(justify right bottom)
-		)
-	)
-	(hierarchical_label "FL_INT#"
-		(shape output)
-		(at 182.88 90.17 0)
-		(effects
-			(font
-				(size 1.27 1.27)
-			)
-			(justify left)
 		)
 	)
@@
 	(symbol
 		(lib_id "Device:R")
-		(at 129.54 74.93 90)
-		(unit 1)
-		(body_style 1)
-		(exclude_from_sim no)
-		(in_bom yes)
-		(on_board yes)
-		(in_pos_files yes)
-		(dnp no)
-		(property "Reference" "R509"
-			(at 125.73 67.31 270)
-			(show_name no)
-			(do_not_autoplace no)
-			(effects
-				(font
-					(size 1.27 1.27)
-				)
-				(justify left)
-			)
-		)
-		(property "Value" "0R"
-			(at 125.73 64.77 270)
-			(show_name no)
-			(do_not_autoplace no)
-			(effects
-				(font
-					(size 1.27 1.27)
-				)
-				(justify left)
-			)
-		)
-		(property "Footprint" "Resistor_SMD:R_0402_1005Metric"
-			(at 129.54 74.93 270)
-			(hide yes)
-			(show_name no)
-			(do_not_autoplace no)
-			(effects
-				(font
-					(size 1.27 1.27)
-				)
-			)
-		)
-		(property "Datasheet" ""
-			(at 129.54 74.93 270)
-			(hide yes)
-			(show_name no)
-			(do_not_autoplace no)
-			(effects
-				(font
-					(size 1.27 1.27)
-				)
-			)
-		)
-		(property "Description" "SEL -> IN: I2C address 0x38. Grounded SEL is 0x36, which collides with U2 (MAX17048), whose address is fixed. Drawn as a link so the alternative stays a stuffing option."
-			(at 129.54 74.93 270)
-			(hide yes)
-			(show_name no)
-			(do_not_autoplace no)
-			(effects
-				(font
-					(size 1.27 1.27)
-				)
-			)
-		)
-		(pin "1"
-		)
-		(pin "2"
-		)
-		(instances
-			(project "r2"
-				(path "/dee825bf-c2f1-415d-afdf-cf702072a6e8/5c8ce93f-26c8-4450-ba3a-dff03cacb9ae"
-					(reference "R509")
-					(unit 1)
-				)
-			)
-		)
-	)
-	(symbol
-		(lib_id "Device:R")
 		(at 177.8 99.06 0)
 		(unit 1)
@@
 		(exclude_from_sim no)
 		(in_bom yes)
-		(on_board yes)
+		(on_board no)
 		(in_pos_files yes)
-		(dnp no)
+		(dnp yes)
 		(property "Reference" "R508"
 			(at 180.34 97.79 0)

Commit message: change layout and reduce board size + add second usb host only
Parts:
- J24: footprint footprints:HC-FPC-05-09-8RLTAG -> r2:HC-FPC-05-09-8RLTAG_Mirrored
Changed lines of the file:
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@@
 			)
 		)
-		(property "Footprint" "footprints:HC-FPC-05-09-8RLTAG"
+		(property "Footprint" "r2:HC-FPC-05-09-8RLTAG_Mirrored"
 			(at 200.66 121.92 0)
 			(hide yes)
