File: pcb/r2-mainboard/frontlight.kicad_sch (KiCad schematic)
At the start: 9 parts, among them J24 HC-FPC-05-09-8RLTAG, U53 LM3630A

Commit message: R2: renumber every sheet to the page-based designator scheme
The owner's scheme is classifier + sheet page + two-digit part from 00. Four
sheets already used it; this converts the remaining nine, so all thirteen now
agree: pages 2-9 take three digits, pages 10-14 four. 292 of 333 designators
changed. A part shared by several sheets takes its lowest page, so the FPGA is
U700 (pages 7-9) and the two SoM connectors are J501/J502 (pages 5-6).

The whole risk here is silently rewiring the board, so the netlist was diffed
rather than eyeballed:

  nets 519 -> 519, total pin connections 1563 -> 1563
  named nets present in both whose pin multiset changed: 0
  ERC unchanged at 14 errors / 20 warnings
  check_ucf.py: 99 balls matched, 0 failures

That last one matters most: it resolves the gateware's 113 UCF constraints to
board nets *by ball name*, so it is the sharpest detector of the corruption
this change could cause.

Two earlier attempts did cause exactly that. A bare quoted-string substitution
also rewrites FPGA ball names (C1, D2, N11, T1) and BTH-060 pin names (A1-D60),
which are spelled exactly like designators; one run left ERC identical while 40
nets came back with a different pin multiset. The tool now substitutes only at
the two positions that store an instance's designator, and excludes every pin
name everywhere else. docs/layout.md 9.5 records the hazard and how to prove a
renumber was clean.

Only the three scripts that read the design are updated. The gen_*/patch_*/
port_r1.py scripts keep the old names deliberately: each wrote a sheet once and
has not been re-runnable since it was hand-edited in Eeschema, so they are a
historical record -- and port_r1.py's dict keys are R1 designators that were
never renumbered at all.

Co-Authored-By: Claude Opus 5 <noreply@anthropic.com>
Claude-Session: https://claude.ai/code/session_01MHTAe6ZnhogTEgtyPcLhwG
Parts:
- renumbered C514 to C1300, C515 to C1301, C516 to C1302, D34 to D1300, J24 to J1300, L33 to L1300, R507 to R1300, R508 to R1301, U53 to U1300
Changed lines of the file:
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@@
 		(in_pos_files yes)
 		(dnp no)
-		(property "Reference" "L33"
+		(property "Reference" "L1300"
 			(at 130.81 53.34 270)
 			(show_name no)
@@
 			(project "r2"
 				(path "/dee825bf-c2f1-415d-afdf-cf702072a6e8/5c8ce93f-26c8-4450-ba3a-dff03cacb9ae"
-					(reference "L33")
+					(reference "L1300")
 					(unit 1)
 				)
@@
 		(in_pos_files yes)
 		(dnp no)
-		(property "Reference" "R507"
+		(property "Reference" "R1300"
 			(at 129.54 97.79 0)
 			(show_name no)
@@
 			(project "r2"
 				(path "/dee825bf-c2f1-415d-afdf-cf702072a6e8/5c8ce93f-26c8-4450-ba3a-dff03cacb9ae"
-					(reference "R507")
+					(reference "R1300")
 					(unit 1)
 				)
@@
 		(in_pos_files yes)
 		(dnp no)
-		(property "Reference" "U53"
+		(property "Reference" "U1300"
 			(at 139.7 100.33 0)
 			(show_name no)
@@
 			(project "r2"
 				(path "/dee825bf-c2f1-415d-afdf-cf702072a6e8/5c8ce93f-26c8-4450-ba3a-dff03cacb9ae"
-					(reference "U53")
+					(reference "U1300")
 					(unit 1)
 				)
@@
 		(in_pos_files yes)
 		(dnp no)
-		(property "Reference" "C516"
+		(property "Reference" "C1302"
 			(at 114.3 64.77 0)
 			(show_name no)
@@
 			(project "r2"
 				(path "/dee825bf-c2f1-415d-afdf-cf702072a6e8/5c8ce93f-26c8-4450-ba3a-dff03cacb9ae"
-					(reference "C516")
+					(reference "C1302")
 					(unit 1)
 				)
@@
 		(in_pos_files yes)
 		(dnp no)
-		(property "Reference" "D34"
+		(property "Reference" "D1300"
 			(at 144.78 45.72 0)
 			(show_name no)
@@
 			(project "r2"
 				(path "/dee825bf-c2f1-415d-afdf-cf702072a6e8/5c8ce93f-26c8-4450-ba3a-dff03cacb9ae"
-					(reference "D34")
+					(reference "D1300")
 					(unit 1)
 				)
@@
 		(in_pos_files yes)
 		(dnp no)
-		(property "Reference" "C514"
+		(property "Reference" "C1300"
 			(at 99.06 64.77 0)
 			(show_name no)
@@
 			(project "r2"
 				(path "/dee825bf-c2f1-415d-afdf-cf702072a6e8/5c8ce93f-26c8-4450-ba3a-dff03cacb9ae"
-					(reference "C514")
+					(reference "C1300")
 					(unit 1)
 				)
@@
 		(in_pos_files yes)
 		(dnp yes)
-		(property "Reference" "R508"
+		(property "Reference" "R1301"
 			(at 180.34 97.79 0)
 			(show_name no)
@@
 			(project "r2"
 				(path "/dee825bf-c2f1-415d-afdf-cf702072a6e8/5c8ce93f-26c8-4450-ba3a-dff03cacb9ae"
-					(reference "R508")
+					(reference "R1301")
 					(unit 1)
 				)
@@
 		(in_pos_files yes)
 		(dnp no)
-		(property "Reference" "J24"
+		(property "Reference" "J1300"
 			(at 203.2 109.22 0)
 			(show_name no)
@@
 			(project "r2"
 				(path "/dee825bf-c2f1-415d-afdf-cf702072a6e8/5c8ce93f-26c8-4450-ba3a-dff03cacb9ae"
-					(reference "J24")
+					(reference "J1300")
 					(unit 1)
 				)
@@
 		(in_pos_files yes)
 		(dnp no)
-		(property "Reference" "C515"
+		(property "Reference" "C1301"
 			(at 177.8 64.77 0)
 			(show_name no)
@@
 			(project "r2"
 				(path "/dee825bf-c2f1-415d-afdf-cf702072a6e8/5c8ce93f-26c8-4450-ba3a-dff03cacb9ae"
-					(reference "C515")
-					(unit 1)
-				)
+					(reference "C1301")
+					(unit 1)
+				)
