File: pcb/r2-mainboard/frontlight.kicad_sch (KiCad schematic)
At the start: 9 parts, among them J1300 HC-FPC-05-09-8RLTAG, U1300 LM3630A

Commit message: Schematics update for new chip.
Parts:
- C1300: value 4.7uF/10V -> 4.7uF/25V; footprint Capacitor_SMD:C_0603_1608Metric -> Capacitor_SMD:C_0805_2012Metric
- C1302: value 100nF/16V -> 100nF/50V
- R1300: value 100k -> 100k/1%
- R1301: value 10k -> 10k/1%
Changed lines of the file:
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@@
 			)
 		)
-		(property "Value" "100k"
+		(property "Value" "100k/1%"
 			(at 129.54 101.092 0)
 			(show_name no)
@@
 			)
 		)
-		(property "Value" "100nF/16V"
+		(property "Value" "100nF/50V"
 			(at 114.3 68.072 0)
 			(show_name no)
@@
 			)
 		)
-		(property "Value" "4.7uF/10V"
+		(property "Value" "4.7uF/25V"
 			(at 99.06 68.072 0)
 			(show_name no)
@@
 			)
 		)
-		(property "Footprint" "Capacitor_SMD:C_0603_1608Metric"
+		(property "Footprint" "Capacitor_SMD:C_0805_2012Metric"
 			(at 96.52 66.04 0)
 			(hide yes)
@@
 			)
 		)
-		(property "Value" "10k"
+		(property "Value" "10k/1%"
 			(at 180.34 101.092 0)
 			(show_name no)
