File: pcb/r2-mainboard/r2.kicad_pcb (KiCad board)
At the start: 4 copper layers, 245.3 x 165.7 mm, 324 parts, among them J1 USB-C 16P, J2 Pico-Lock 504050-0391, J20 SWD+JTAG (DNP), J21 MICRO_SD(TFC-WPAPR-08), J22 HC-FPC-05-09-6RLTAG, J23 HC-FPC-05-09-6RLTAG, J24 HC-FPC-05-09-8RLTAG, J25 SolderPads 3x, J26 BTH-060-01-L-D-A-K-TR, J27 BTH-060-01-L-D-A-K-TR, J6 FPC-05F-50PH20, Q1 AO3401A, Q2 S8050, Q6 AO3400A, Q7 AO3401A, Q8 AO3401A, Q9 AO3400A, SW20 SW, SW21 SW, SW22 SW, U1 BQ25892RTW, U10 TPS7A0233DBVR, U12 TPS61022RWUR, U13 TPS63802DLAR, U14 TPS62A02DRLR, U15 TPS62A02DRLR, U2 MAX17048G+T10, U20 STM32G0B1RCT6, U21 INA3221, U22 INA3221, U23 LGS6302B5, U24 LGS6302B5, U26 LGS5145, U27 INA3221, U3 USBLC6-2SC6, U31 LM321, U41 XC6SLX-FTG256, U42 W25Q128JVSIQ, U52 MT41K64M16TW, U53 LM3630A, U54 TPS22914BYFPR, U55 TPS22914BYFPR, U6 MT9700, U7 TPS22914BYFPR, U8 TPS22914BYFPR, U9 LGS5145, X1 33.33MHz, X2 PCM-071, Y20 32.768kHz

Commit message: routing and board layout
Parts:
- removed R508: 10k, Resistor_SMD:R_0402_1005Metric
- removed R509: 0R, Resistor_SMD:R_0402_1005Metric
- C40: footprint Capacitor_SMD:C_0603_1608Metric -> Capacitor_SMD:C_0402_1005Metric; moved to B.Cu
- C41, C43, C44, FB20: moved to B.Cu
- SW20: value SW -> EVQPUC02K; footprint Button_Switch_SMD:SW_Push_1P1T_XKB_TS-1187A -> Button_Switch_SMD:Panasonic_EVQPUL_EVQPUC
- moved J1 231.1 mm to (270.0, 84.2), turned to 90 degrees
- moved D20 230.6 mm to (255.5, 20.0)
- moved SW20 230.1 mm to (264.5, 20.4)
- moved R1 228.5 mm to (267.1, 90.2), turned to 180 degrees
- moved R44 228.1 mm to (258.0, 20.0)
- moved R2 219.5 mm to (265.3, 78.0), turned to 0 degrees
- moved U3 215.7 mm to (262.1, 84.1), turned to 180 degrees
- moved R10 212.8 mm to (259.9, 105.5), turned to 90 degrees
- moved J20 210.9 mm to (268.2, 115.2)
- moved R9 209.3 mm to (257.4, 106.0), turned to 0 degrees
- moved SW22 208.7 mm to (278.0, 144.5)
- moved SW21 208.4 mm to (277.5, 135.5)
- moved C2 208.3 mm to (255.3, 103.5), turned to -90 degrees
- moved F1 207.7 mm to (252.6, 99.0), turned to -90 degrees
- moved C3 207.5 mm to (256.9, 108.0), turned to -90 degrees
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Connections:
- net Net-(C3-Pad2) renamed /battery/CHG_SW
- net Net-(F1-Pad1) renamed /battery/+VBUS_PRE
- net Net-(U13-L1) renamed /power/OSCIL_1
- net Net-(U13-L2) renamed /power/OSCIL_2
- net Net-(U14-SW) renamed /power/1V2_SW
- net Net-(U15-SW) renamed /power/1V5_SW
- J1 pad A6: Net-(J1-D+-PadA6) -> /USBD+
- J1 pad A7: Net-(J1-D--PadA7) -> /USBD-
- J1 pad B6: Net-(J1-D+-PadA6) -> /USBD+
- J1 pad B7: Net-(J1-D--PadA7) -> /USBD-
- U1 pad 24: /battery/CHG_DSEL -> unconnected-(U1-NC/DSEL-Pad24)
- U20 pad 32: /FL_INT# -> unconnected-(U20-PB12-Pad32)
- U3 pad 1: Net-(J1-D--PadA7) -> /USBD-
- U3 pad 3: Net-(J1-D+-PadA6) -> /USBD+
- U53 pad B2: /FL_INT# -> unconnected-(U53-~{INTN}-PadB2)
- U53 pad C2: Net-(U53-SEL) -> +VSYS_FL
Routing:
- net +VBAT: track 55.8 -> 7.75 mm
- net /frontlight/FL_LEDA: track 0.00 -> 26.8 mm, vias 0 -> 2
- net GND: track 53.3 -> 76.0 mm, vias 7 -> 29
- net /frontlight/FL_LED1K: track 0.00 -> 16.8 mm
- net /FPGA_CLK33: track 0.00 -> 12.9 mm, vias 0 -> 2
- net +3V3_AON: track 0.00 -> 11.5 mm, vias 0 -> 2
- net +1V5: track 0.00 -> 11.3 mm, vias 0 -> 3
- net +VSYS_FL: track 0.00 -> 11.1 mm
- net +1V5_DCDC: track 10.5 -> 20.5 mm, vias 2 -> 3
- net /frontlight/FL_LED2K: track 0.00 -> 9.72 mm
- net Net-(D34-A): track 0.00 -> 9.67 mm
- net +1V2_DCDC: track 0.00 -> 8.11 mm
- net /battery/CHG_PSEL: track 0.00 -> 7.11 mm, vias 0 -> 2
- net +1V2_FPGA: track 0.00 -> 6.59 mm, vias 0 -> 3
- net /SOM_MCU_NRST: track 0.00 -> 6.16 mm
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Other:
- board size 245.3 x 165.7 mm -> 230.6 x 135.6 mm

Commit message: placed almost all accessory electronics
Parts:
- C144, C316, C318, C319, C320, C321, C322, C323, C324, C325, C357, C358, C359, C368, C392, C393, C449, C450, C456, C457, C482, C483, C484, C485, C487, C488, C489, C490, C509, C70, C73, C76, C81, C83, C84, C87, C88, R100, R103, R104, R105, R340: moved to B.Cu
- moved J27 101.3 mm to (190.7, 142.1), turned to -90 degrees
- moved R500 88.3 mm to (201.3, 133.7), turned to 180 degrees
- moved C510 85.4 mm to (197.6, 133.2), turned to 180 degrees
- moved C512 85.2 mm to (194.0, 133.8), turned to 180 degrees
- moved R501 84.5 mm to (201.3, 131.8), turned to 180 degrees
- moved R511 84.0 mm to (209.6, 127.8), turned to 180 degrees
- moved R502 80.7 mm to (201.3, 129.8), turned to 180 degrees
- moved C484 80.3 mm to (176.7, 90.5)
- moved C511 79.5 mm to (197.6, 130.2), turned to 180 degrees
- moved C86 79.5 mm to (172.0, 79.8), turned to -90 degrees
- moved X2 79.3 mm to (193.1, 130.9), turned to -90 degrees
- moved C70 79.1 mm to (177.2, 89.2)
- moved C85 78.7 mm to (171.0, 82.0)
- moved C321 77.5 mm to (169.7, 99.2), turned to -90 degrees
- moved R510 77.4 mm to (208.6, 124.6), turned to 180 degrees
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Routing:
- net /FPGA_CLK33: track 12.9 -> 3.41 mm, vias 2 -> 1
- net +1V2_FPGA: track 6.59 -> 13.0 mm
- net GND: track 76.0 -> 80.6 mm, vias 29 -> 19
- net +3V3: track 3.31 -> 7.29 mm, vias 0 -> 13
- added copper zone on In1.Cu, net +3V3
- added copper zone on In2.Cu, net GND
- removed copper zone on In1.Cu, net GND

Commit message: change layout and reduce board size + add second usb host only
Parts:
- removed C147: 100nF/50V, Capacitor_SMD:C_0402_1005Metric
- added C519: 100nF/50V, Capacitor_SMD:C_0402_1005Metric, F.Cu at (256.6, 149.5)
- added C520: 22uF/10V, Capacitor_SMD:C_0805_2012Metric, F.Cu at (257.4, 147.0)
- added C521: 100nF/50V, Capacitor_SMD:C_0402_1005Metric, F.Cu at (256.6, 151.4)
- added J28: USB-C 16P, Connector_USB:USB_C_Receptacle_HRO_TYPE-C-31-M-12, F.Cu at (270.0, 101.0)
- added R520: 56k, Resistor_SMD:R_0402_1005Metric, F.Cu at (253.7, 146.5)
- added R521: 56k, Resistor_SMD:R_0402_1005Metric, F.Cu at (253.7, 148.5)
- added R522: 49.9k/1%, Resistor_SMD:R_0402_1005Metric, F.Cu at (253.7, 150.4)
- added R523: 100k, Resistor_SMD:R_0402_1005Metric, F.Cu at (253.7, 152.4)
- added U56: TPS2553DBVR, Package_TO_SOT_SMD:SOT-23-6, F.Cu at (266.5, 137.4)
- added U57: USBLC6-2SC6, Package_TO_SOT_SMD:SOT-23-6, F.Cu at (266.5, 142.0)
- J24: footprint footprints:HC-FPC-05-09-8RLTAG -> r2:HC-FPC-05-09-8RLTAG_Mirrored; moved to B.Cu
- J6: value FPC-05F-50PH20 -> XF2M-4015-1A; footprint footprints:Xunpu_FPC-05F-50PH20_1x50-1MP_P0.50mm_Horizontal -> r2:Omron_XF2M-4015-1A_1x40-1MP_P0.5mm_Horizontal_Mirrored; moved to B.Cu
- moved J2 197.3 mm to (240.2, 121.0)
- moved J25 197.2 mm to (251.8, 122.0)
- moved U31 196.9 mm to (221.7, 45.2)
- moved R66 195.4 mm to (228.4, 45.8), turned to 90 degrees
- moved D5 195.4 mm to (222.7, 41.5)
- moved R65 194.5 mm to (226.9, 43.0), turned to 180 degrees
- moved Q8 193.7 mm to (225.9, 45.2), turned to 180 degrees
- moved R64 191.8 mm to (224.9, 43.0), turned to 180 degrees
- moved R63 191.3 mm to (228.4, 49.2), turned to -90 degrees
- moved Q7 190.5 mm to (225.9, 48.8), turned to 180 degrees
- moved D15 189.6 mm to (209.2, 40.2), turned to 180 degrees
- moved U26 188.5 mm to (215.4, 46.8)
- moved R227 186.2 mm to (220.2, 41.5), turned to 90 degrees
- moved Q6 184.8 mm to (221.7, 48.8), turned to 180 degrees
- moved R226 182.8 mm to (218.9, 44.0), turned to 90 degrees
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Connections:
- J26 pad B39: unconnected-(J26D-X_USB1_DM-PadB39) -> /USB1_DM
- J26 pad B40: unconnected-(J26D-X_USB1_DP-PadB40) -> /USB1_DP
- J26 pad B41: unconnected-(J26D-X_USB1_VBUS-PadB41) -> /USB1_VBUS
- J26 pad B42: unconnected-(J26D-X_USB1_DRVVBUS-PadB42) -> /USB1_DRVVBUS
- J6 pad 10: /EPDC_SDCE0 -> -VCOM
- J6 pad 11: /EPDC_GDOE -> +3V3
- J6 pad 12: /EPDC_GDSP -> GND
- J6 pad 13: /EPDC_GDCLK -> /EPDC_SE_CLK
- J6 pad 14: GND -> /EPDC_D0P
- J6 pad 15: /EPDC_SE_CLK -> /EPDC_D0N
- J6 pad 16: GND -> /EPDC_D1P
- J6 pad 17: /EPDC_D7N -> /EPDC_D1N
- J6 pad 18: /EPDC_D7P -> /EPDC_D2P
- J6 pad 19: GND -> /EPDC_D2N
- J6 pad 20: /EPDC_D6N -> /EPDC_D3P
- J6 pad 21: /EPDC_D6P -> /EPDC_D3N
- J6 pad 23: /EPDC_D5N -> /EPDC_D4P
- J6 pad 24: /EPDC_D5P -> /EPDC_D4N
- J6 pad 25: GND -> /EPDC_D5P
- J6 pad 26: /EPDC_D4N -> /EPDC_D5N
- J6 pad 27: /EPDC_D4P -> /EPDC_D6P
- J6 pad 28: GND -> /EPDC_D6N
- J6 pad 29: /EPDC_D3N -> /EPDC_D7P
- J6 pad 30: /EPDC_D3P -> /EPDC_D7N
- J6 pad 31: GND -> /EPDC_SDCE0
- J6 pad 32: /EPDC_D2N -> /EPDC_SDLE
- J6 pad 33: /EPDC_D2P -> /EPDC_SDOE
- J6 pad 34: GND -> unconnected-(J6-Pin_34-Pad34)
- J6 pad 35: /EPDC_D1N -> unconnected-(J6-Pin_35-Pad35)
- J6 pad 36: /EPDC_D1P -> +VP
- J6 pad 37: GND -> unconnected-(J6-Pin_37-Pad37)
- J6 pad 38: /EPDC_D0N -> -VN
- J6 pad 39: /EPDC_D0P -> unconnected-(J6-Pin_39-Pad39)
- J6 pad 40: GND -> -VCOM
- J6 pad 5: -VCOM -> +3V3
- J6 pad 6: +3V3 -> /EPDC_GDOE
- J6 pad 7: +5V2_FL -> /EPDC_GDCLK
- J6 pad 8: /EPDC_SDOE -> /EPDC_GDSP
- J6 pad 9: /EPDC_SDLE -> GND
- U20 pad 61: /FL_PWM2 -> /USB1_FAULT#
Routing:
- net /frontlight/FL_LEDA: track 26.8 -> 9.50 mm
- net /frontlight/FL_LED1K: track 16.8 -> 0.00 mm
- net /frontlight/FL_LED2K: track 9.72 -> 0.00 mm
- net +1V5: track 11.3 -> 3.00 mm, vias 3 -> 0
- net +1V5_DCDC: track 20.5 -> 13.4 mm
- net +1V2_FPGA: track 13.0 -> 8.91 mm, vias 3 -> 0
- net GND: track 80.6 -> 76.7 mm, vias 19 -> 20
- net /FPGA_CLK33: track 3.41 -> 0.00 mm, vias 1 -> 0
- net /battery/USB_CC1: track 6.99 -> 10.4 mm
- net /FPGA_DONE: track 0.00 -> 3.06 mm
- net +1V2_DCDC: track 8.11 -> 5.20 mm
- net /FPGA_SUSP: track 0.00 -> 2.85 mm
- net /FPGA_PROG#: track 0.00 -> 2.60 mm
- net /FPGA_INIT: track 0.00 -> 2.09 mm
- net +VBUS: track 4.68 -> 6.74 mm
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- removed copper zone on F.Cu, net GND
- removed copper zone on F.Cu, net Net-(U12-SW)
Other:
- board size 230.6 x 135.6 mm -> 88.2 x 106.2 mm
- board text added: "EPD"
- board text added: "VCOM"
- board text added: "VGH"
- board text added: "VGL"
- board text added: "VN"
- board text added: "VP"
