File: pcb/r2-mainboard/r2.kicad_pcb (KiCad board)
At the start: 4 copper layers, 85.5 x 82.8 mm, 328 parts, among them J20 SWD+JTAG (DNP), J200 USB-C 16P, J201 Pico-Lock 504050-0391, J202 SolderPads 3x, J21 MICRO_SD(TFC-WPAPR-08), J22 HC-FPC-05-09-6RLTAG, J24 HC-FPC-05-09-8RLTAG, J26 BTH-060-01-L-D-A-K-TR, J27 BTH-060-01-L-D-A-K-TR, J28 USB-C 16P, J6 XF2M-4015-1A, Q1 AO3401A, Q2 S8050, Q6 AO3400A, Q7 AO3401A, Q8 AO3401A, Q9 AO3400A, SW20 EVQPUC02K, SW21 SW, SW22 SW, U20 STM32G0B1RCT6, U200 BQ25892RTW, U201 MAX17048G+T10, U21 INA3221, U22 INA3221, U23 LGS6302B5, U24 LGS6302B5, U26 LGS5145, U27 INA3221, U3 USBLC6-2SC6, U300 TPS7A0233DBVR, U301 TPS61022RWUR, U302 TPS63802DLAR, U303 TPS62A02DRLR, U304 TPS62A02DRLR, U31 LM321, U41 XC6SLX-FTG256, U52 MT41K64M16TW, U53 LM3630A, U54 TPS22914BYFPR, U56 TPS2553DBVR, U57 USBLC6-2SC6, U6 MT9700, U7 TPS22914BYFPR, U8 TPS22914BYFPR, U9 LGS5145, U902 W25Q128JVSIQ, X1 33.33MHz, X2 PCM-071, Y20 32.768kHz

Commit message: Renumber io_expansion to the page-14 scheme
The owner's designator scheme is classifier + sheet page number + a
two-digit part number, counted from 00 -- battery (page 2) is U200/J201,
power (page 3) is U300-U304, fpga_config (page 9) is U902. Pages 10-14
therefore need four digits, which the owner confirmed.

io_expansion is page 14:

  U54  -> U1400   touch load switch      J22  -> J1400   touch FPC
  U55  -> U1401   pen load switch        J23  -> J1401   pen FPC
  U56  -> U1402   TPS2553 USB switch     J28  -> J1402   USB-C host
  U57  -> U1403   USBLC6 ESD
  R520 -> R1400   CC1 pull-up            C517 -> C1400   touch rail
  R521 -> R1401   CC2 pull-up            C518 -> C1401   pen rail
  R522 -> R1402   ILIM                   C519 -> C1402   TPS2553 IN
  R523 -> R1403   FAULT pull-up          C520 -> C1403   VBUS bulk
                                         C521 -> C1404   VBUS bypass

Applied to io_expansion.kicad_sch and r2.kicad_pcb by quoted-string
match, and to the docs and tools/ by word boundary so R52 could never
eat R520. All sixteen target designators were checked free first.

Verified: 519 nets before and after, and *no* net membership changed --
the only differences are the five auto-generated names that embed a
designator (Net-(J28-CC1) -> Net-(J1402-CC1) and friends). ERC unchanged
at 14 errors / 20 warnings. Schematic and board designators agree in
both directions.

The scheme is now recorded in CLAUDE.md, including the warning that
check_pcb.py and check_ucf.py still assert on legacy names.

Co-Authored-By: Claude Opus 5 <noreply@anthropic.com>
Claude-Session: https://claude.ai/code/session_01MHTAe6ZnhogTEgtyPcLhwG
Parts:
- renumbered C517 to C1400, C519 to C1402, C520 to C1403, C521 to C1404, J22 to J1400, J28 to J1402, R520 to R1400, R521 to R1401, R522 to R1402, R523 to R1403, U54 to U1400, U56 to U1402, U57 to U1403
Changed lines of the file:
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@@
 		(descr "Resistor SMD 0402 (1005 Metric), square (rectangular) end terminal, IPC-7351 nominal, (Body size source: IPC-SM-782 page 72, https://www.pcb-3d.com/wordpress/wp-content/uploads/ipc-sm-782a_amendment_1_and_2.pdf)")
 		(tags "resistor")
-		(property "Reference" "R522"
+		(property "Reference" "R1402"
 			(at 0 -1.17 0)
 			(layer "F.SilkS")
@@
 		(descr "Resistor SMD 0402 (1005 Metric), square (rectangular) end terminal, IPC-7351 nominal, (Body size source: IPC-SM-782 page 72, https://www.pcb-3d.com/wordpress/wp-content/uploads/ipc-sm-782a_amendment_1_and_2.pdf)")
 		(tags "resistor")
-		(property "Reference" "R523"
+		(property "Reference" "R1403"
 			(at 0 -1.17 0)
 			(layer "F.SilkS")
@@
 		(descr "Capacitor SMD 0402 (1005 Metric), square (rectangular) end terminal, IPC-7351 nominal, (Body size source: IPC-SM-782 page 76, https://www.pcb-3d.com/wordpress/wp-content/uploads/ipc-sm-782a_amendment_1_and_2.pdf)")
 		(tags "capacitor")
-		(property "Reference" "C517"
+		(property "Reference" "C1400"
 			(at 0 -1.16 0)
 			(layer "F.SilkS")
@@
 		(descr "Capacitor SMD 0805 (2012 Metric), square (rectangular) end terminal, IPC-7351 nominal, (Body size source: IPC-SM-782 page 76, https://www.pcb-3d.com/wordpress/wp-content/uploads/ipc-sm-782a_amendment_1_and_2.pdf, https://docs.google.com/spreadsheets/d/1BsfQQcO9C6DZCsRaXUlFlo91Tg2WpOkGARC1WS5S8t0/edit?usp=sharing)")
 		(tags "capacitor")
-		(property "Reference" "C520"
+		(property "Reference" "C1403"
 			(at 0 -1.68 90)
 			(layer "F.SilkS")
@@
 		(descr "WLP-4_0.83x0.83mm_P0.4mm https://pdfserv.maximintegrated.com/package_dwgs/21-100107.PDF, https://www.maximintegrated.com/en/app-notes/index.mvp/id/1891")
 		(tags "WLP-4")
-		(property "Reference" "U54"
+		(property "Reference" "U1400"
 			(at 0 -2.25 90)
 			(layer "F.SilkS")
@@
 		(descr "SOT, 6 Pin (JEDEC MO-178 Var AB https://www.jedec.org/document_search?search_api_views_fulltext=MO-178)")
 		(tags "SOT TO_SOT_SMD")
-		(property "Reference" "U56"
+		(property "Reference" "U1402"
 			(at 0 -2.4 0)
 			(layer "F.SilkS")
@@
 		(descr "USB Type-C receptacle for USB 2.0 and PD, http://www.krhro.com/uploads/soft/180320/1-1P320120243.pdf")
 		(tags "usb usb-c 2.0 pd")
-		(property "Reference" "J28"
+		(property "Reference" "J1402"
 			(at 0 -6.145 90)
 			(layer "F.SilkS")
@@
 		(descr "Hirose FH12, FFC/FPC connector, FH12-8S-0.5SH, 8 Pins per row (https://www.hirose.com/product/en/products/FH12/FH12-24S-0.5SH(55)/), generated with kicad-footprint-generator")
 		(tags "connector Hirose FH12 horizontal")
-		(property "Reference" "J22"
+		(property "Reference" "J1400"
 			(at 0 -3.7 90)
 			(layer "F.SilkS")
@@
 		(descr "SOT, 6 Pin (JEDEC MO-178 Var AB https://www.jedec.org/document_search?search_api_views_fulltext=MO-178)")
 		(tags "SOT TO_SOT_SMD")
-		(property "Reference" "U57"
+		(property "Reference" "U1403"
 			(at 1.5 2.75 0)
 			(layer "F.SilkS")
@@
 		(descr "Capacitor SMD 0402 (1005 Metric), square (rectangular) end terminal, IPC-7351 nominal, (Body size source: IPC-SM-782 page 76, https://www.pcb-3d.com/wordpress/wp-content/uploads/ipc-sm-782a_amendment_1_and_2.pdf)")
 		(tags "capacitor")
-		(property "Reference" "C521"
+		(property "Reference" "C1404"
 			(at 0 -1.16 90)
 			(layer "F.SilkS")
@@
 		(descr "Resistor SMD 0402 (1005 Metric), square (rectangular) end terminal, IPC-7351 nominal, (Body size source: IPC-SM-782 page 72, https://www.pcb-3d.com/wordpress/wp-content/uploads/ipc-sm-782a_amendment_1_and_2.pdf)")
 		(tags "resistor")
-		(property "Reference" "R521"
+		(property "Reference" "R1401"
 			(at 0 -1.17 0)
 			(layer "F.SilkS")
@@
 		(descr "Capacitor SMD 0402 (1005 Metric), square (rectangular) end terminal, IPC-7351 nominal, (Body size source: IPC-SM-782 page 76, https://www.pcb-3d.com/wordpress/wp-content/uploads/ipc-sm-782a_amendment_1_and_2.pdf)")
 		(tags "capacitor")
-		(property "Reference" "C519"
+		(property "Reference" "C1402"
 			(at 0 -1.16 90)
 			(layer "F.SilkS")
@@
 		(descr "Resistor SMD 0402 (1005 Metric), square (rectangular) end terminal, IPC-7351 nominal, (Body size source: IPC-SM-782 page 72, https://www.pcb-3d.com/wordpress/wp-content/uploads/ipc-sm-782a_amendment_1_and_2.pdf)")
 		(tags "resistor")
-		(property "Reference" "R520"
+		(property "Reference" "R1400"
 			(at 0 -1.17 0)
 			(layer "F.SilkS")

Commit message: R2: renumber every sheet to the page-based designator scheme
The owner's scheme is classifier + sheet page + two-digit part from 00. Four
sheets already used it; this converts the remaining nine, so all thirteen now
agree: pages 2-9 take three digits, pages 10-14 four. 292 of 333 designators
changed. A part shared by several sheets takes its lowest page, so the FPGA is
U700 (pages 7-9) and the two SoM connectors are J501/J502 (pages 5-6).

The whole risk here is silently rewiring the board, so the netlist was diffed
rather than eyeballed:

  nets 519 -> 519, total pin connections 1563 -> 1563
  named nets present in both whose pin multiset changed: 0
  ERC unchanged at 14 errors / 20 warnings
  check_ucf.py: 99 balls matched, 0 failures

That last one matters most: it resolves the gateware's 113 UCF constraints to
board nets *by ball name*, so it is the sharpest detector of the corruption
this change could cause.

Two earlier attempts did cause exactly that. A bare quoted-string substitution
also rewrites FPGA ball names (C1, D2, N11, T1) and BTH-060 pin names (A1-D60),
which are spelled exactly like designators; one run left ERC identical while 40
nets came back with a different pin multiset. The tool now substitutes only at
the two positions that store an instance's designator, and excludes every pin
name everywhere else. docs/layout.md 9.5 records the hazard and how to prove a
renumber was clean.

Only the three scripts that read the design are updated. The gen_*/patch_*/
port_r1.py scripts keep the old names deliberately: each wrote a sheet once and
has not been re-runnable since it was hand-edited in Eeschema, so they are a
historical record -- and port_r1.py's dict keys are R1 designators that were
never renumbered at all.

Co-Authored-By: Claude Opus 5 <noreply@anthropic.com>
Claude-Session: https://claude.ai/code/session_01MHTAe6ZnhogTEgtyPcLhwG
Parts:
- renumbered C60 to C1000, C61 to C1001, C62 to C1002, C63 to C1003, C158 to C1004, C159 to C1005, C17 to C1100, C35 to C1101, C37 to C1102, C38 to C1103, C51 to C1104, C52 to C1105, C53 to C1106, C54 to C1107, C56 to C1108, C104 to C1109, C160 to C1110, C165 to C1111, C166 to C1112, C167 to C1113, C171 to C1114, C172 to C1115, C173 to C1116, C174 to C1117, C175 to C1118, C176 to C1119, C177 to C1120, C178 to C1121, C232 to C1122, C233 to C1123, C241 to C1124, C242 to C1125, C244 to C1126, C245 to C1127, C246 to C1128, C249 to C1129, C91 to C1200, C141 to C1201, C142 to C1202, C143 to C1203, C163 to C1204, C164 to C1205, C168 to C1206, C169 to C1207, C514 to C1300, C515 to C1301, C516 to C1302, C1 to C200, C2 to C201, C3 to C202, C4 to C203, C5 to C204, C6 to C205, C7 to C206, C8 to C207, C20 to C300, C21 to C301, C22 to C302, C25 to C303, C26 to C304, C27 to C305, C28 to C306, C29 to C307, C30 to C308, C31 to C309, C32 to C310, C33 to C311, C34 to C312, C40 to C400, C41 to C401, C43 to C402, C44 to C403, C45 to C404, C46 to C405, C47 to C406, C48 to C407, C49 to C408, C50 to C409, C69 to C800, C70 to C801, C71 to C802, C72 to C803, C73 to C804, C74 to C805, C75 to C806, C76 to C807, C77 to C808, C78 to C809, C79 to C810, C80 to C811, C81 to C812, C82 to C813, C83 to C814, C84 to C815, C85 to C816, C86 to C817, C87 to C818, C88 to C819, C144 to C820, C318 to C821, C319 to C822, C320 to C823, C321 to C824, C322 to C825, C323 to C826, C324 to C827, C325 to C828, C357 to C829, C358 to C830, C359 to C831, C368 to C832, C509 to C833, C316 to C900, C326 to C901, C392 to C902, C393 to C903, C448 to C904, C449 to C905, C450 to C906, C456 to C907, C457 to C908, C482 to C909, C483 to C910, C484 to C911, C485 to C912, C486 to C913, C487 to C914, C488 to C915, C489 to C916, C490 to C917, C507 to C918, C508 to C919, D1 to D1100, D2 to D1101, D3 to D1102, D4 to D1103, D5 to D1104, D6 to D1105, D15 to D1106, D17 to D1107, D34 to D1300, D7 to D200, D20 to D400, D308 to D700, F1 to F200, FB20 to FB400, J6 to J1000, J24 to J1300, J20 to J400, J21 to J500, J26 to J501, J27 to J502, L5 to L1100, L6 to L1101, L30 to L1102, L32 to L1103, L33 to L1300, L1 to L200, L10 to L300, L11 to L301, L12 to L302, L13 to L303, Q1 to Q1100, Q2 to Q1101, Q6 to Q1102, Q7 to Q1103, Q8 to Q1104, Q9 to Q400, R62 to R1100, R63 to R1101, R64 to R1102, R65 to R1103, R66 to R1104, R78 to R1105, R79 to R1106, R88 to R1107, R89 to R1108, R92 to R1109, R93 to R1110, R94 to R1111, R213 to R1112, R217 to R1113, R218 to R1114, R219 to R1115, R224 to R1116, R225 to R1117, R226 to R1118, R227 to R1119, R228 to R1120, R229 to R1121, R230 to R1122, R234 to R1123, R50 to R1200, R51 to R1201, R53 to R1202, R54 to R1203, R56 to R1204, R60 to R1205, R61 to R1206, R72 to R1207, R87 to R1208, R96 to R1209, R97 to R1210, R98 to R1211, R115 to R1212, R116 to R1213, R117 to R1214, R118 to R1215, R207 to R1216, R208 to R1217, R507 to R1300, R1 to R200, R2 to R201, R3 to R202, R4 to R203, R5 to R204, R6 to R205, R7 to R206, R8 to R207, R9 to R208, R10 to R209, R11 to R210, R12 to R211, R13 to R212, R17 to R213, R18 to R214, R19 to R215, R37 to R216, R38 to R217, R20 to R300, R21 to R301, R22 to R302, R23 to R303, R24 to R304, R25 to R305, R26 to R306, R27 to R307, R28 to R308, R29 to R309, R30 to R310, R31 to R311, R32 to R312, R33 to R313, R34 to R314, R35 to R315, R36 to R316, R40 to R400, R41 to R401, R42 to R402, R43 to R403, R44 to R404, R45 to R405, R510 to R406, R511 to R407, R512 to R408, R311 to R700, R100 to R800, R101 to R801, R102 to R802, R103 to R803, R104 to R804, R105 to R805, R340 to R806, R344 to R807, R335 to R900, R336 to R901, R337 to R902, R409 to R903, R410 to R904, R411 to R905, R412 to R906, R413 to R907, R414 to R908, SW20 to SW400, SW21 to SW401, SW22 to SW402, U6 to U1100, U7 to U1101, U8 to U1102, U9 to U1103, U23 to U1104, U24 to U1105, U26 to U1106, U31 to U1107, U21 to U1200, U22 to U1201, U27 to U1202, U53 to U1300, U3 to U202, U20 to U400, U41 to U700, U52 to U800, X2 to X500, X1 to X900, Y20 to Y400
