File: pcb/r2-mainboard/r2.kicad_pcb (KiCad board)
At the start: 4 copper layers, 85.5 x 82.8 mm, 328 parts, among them J1000 XF2M-4015-1A, J1300 HC-FPC-05-09-8RLTAG, J1400 HC-FPC-05-09-6RLTAG, J1402 USB-C 16P, J200 USB-C 16P, J201 Pico-Lock 504050-0391, J202 SolderPads 3x, J400 SWD+JTAG (DNP), J500 MICRO_SD(TFC-WPAPR-08), J501 BTH-060-01-L-D-A-K-TR, J502 BTH-060-01-L-D-A-K-TR, Q1100 AO3401A, Q1101 S8050, Q1102 AO3400A, Q1103 AO3401A, Q1104 AO3401A, Q400 AO3400A, SW400 EVQPUC02K, SW401 SW, SW402 SW, U1100 MT9700, U1101 TPS22914BYFPR, U1102 TPS22914BYFPR, U1103 LGS5145, U1104 LGS6302B5, U1105 LGS6302B5, U1106 LGS5145, U1107 LM321, U1200 INA3221, U1201 INA3221, U1202 INA3221, U1300 LM3630A, U1400 TPS22914BYFPR, U1402 TPS2553DBVR, U1403 USBLC6-2SC6, U200 BQ25892RTW, U201 MAX17048G+T10, U202 USBLC6-2SC6, U300 TPS7A0233DBVR, U301 TPS61022RWUR, U302 TPS63802DLAR, U303 TPS62A02DRLR, U304 TPS62A02DRLR, U400 STM32G0B1RCT6, U700 XC6SLX-FTG256, U800 MT41K64M16TW, U902 W25Q128JVSIQ, X500 PCM-071, X900 33.33MHz, Y400 32.768kHz

Commit message: routing
Parts:
- C804: moved to F.Cu
- C817, R405: moved to B.Cu
- moved C904 38.6 mm to (187.9, 71.8)
- moved L304 22.9 mm to (191.0, 41.9), turned to 90 degrees
- moved C312 22.3 mm to (194.6, 39.8), turned to 0 degrees
- moved C802 20.8 mm to (187.4, 74.9), turned to 90 degrees
- moved R314 19.3 mm to (197.4, 40.8), turned to 180 degrees
- moved U304 19.1 mm to (194.5, 42.5), turned to 0 degrees
- moved R313 17.9 mm to (197.4, 41.9), turned to 180 degrees
- moved C818 17.7 mm to (187.1, 77.6), turned to -90 degrees
- moved C803 17.6 mm to (187.4, 77.1), turned to -90 degrees
- moved R804 17.0 mm to (188.5, 76.5), turned to -90 degrees
- moved C311 16.6 mm to (194.5, 44.6), turned to 0 degrees
- moved C816 16.4 mm to (187.4, 87.8), turned to -90 degrees
- moved R802 16.4 mm to (187.1, 78.6), turned to 180 degrees
- moved C811 16.2 mm to (199.1, 76.5), turned to 90 degrees
- moved R316 16.2 mm to (197.4, 43.1), turned to 180 degrees
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- renumbered L300 to L301, L301 to L302, L302 to L303, L303 to L304
Connections:
- net Net-(D15-A) renamed /epd_power/SW_VP
- net Net-(D2-A) renamed /epd_power/SW_VGH
- net Net-(U23-FB) renamed /epd_power/FB_VP
- net Net-(U24-FB) renamed /epd_power/FB_VGH
- net Net-(U26-FB) renamed /epd_power/FB_-VN
- C1400 pad 1: Net-(U54-OUT) -> /io_expansion/+3V3_TOUCH
- J1402 pad A6: /io_expansion/USB1_D+ -> /USB1_D+
- J1402 pad A7: /io_expansion/USB1_D- -> /USB1_D-
- J1402 pad B6: /io_expansion/USB1_D+ -> /USB1_D+
- J1402 pad B7: /io_expansion/USB1_D- -> /USB1_D-
- J501 pad B39: /USB1_DM -> /USB1_D-
- J501 pad B40: /USB1_DP -> /USB1_D+
- R1213 pad 2: +3V3_DCDC -> +3V3_AON
- R1215 pad 2: +3V3_DCDC -> +3V3_AON
- U1400 pad A1: Net-(U54-OUT) -> /io_expansion/+3V3_TOUCH
- U1403 pad 1: /io_expansion/USB1_D- -> /USB1_D-
- U1403 pad 3: /io_expansion/USB1_D+ -> /USB1_D+
- U1403 pad 4: /io_expansion/USB1_+ -> /USB1_D+
- U1403 pad 6: /io_expansion/USB1_D- -> /USB1_D-
- U800 pad A2: /fpga_ddr/DRAM_DATA13 -> /fpga_ddr/DRAM_DATA10
- U800 pad A3: /fpga_ddr/DRAM_DATA15 -> /fpga_ddr/DRAM_DATA11
- U800 pad A7: /fpga_ddr/DRAM_DATA12 -> /fpga_ddr/DRAM_DATA15
- U800 pad C2: /fpga_ddr/DRAM_DATA11 -> /fpga_ddr/DRAM_DATA9
- U800 pad C3: /fpga_ddr/DRAM_DATA9 -> /fpga_ddr/DRAM_DATA12
- U800 pad C8: /fpga_ddr/DRAM_DATA10 -> /fpga_ddr/DRAM_DATA13
Routing:
- net GND: track 74.6 -> 212.0 mm, vias 22 -> 127
- net -VN: track 0.00 -> 108.2 mm, vias 0 -> 7
- net +5V_EPD: track 0.00 -> 96.9 mm, vias 0 -> 6
- net +5V_DCDC: track 10.1 -> 102.4 mm, vias 0 -> 6
- net /VCOM_EN: track 0.00 -> 90.6 mm, vias 0 -> 2
- net /VCOM_MEA_EN: track 0.00 -> 87.6 mm, vias 0 -> 2
- net -VGL: track 0.00 -> 80.5 mm, vias 0 -> 4
- net /EPD_PWR_EN: track 0.00 -> 80.4 mm, vias 0 -> 3
- net +3V3: track 7.29 -> 84.4 mm, vias 10 -> 20
- net /MCU_EN_3V3: track 1.92 -> 71.9 mm, vias 0 -> 2
- net +1V5: track 0.00 -> 67.0 mm, vias 0 -> 23
- net /VGH_DAC: track 0.00 -> 65.7 mm, vias 0 -> 2
- net +VP: track 0.00 -> 63.3 mm, vias 0 -> 5
- net /VCOM_DAC: track 0.00 -> 61.1 mm, vias 0 -> 2
- net +3V3_AON: track 6.47 -> 62.8 mm, vias 1 -> 12
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- added copper zone on In2.Cu, net +1V5
- added copper zone on In2.Cu, net +3V3
- added copper zone on In2.Cu, net +3V3_AON
- added copper zone on In1.Cu, net GND
- removed copper zone on In1.Cu, net +3V3
- removed copper zone on In2.Cu, net GND
Other:
- board size 85.5 x 82.8 mm -> 89.8 x 82.8 mm
- copper layers 4 -> 6

Commit message: changing to osb62x-pm
Parts:
- added IC1: OSD6254-1G-IPM, Reflow:BGA500C50P28X18_1400X900X130, F.Cu at (254.0, 69.5)
- moved J501 202.1 mm to (41.0, 69.2)
- moved X500 202.1 mm to (52.2, 71.7)
- moved J502 202.1 mm to (63.4, 74.0)
- moved C510 200.2 mm to (56.5, 75.9)
- moved Q400 200.2 mm to (48.8, 68.0)
- moved R406 200.2 mm to (47.8, 65.0)
- moved R407 200.2 mm to (51.1, 64.0)
- moved R500 200.2 mm to (57.0, 72.2)
- moved R502 200.2 mm to (53.0, 72.2)
- moved R503 200.2 mm to (51.0, 72.2)
- moved C511 200.2 mm to (53.5, 75.9)
- moved C512 200.2 mm to (57.0, 79.6)
- moved C513 200.2 mm to (50.5, 75.9)
- moved R501 200.2 mm to (55.0, 72.2)
- moved R504 200.2 mm to (49.0, 72.2)
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Connections:
- U800 pad C3: /fpga_ddr/DRAM_DATA12 -> /fpga_ddr/DRAM_DATA8
- U800 pad C8: /fpga_ddr/DRAM_DATA13 -> /fpga_ddr/DRAM_DATA12
- U800 pad D7: /fpga_ddr/DRAM_DATA8 -> /fpga_ddr/DRAM_DATA13
- U800 pad F7: /fpga_ddr/DRAM_DATA1 -> /fpga_ddr/DRAM_DATA7
- U800 pad F8: /fpga_ddr/DRAM_DATA3 -> /fpga_ddr/DRAM_DATA1
- U800 pad G2: /fpga_ddr/DRAM_DATA6 -> /fpga_ddr/DRAM_DATA3
- U800 pad H3: /fpga_ddr/DRAM_DATA4 -> /fpga_ddr/DRAM_DATA6
- U800 pad H7: /fpga_ddr/DRAM_DATA7 -> /fpga_ddr/DRAM_DATA5
- U800 pad H8: /fpga_ddr/DRAM_DATA5 -> /fpga_ddr/DRAM_DATA4
Routing:
- net +5V_DCDC: track 102.4 -> 10.8 mm, vias 6 -> 0
- net /VCOM_MEA: track 7.51 -> 84.0 mm, vias 0 -> 2
- net /VCOM_DAC: track 61.1 -> 2.59 mm, vias 2 -> 1
- net /VN_MEA: track 45.0 -> 2.96 mm, vias 2 -> 1
- net /VP_MEA: track 56.6 -> 21.0 mm, vias 1 -> 2
- net +3V3_DCDC: track 36.9 -> 5.48 mm
- net /SDA_AON: track 4.88 -> 34.7 mm, vias 1 -> 2
- net /SCL_AON: track 6.03 -> 33.0 mm, vias 1 -> 2
- net +1V5_DCDC: track 37.2 -> 10.5 mm, vias 3 -> 2
- net +5V_EPD: track 96.9 -> 70.4 mm
- net /fpga_ddr/DRAM_LDM: track 0.00 -> 20.0 mm, vias 0 -> 2
- net /fpga_ddr/DRAM_CKP: track 3.83 -> 23.3 mm, vias 1 -> 2
- net /fpga_ddr/DRAM_CKN: track 2.29 -> 21.7 mm, vias 1 -> 2
- net /fpga_ddr/DRAM_UDM: track 0.75 -> 20.1 mm
- net /fpga_ddr/DRAM_DATA4: track 0.66 -> 19.1 mm, vias 0 -> 2
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- added copper zone on In2.Cu, net +1V2_FPGA
- added copper zone on F.Cu, net +VBAT
- added copper zone on In2.Cu, net +VSYS
- added copper zone on F.Cu, net GND
- added copper zone on In4.Cu, net GND
