File: pcb/r2-mainboard/epd.kicad_sch (KiCad schematic)
At the start: 7 parts, among them J6 XF2M-4015-1A

Commit message: R2: renumber every sheet to the page-based designator scheme
The owner's scheme is classifier + sheet page + two-digit part from 00. Four
sheets already used it; this converts the remaining nine, so all thirteen now
agree: pages 2-9 take three digits, pages 10-14 four. 292 of 333 designators
changed. A part shared by several sheets takes its lowest page, so the FPGA is
U700 (pages 7-9) and the two SoM connectors are J501/J502 (pages 5-6).

The whole risk here is silently rewiring the board, so the netlist was diffed
rather than eyeballed:

  nets 519 -> 519, total pin connections 1563 -> 1563
  named nets present in both whose pin multiset changed: 0
  ERC unchanged at 14 errors / 20 warnings
  check_ucf.py: 99 balls matched, 0 failures

That last one matters most: it resolves the gateware's 113 UCF constraints to
board nets *by ball name*, so it is the sharpest detector of the corruption
this change could cause.

Two earlier attempts did cause exactly that. A bare quoted-string substitution
also rewrites FPGA ball names (C1, D2, N11, T1) and BTH-060 pin names (A1-D60),
which are spelled exactly like designators; one run left ERC identical while 40
nets came back with a different pin multiset. The tool now substitutes only at
the two positions that store an instance's designator, and excludes every pin
name everywhere else. docs/layout.md 9.5 records the hazard and how to prove a
renumber was clean.

Only the three scripts that read the design are updated. The gen_*/patch_*/
port_r1.py scripts keep the old names deliberately: each wrote a sheet once and
has not been re-runnable since it was hand-edited in Eeschema, so they are a
historical record -- and port_r1.py's dict keys are R1 designators that were
never renumbered at all.

Co-Authored-By: Claude Opus 5 <noreply@anthropic.com>
Claude-Session: https://claude.ai/code/session_01MHTAe6ZnhogTEgtyPcLhwG
Parts:
- renumbered C60 to C1000, C61 to C1001, C62 to C1002, C63 to C1003, C158 to C1004, C159 to C1005, J6 to J1000
Changed lines of the file:
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@@
 		(in_pos_files yes)
 		(dnp no)
-		(property "Reference" "C159"
+		(property "Reference" "C1005"
 			(at 104.14 156.21 90)
 			(show_name no)
@@
 			(project "r2"
 				(path "/dee825bf-c2f1-415d-afdf-cf702072a6e8/a2610316-2c52-4df4-b890-bf21654f6608"
-					(reference "C159")
+					(reference "C1005")
 					(unit 1)
 				)
@@
 		(in_pos_files yes)
 		(dnp no)
-		(property "Reference" "C62"
+		(property "Reference" "C1002"
 			(at 74.93 46.99 90)
 			(show_name no)
@@
 			(project "r2"
 				(path "/dee825bf-c2f1-415d-afdf-cf702072a6e8/a2610316-2c52-4df4-b890-bf21654f6608"
-					(reference "C62")
+					(reference "C1002")
 					(unit 1)
 				)
@@
 		(dnp no)
 		(fields_autoplaced yes)
-		(property "Reference" "J6"
+		(property "Reference" "J1000"
 			(at 142.24 91.7955 0)
 			(show_name no)
@@
 			(project "r2"
 				(path "/dee825bf-c2f1-415d-afdf-cf702072a6e8/a2610316-2c52-4df4-b890-bf21654f6608"
-					(reference "J6")
+					(reference "J1000")
 					(unit 1)
 				)
@@
 		(in_pos_files yes)
 		(dnp no)
-		(property "Reference" "C60"
+		(property "Reference" "C1000"
 			(at 105.41 153.67 90)
 			(show_name no)
@@
 			(project "r2"
 				(path "/dee825bf-c2f1-415d-afdf-cf702072a6e8/a2610316-2c52-4df4-b890-bf21654f6608"
-					(reference "C60")
+					(reference "C1000")
 					(unit 1)
 				)
@@
 		(in_pos_files yes)
 		(dnp no)
-		(property "Reference" "C63"
+		(property "Reference" "C1003"
 			(at 74.93 41.91 90)
 			(show_name no)
@@
 			(project "r2"
 				(path "/dee825bf-c2f1-415d-afdf-cf702072a6e8/a2610316-2c52-4df4-b890-bf21654f6608"
-					(reference "C63")
+					(reference "C1003")
 					(unit 1)
 				)
@@
 		(in_pos_files yes)
 		(dnp no)
-		(property "Reference" "C61"
+		(property "Reference" "C1001"
 			(at 74.93 52.07 90)
 			(show_name no)
@@
 			(project "r2"
 				(path "/dee825bf-c2f1-415d-afdf-cf702072a6e8/a2610316-2c52-4df4-b890-bf21654f6608"
-					(reference "C61")
+					(reference "C1001")
 					(unit 1)
 				)
@@
 		(in_pos_files yes)
 		(dnp no)
-		(property "Reference" "C158"
+		(property "Reference" "C1004"
 			(at 104.14 161.29 90)
 			(show_name no)
@@
 			(project "r2"
 				(path "/dee825bf-c2f1-415d-afdf-cf702072a6e8/a2610316-2c52-4df4-b890-bf21654f6608"
-					(reference "C158")
-					(unit 1)
-				)
+					(reference "C1004")
+					(unit 1)
+				)
