File: pcb/r2-mainboard/sic.kicad_sch (KiCad schematic)
At the start: 2 parts, among them IC1 OSD6254-1G-IPM, U1 OSD6254-1G-IPM

Commit message: Schematics update for new chip.
Parts:
- removed unit 11 of U1
- removed unit 9 of U1
- removed unit 4 of U1
- removed unit 10 of U1
- added C1500, C1519, C1534, C1535, C1536, C1540, C1542, C1544, C1545, C1546, C1547: 10uF/25V, Capacitor_SMD:C_0805_2012Metric, symbol Device:C
- added C1501, C1502, C1503, C1504, C1505, C1506, C1507, C1508, C1509, C1510, C1511, C1512, C1513, C1517, C1518, C1520, C1521, C1522, C1523, C1524, C1525, C1526, C1527, C1528, C1529: 100nF/50V, Capacitor_SMD:C_0402_1005Metric, symbol Device:C
- added C1514, C1530, C1531, C1532, C1533: 4.7uF/25V, Capacitor_SMD:C_0805_2012Metric, symbol Device:C
- added C1515, C1516: 1uF/25V, Capacitor_SMD:C_0402_1005Metric, symbol Device:C
- added C1537, C1538, C1539, C1541, C1543, C1549, C1550, C1551: 22uF/25V, Capacitor_SMD:C_0805_2012Metric, symbol Device:C
- added C1548: 1nF/50V, Capacitor_SMD:C_0402_1005Metric, symbol Device:C
- added C1552, C1553: 18pF/50V, Capacitor_SMD:C_0402_1005Metric, symbol Device:C
- added L1500, L1501, L1502: 0.47uH/4.9A, Inductor_SMD:L_1008_2520Metric, symbol Device:L
- added R1500, R1501, R1502, R1503, R1504, R1507, R1511, R1512, R1513, R1514, R1515, R1516, R1517, R1518, R1519, R1520, R1521, R1522, R1523, R1524: 10k/1%, Resistor_SMD:R_0402_1005Metric, symbol Device:R
- added R1505, R1506: 4.7k/1%, Resistor_SMD:R_0402_1005Metric, symbol Device:R
- added R1508, R1509: 100k/1%, Resistor_SMD:R_0402_1005Metric, symbol Device:R
- added R1510: 16.9k/1%, Resistor_SMD:R_0402_1005Metric, symbol Device:R
- added U1501: TPS6521903RHBR, Package_DFN_QFN:Texas_RHB0032E_VQFN-32-1EP_5x5mm_P0.5mm_EP3.45x3.45mm_ThermalVias, symbol Reflow:TPS6521903
- added U1502, U1503: TPS22965DSGR, Package_SON:Texas_DSG0008A_WSON-8-1EP_2x2mm_P0.5mm_EP0.9x1.6mm, symbol r2:TPS22965DSG
- added Y1: Crystal, symbol Device:Crystal
- added Y1500: SX3B25.000F1010F30, Crystal:Crystal_SMD_3225-4Pin_3.2x2.5mm, symbol Device:Crystal_GND24
- renumbered U1 to U600, IC1 to U600
Connections:
- net BOOT7: now reaches U600.D27 (GPMC0_AD7)
- net BOOT7: now also R1518.1
- net BOOT6: now reaches U600.D28 (GPMC0_AD6)
- net BOOT6: now also R1517.2
- net BOOT5: now reaches U600.E27 (GPMC0_AD5)
- net BOOT5: now also R1516.1
- net BOOT4: now reaches U600.E28 (GPMC0_AD4)
- net BOOT4: now also R1515.1
- net BOOT3: now reaches U600.F27 (GPMC0_AD3)
- net BOOT3: now also R1514.1
- net BOOT2: now reaches U600.F28 (GPMC0_AD2)
- net BOOT2: now also R1513.1
- net BOOT1: now reaches U600.G27 (GPMC0_AD1)
- net BOOT1: now also R1512.2
- net BOOT0: now reaches U600.G28 (GPMC0_AD0)
- net BOOT0: now also R1511.2
- net BOOT15: now reaches U600.H27 (GPMC0_AD15)
- net BOOT15: now also R1524.1
- net BOOT14: now reaches U600.H28 (GPMC0_AD14)
- net BOOT14: now also R1523.1
- net BOOT13: now reaches U600.J27 (GPMC0_AD13)
- net BOOT13: now also R1522.1
- net BOOT12: now reaches U600.J28 (GPMC0_AD12)
- net BOOT12: now also R1521.1
- net BOOT10: now reaches U600.K27 (GPMC0_AD10)
- net BOOT10: now also R1519.2
- net BOOT11: now reaches U600.K28 (GPMC0_AD11)
- net BOOT11: now also R1520.1
- net GND: now reaches U600.A14 (VSS)
- net GND: now also U600.A2 (VSS), U600.A27 (VSS), U600.B1 (VSS), U600.B14 (VSS), U600.B28 (VSS), U600.C14 (VSS), U600.C3 (VSS), U600.C4 (VSS), U600.D14 (VSS), U600.D3 (VSS), U600.D4 (VSS), U600.E10 (VSS), U600.E11 (VSS), U600.E12 (VSS), U600.E13 (VSS), U600.E16 (VSS), U600.E17 (VSS), U600.E18 (VSS), U600.E19 (VSS), U600.E20 (VSS), U600.E21 (VSS), U600.E22 (VSS), U600.E23 (VSS), U600.E24 (VSS), U600.E3 (VSS), U600.E4 (VSS), U600.E5 (VSS), U600.E6 (VSS), U600.E7 (VSS), U600.E8 (VSS), U600.E9 (VSS), U600.F19 (VSS), U600.F20 (VSS), U600.F21 (VSS), U600.F22 (VSS), U600.F23 (VSS), U600.F24 (VSS), U600.G19 (VSS), U600.G20 (VSS), U600.G23 (VSS), U600.G24 (VSS), U600.H1 (WKUP_LFOSC0_XI), U600.H19 (VSS), U600.H20 (VSS), U600.H24 (VSS), U600.J14 (VSS), U600.J15 (VSS), U600.J19 (VSS), U600.J20 (VSS), U600.J24 (VSS), U600.K14 (VSS), U600.K15 (VSS), U600.K19 (VSS), U600.K20 (VSS), U600.K24 (VSS), U600.K6 (VSS), U600.K7 (VSS), U600.K8 (VSS), U600.K9 (VSS), U600.L19 (VSS), U600.L20 (VSS), U600.L24 (VSS), U600.L5 (VSS), U600.L6 (VSS), U600.L7 (VSS), U600.L8 (VSS), U600.M20 (VSS), U600.M23 (VSS), U600.M24 (VSS), U600.M4 (VSS), U600.M5 (VSS), U600.M6 (VSS), U600.M7 (VSS), U600.N20 (VSS), U600.N21 (VSS), U600.N22 (VSS), U600.N23 (VSS), U600.N24 (VSS), U600.N3 (VSS), U600.N4 (VSS), U600.N5 (VSS), U600.N6 (VSS), U600.P16 (VSS), U600.P17 (VSS), U600.P18 (VSS), U600.P19 (VSS), U600.P20 (VSS), U600.P21 (VSS), U600.P22 (VSS), U600.P23 (VSS), U600.P24 (VSS), U600.P3 (VSS), U600.P4 (VSS), U600.P5 (VSS), U600.R3 (VSS), U600.R4 (VSS), U600.T19 (VSS), U600.T3 (VSS), U600.U1 (VSS), U600.U19 (VSS), U600.U28 (VSS), U600.V19 (VSS), U600.V2 (VSS), U600.V27 (VSS), C1500.2, C1501.2, C1502.2, C1503.2, C1504.2, C1505.2, C1506.2, C1507.2, C1508.2, C1509.2, C1510.2, C1511.2, C1512.2, C1513.2, C1514.2, C1515.2, C1516.2, C1517.2, C1518.2, C1519.2, C1520.2, C1521.2, C1522.2, C1523.2, C1524.2, C1525.2, C1526.2, C1527.2, C1528.2, C1529.2, C1530.2, C1531.2, C1532.2, C1533.2, C1534.2, C1535.2, C1536.2, C1537.2, C1538.2, C1539.2, C1540.2, C1541.2, C1542.2, C1543.2, C1544.2, C1545.2, C1546.2, C1547.2, C1548.2, C1549.2, C1550.2, C1551.2, C1552.2, C1553.2, R1508.2, R1510.2, R1513.2, R1514.2, R1515.2, R1516.2, R1518.2, R1520.2, R1521.2, R1522.2, R1523.2, R1524.2, U1501.15 (AGND), U1501.33 (PGND), U1502.5 (GND), U1502.9 (EP), U1503.5 (GND), U1503.9 (EP), Y1500.2 (G), Y1500.4 (G)
- net +0V75_SIC: now reaches U600.G12 (VDD_CANUART)
- net +0V75_SIC: now also U600.G13 (VDD_CORE), U600.G14 (VDD_CORE), U600.G15 (VDD_CORE), U600.G16 (VDD_CORE), U600.H12 (VDD_CORE), U600.H13 (VDD_CORE), U600.H14 (VDD_CORE), U600.H15 (VDD_CORE), U600.H16 (VDD_CORE), U600.J12 (VDD_CORE), U600.J13 (VDD_CORE), U600.J16 (VDD_CORE), U600.K12 (VDD_CORE), U600.K13 (VDD_CORE), U600.K16 (VDD_CORE), U600.L13 (VDD_CORE), U600.L14 (VDD_CORE), U600.L15 (VDD_CORE), U600.M12 (VDDA_CORE_USB), U600.M13 (VDDA_CORE_CSIRX0), C1500.1, C1501.1, C1502.1, C1503.1, C1504.1, C1505.1, C1506.1, C1539.1, C1540.1, C1549.1, L1500.2, U1501.1 (FB_B1)
- net +0V85_SIC: now reaches U600.H17 (VDDR_CORE)
- net +0V85_SIC: now also U600.H18 (VDDR_CORE), U600.J17 (VDDR_CORE), U600.J18 (VDDR_CORE), U600.K17 (VDDR_CORE), U600.K18 (VDDR_CORE), U600.L17 (VDDR_CORE), U600.L18 (VDDR_CORE), C1507.1, C1508.1, C1509.1, C1545.1, U1501.19 (VLDO2)
- net +1V2_SIC: now reaches U600.K10 (VDDS_DDR)
- net +1V2_SIC: now also U600.K11 (VDDS_DDR), U600.L10 (VDDS_DDR), U600.L11 (VDDS_DDR), U600.L9 (VDDS_DDR), U600.M10 (VDDS_DDR), U600.M8 (VDDS_DDR), U600.M9 (VDDS_DDR), U600.N8 (VDDS_DDR), U600.N9 (VDDS_DDR), C1510.1, C1511.1, C1512.1, C1543.1, C1544.1, C1551.1, L1502.2, U1501.24 (FB_B3)
- net +2V5_SIC: now reaches U600.N10 (DDR_VPP)
- net +2V5_SIC: now also C1513.1, C1547.1, U1501.23 (VLDO4)
- net OSC_XI: now reaches U600.G1 (MCU_OSC0_XI)
- net OSC_XI: now also C1552.1, Y1500.1
- net OSC_XO: now reaches U600.G2 (MCU_OSC0_XO)
- net OSC_XO: now also C1553.1, Y1500.3
- net VMON_VSYS: now reaches U600.A15 (VMON_VSYS)
- net VMON_VSYS: now also R1509.2, R1510.1
- net +3V3_SIC: now reaches U600.B15 (VMON_3P3_SOC)
- net +3V3_SIC: now also U600.F11 (VDDSHV_CANUART), U600.F12 (VDDSHV_MCU), U600.G10 (VDDSHV_CANUART), U600.G11 (VDDSHV_MCU), U600.G21 (VDDSHV5), U600.G22 (VDDSHV5), U600.H21 (VDDSHV6), U600.H22 (VDDSHV6), U600.J21 (VDDSHV0), U600.J22 (VDDSHV0), U600.K21 (VDDSHV1), U600.K22 (VDDSHV1), U600.L21 (VDDSHV3), U600.L22 (VDDSHV3), U600.M21 (VDDSHV2), U600.M22 (VDDSHV2), U600.N11 (VDDSHV4), U600.N7 (VDDA_3P3_USB), U600.P10 (VDDSHV4), C1519.1, C1520.1, C1521.1, C1522.1, C1523.1, C1524.1, C1525.1, C1526.1, C1527.1, C1528.1, C1529.1, R1501.1, R1502.1, R1503.1, R1505.1, R1506.1, R1511.1, R1512.1, R1517.1, R1519.1, U1502.7 (VOUT), U1502.8 (VOUT)
- net +1V8_SIC: now reaches U600.C15 (VMON_1P8_SOC)
- net +1V8_SIC: now also C1541.1, C1542.1, C1550.1, L1501.2, U1501.32 (FB_B2)
- net +1V8A_SIC: now reaches U600.D15 (VDDS_OSC0)
- net +1V8A_SIC: now also U600.F13 (VDDA_MCU), U600.F14 (VDDA_PLL2), U600.N12 (VDDA_TEMP), U600.N13 (VDDA_PLL0), U600.N14 (VDDA_PLL1), U600.P11 (VDDA_1P8_OLDI0), U600.P12 (VDDA_1P8_USB), U600.P13 (VDDA_1P8_CSIRX0), C1514.1, C1515.1, C1516.1, C1517.1, C1518.1, C1546.1, R1504.1, U1501.20 (PVIN_LDO2), U1501.21 (VLDO3), U1501.22 (PVIN_LDO34), U1501.6 (PVIN_LDO1)
- new net +3V3_DCDC: U1502.1 (VIN), U1502.2 (VIN), U1502.4 (VBIAS)
- new net +VSYS: U1503.1 (VIN), U1503.2 (VIN), U1503.4 (VBIAS)
- new net +VSYS_SIC: C1532.1, C1533.1, C1534.1, C1535.1, C1536.1, C1537.1, C1538.1, R1500.1, R1507.1, R1509.1, U1501.13 (VSYS), U1501.26 (PVIN_B3), U1501.30 (PVIN_B2), U1501.4 (PVIN_B1_1), U1501.5 (PVIN_B1_2), U1503.7 (VOUT), U1503.8 (VOUT)
- new net B1_SW: L1500.1, U1501.2 (LX_B1_1), U1501.3 (LX_B1_2)
- new net B2_SW: L1501.1, U1501.29 (LX_B2)
- new net B3_SW: L1502.1, U1501.27 (LX_B3)
- new net EXTINTN: R1503.2, U1501.11 (nINT)
- new net I2C0_SCL: R1506.2, U1501.10 (SCL)
- new net I2C0_SDA: R1505.2, U1501.9 (SDA)
- new net MCU_EN_SOC: R1508.1, U1503.3 (ON)
- new net MCU_PORZ: R1504.2, U1501.18 (nRSTOUT)
- new net PMIC_EN: R1500.2, U1501.25 (EN/PB/VSENSE)
- new net PMIC_GPO2: R1507.2, U1501.17 (GPO2), U1502.3 (ON)
- new net PMIC_LPM_EN0: R1501.2, U1501.31 (MODE/STBY)
- new net PMIC_VSEL: R1502.2, U1501.12 (VSEL_SD/VSEL_DDR)
- new net RESETSTATZ: U1501.28 (MODE/RESET)
- new net U1502_CT: C1548.1, U1502.6 (CT)
- new net VDD1P8: C1531.1, U1501.14 (VDD1P8)
- new net VLDO1_UNUSED: C1530.1, U1501.7 (VLDO1)
- no-connect marks 0 -> 5
Other:
- note added: "+0V75_SIC: 10 uF bulk + one 100 nF per VDD_CORE cluster (G13..K16, 18 balls)"
- note added: "+0V85_SIC: 3 x 100 nF at VDDR_CORE (H17..K18)"
- note added: "+1V2_SIC: 3 x 100 nF at VDDS_DDR (K10..M11)"
- note added: "+1V8A_SIC: 4.7 uF at CSIRX0 P13, 1 uF at OLDI0 P11, 1 uF bulk, 100 nF at PLL0/1/2 + MCU"
- note added: "+2V5_SIC: 100 nF at DDR_VPP N10"
- note added: "+3V3_SIC: 10 uF bulk + one 100 nF per VDDSHV ball pair (9 pairs) + 100 nF at VDDA_3P3_USB N7"
- note added: "BOOT3 up instead = eMMC boot (1001); BOOT8/BOOT9 are DPI_R6/R7 and live on dpi_in as R600/R601"
- note added: "Boot straps - docs/sic.md 6: PLL 011 = 25 MHz, primary boot 1000 = MMCSD, port 1 = SD, backup 001 = USB DFU"
- note added: "Decoupling, docs/sic.md §2 - the net is what the schematic fixes; these notes say where each part goes on the board (Octavo Table 4-3)"
- note added: "PMIC input bank and output capacitors - keep the 22 uF/10 uF pair at PVIN, the 47 uF + 10 uF at each buck output, close to U1501"
- note added: "Second 22 uF per buck output - replaces the 47 uF/1206, which LCSC does not stock (see tools/normalise_passives.py)"
- note added: "VMON_VSYS divider: trips the PMIC power-fail comparator (0.45 V) at 0.45 x (100k+16k9)/16k9 = 3.11 V at the cell"
- note added: "Y1500 25 MHz, CL 10 pF, ESR 30 ohm - load caps 2 x CL minus ~2 pF pin+trace; trim at bring-up (docs/sic.md 5)"
- moved on the sheet: U600A, U600B, U600C, U600E, U600F, U600G, U600H
